File: 4_Schematics and Boards Layout/4_6_Schematics/MainBoard/RADAR_Main_Board.brd (EAGLE design)
At the start: 260 x 300 mm, 791 parts, among them IC1 AT93C46A-10SQ-2.7, J1 142-0731-211, J18 142-0731-211, J19 CJT-T-P-HH-ST-TH1, J20 142-0731-211, J21 CJT-T-P-HH-ST-TH1, J22 142-0731-211, J23 142-0731-211, J24 142-0731-211, J25 142-0731-211, J26 142-0731-211, J27 142-0731-211, J28 142-0731-211, J29 142-0731-211, J30 142-0731-211, J31 142-0731-211, J32 142-0731-211, J33 142-0731-211, J34 142-0731-211, J35 142-0731-211, J36 142-0731-211, J37 142-0731-211, J38 142-0731-211, J39 142-0731-211, J40 142-0731-211, J41 142-0731-211, J42 142-0731-211, J43 142-0731-211, J44 142-0731-211, J45 142-0731-211, J46 142-0731-211, J47 142-0731-211, J48 142-0731-211, J49 142-0731-211, J50 142-0731-211, J51 142-0731-211, J52 142-0731-211, J53 142-0731-211, J54 142-0731-211, J55 142-0731-211, U1 AD9484BCPZ-500, U10 ADS7830IPWR, U11 INA241A3IDGKRDGK0008A-MFG, U13 LTC5552IUDBTRMPBF, U14 SZMMSZ5232BT1G, U15 SZMMSZ5232BT1G, U16 EP4RKU+, U17 SZMMSZ5232BT1G, U2 STM32F746ZGT7, U3 AD9708AR, U37 SZMMSZ5232BT1G, U38 SZMMSZ5232BT1G, U39 SZMMSZ5232BT1G, U4 AD8352ACPZ-R7, U40 SZMMSZ5232BT1G, U41 SZMMSZ5232BT1G, U42 XC7A50T-2FTG256I, U43 SZMMSZ5232BT1G, U44 SZMMSZ5232BT1G, U45 SZMMSZ5232BT1G, U46 SZMMSZ5232BT1G, U47 SZMMSZ5232BT1G, U48 SZMMSZ5232BT1G, U49 SZMMSZ5232BT1G, U5 LTC5552IUDBTRMPBF, U50 SZMMSZ5232BT1G, U51 SZMMSZ5232BT1G, U52 SZMMSZ5232BT1G, U53 SZMMSZ5232BT1G, U54 SZMMSZ5232BT1G, U55 SZMMSZ5232BT1G, U56 SZMMSZ5232BT1G, U57 SZMMSZ5232BT1G, U58 SZMMSZ5232BT1G, U59 SZMMSZ5232BT1G, U6 FT2232HQ, U60 SZMMSZ5232BT1G, U61 SZMMSZ5232BT1G, U62 SZMMSZ5232BT1G, U63 SZMMSZ5232BT1G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

Commit message: fix(hw): take the first IF stage from 10 dB to 15 dB (Lane B B1.2)
Stage 1 (`U4`) is set for 10 dB and stage 2 (`U8`) for 15 dB, so the cascade is
25 dB against the ~30 dB the ADC wants. Both stages are AD8352s whose gain comes
from R_G, and the datasheet (Table 5, 200 ohm load) gives 115 ohm for 10 dB and
56 ohm for 15 dB.

Table 5 also pairs each gain with a distortion-cancellation network -- CD of
0.2 pF at 10 dB and 0.6 pF at 15 dB, RD = 4.3k either way -- and stage 2 is built
exactly that way (R22 = 56R, C54 = 0.6pF). So stage 1 needs *two* parts changed,
not one:

    R14  115R  -> 56R      (gain resistor, U4.RGN/U4.RGP)
    C43  0.2pF -> 0.6pF    (CD, with R15 = 4.3k on U4.RDP/U4.RDN)

Changing only R14 would have re-tuned stage 1's distortion cancellation while
claiming a gain change -- the board-respin spec said exactly that, and it is
corrected along with the prefab checklist and the fix plan.

Both replacement part numbers are copied from the stage that already runs at
15 dB in the same BOM, so no MPN was invented:
    RC0201FR-07115RL    -> RC0201FR-0756RL      (as R22)
    GJM0335C1ER20WB01D  -> GJM0335C1ER60WB01D   (as C54)

Applied to the schematic, the board and the production BOM together. Verified:
the CAD files re-parse with identical structure (1978 parts / 744 nets / 2462
segments in the .sch, 791 elements in the .brd), the diff is exactly the four
intended attribute lines, the xlsx round-trip differs in exactly the four
intended cells, and all three artifact gates stay green -- the board/BOM
consistency gate is what proves the three files agree.
Parts:
- C43: value 0.2pF -> 0.6pF
- R14: value 115R -> 56R
Changed lines of the file:
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@@
 <attribute name="VALUE" x="66.115" y="217.975" size="1.27" layer="27" rot="R180"/>
 </element>
-<element name="C43" library="rcl" package="C0201" value="0.2pF" x="58.6" y="142.075" smashed="yes" rot="R180">
+<element name="C43" library="rcl" package="C0201" value="0.6pF" x="58.6" y="142.075" smashed="yes" rot="R180">
 <attribute name="NAME" x="59.235" y="141.44" size="1.27" layer="25" rot="R180"/>
 <attribute name="POPULARITY" value="0" x="-232.23" y="434.175" size="1.778" layer="27" rot="R180" display="off"/>
@@
 <attribute name="VALUE" x="69.665" y="172.4" size="1.27" layer="27" rot="R180"/>
 </element>
-<element name="R14" library="rcl" package="R0201" value="115R" x="58.605" y="143.275" smashed="yes" rot="R180">
+<element name="R14" library="rcl" package="R0201" value="56R" x="58.605" y="143.275" smashed="yes" rot="R180">
 <attribute name="NAME" x="59.24" y="142.64" size="1.27" layer="25" rot="R180"/>
 <attribute name="POPULARITY" value="0" x="-86.175" y="450.615" size="1.778" layer="27" rot="R180" display="off"/>

Commit message: fix(hw): move the PA sense chain to the INA241A4 (Lane B B2.5)
The current-sense amplifier is not on the PA board at all -- the shunt (`R10`,
5 mOhm) is, and 16 x `INA241A3IDGKR` on the main board (`U11`, `U73`-`U87`) read
it.  At the A3's 50 V/V into the ADS7830's 2.5 V internal reference the span is
10 A at 39.2 mA/LSB, so the 1.68 A bias target sits at only 17 % of span.

Decision (owner): INA241A4 = 100 V/V.  TI's datasheet lists the gain options as
10/20/50/100/200 V/V for A1/A2/A3/A4/B4, and the A4 shares the A3's DGK/VSSOP-8
package and pinout, so this is a part-number change with no layout impact:

    span         10 A   -> 5 A
    resolution   39.2   -> 19.6 mA/LSB
    1.68 A       17 %   -> 34 % of span      (2.5 A trip still inside 5 A)

Changed together: the schematic (library deviceset *and* the 16 references --
Eagle resolves the symbol from that name, so leaving it at A3 would describe a
different part than the BOM buys), the board's 16 elements, the production BOM
(value, device and MPN) and `PA_INA_GAIN`.  The gain string occurs in three
shapes that share one literal, so the replacement is counted (21 in the .sch,
32 in the .brd) rather than pattern-guessed.

Tests moved to the Rev B chain, including the ones that encoded the superseded
numbers: `test_pa_sense` now expects a 5 A span, 19.6 mA/LSB, target code 86 (was
43) and the 0.1 ohm-shunt diagnostic's 0.25 A full scale; the legacy gap-3
re-read test carried its own copy of the *old* formula (3.3 V reference and gain
50, i.e. the 32 %-low chain Phase 1 replaced), so its local formula and raw
values were brought onto the chain the firmware actually uses.

Verified: CAD structure unchanged (1978 parts / 791 elements), zero stale A3
references, the xlsx differs from HEAD in exactly 3 cells, all three artifact
gates stay green (the board/BOM consistency gate is what proves the three files
agree), MCU suite 26/26 and `test_pa_sense` 6/6.
Parts:
- U11, U73, U74, U75, U76, U77, U78, U79, U80, U81, U82, U83, U84, U85, U86, U87: value INA241A3IDGKRDGK0008A-MFG -> INA241A4IDGKRDGK0008A-MFG

Commit message: feat(hw): cavity-filter interface on the main board (Lane B B1.3)
Decision (owner): cavity filters rather than microstrip, because >= 40 dB of image
rejection 240 MHz from a 10.5 GHz passband is not a microstrip-with-tuning job.
The filter is therefore off-board, which means the board needs launches and the
two 2-pin `BPF2` placeholders (`U$2`, `U$3`) no longer represent anything.

Added, using only devices that already exist in the repo's libraries:

    4 x SMA jack `142-0731-211`   (J56-J59)  -- the deviceset, symbol and
                                              package were already present
    2 x 0R bridge                 (R174, R175) -- R-EU_ R0201, MPN copied from
                                              the existing 0R parts (R18/R19/
                                              R34/R35 -> RCA02010000ZSEDSR)

Topology: one launch at each end of each off-board filter -- J56 on RF_TX_FIL,
J57 on RF_TX, J58 on RF_RX, J59 on RF_RX_FIL -- with the SMA legs (pads 2-5) on
GND, and a 0R across each pair as the bench bypass so the chain can be brought up
without the filters.  The placeholders are removed rather than left in the signal
path, together with their board contactrefs.

Placement was searched, not guessed: for each new part the closest free position
to its anchor that keeps clearance from every existing element (6.5 mm for the
SMA jacks, 2.2 mm for the resistors) -- achieved 6.6-14.2 mm and 2.7-5.6 mm, and
the pairs stay 13-21 mm apart so a bolt-on cavity can reach both ports.

Verified: both CAD files parse with the expected structure (1982 parts / 795
elements, i.e. -2 placeholders +6 parts), no `U$2`/`U$3` reference survives on
this board, each RF net carries its original part plus the launch centre pin and
one bridge pin, the RF sheet's GND gains the 16 SMA leg pins, and all three
artifact gates are green -- the board/BOM gate is what proves the three files
agree.  DNP_list.csv regenerated: the two placeholders give way to the two
bench-bypass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
Parts:
- removed U$2, U$3: BPF2, My_Library_RADAR:BPF2
- added J56, J57, J58, J59: 142-0731-211, 142-0731-211:1420731211
- added R174, R175: 0R, rcl:R0201
Connections:
- net GND: now also J56.2, J56.3, J56.4, J56.5, J57.2, J57.3, J57.4, J57.5, J58.2, J58.3, J58.4, J58.5, J59.2, J59.3, J59.4, J59.5
- net RF_RX: now also J58.1, R175.1; no longer U$3.P$1
- net RF_RX_FIL: now also J59.1, R175.2; no longer U$3.P$2
- net RF_TX: now also J57.1, R174.2; no longer U$2.P$2
- net RF_TX_FIL: now also J56.1, R174.1; no longer U$2.P$1
Routing:
- net RF_TX_FIL: track 42.1 -> 32.0 mm
- net RF_RX_FIL: track 42.3 -> 35.2 mm
Changed lines of the file:
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@@
 </pass>
 </autorouter>
-<elements>
+<elements><element name="J56" library="142-0731-211" package="1420731211" value="142-0731-211" x="100.86" y="212.01" smashed="yes"/><element name="J57" library="142-0731-211" package="1420731211" value="142-0731-211" x="101.86" y="233.0" smashed="yes"/><element name="J58" library="142-0731-211" package="1420731211" value="142-0731-211" x="71.0" y="162.0" smashed="yes"/><element name="J59" library="142-0731-211" package="1420731211" value="142-0731-211" x="84.0" y="160.0" smashed="yes"/><element name="R174" library="rcl" package="R0201" value="0R" x="110.0" y="220.0" smashed="yes"/><element name="R175" library="rcl" package="R0201" value="0R" x="77.0" y="169.0" smashed="yes"/>
 <element name="C1" library="eagle-ltspice" package="C0201" value="0.1uF" x="64.52" y="156.43" smashed="yes">
 <attribute name="NAME" x="63.885" y="157.065" size="1.27" layer="25"/>
@@
 <attribute name="VALUE" x="137.768421875" y="129.355259375" size="0.508" layer="27" rot="R315"/>
 </element>
-<element name="U$2" library="My_Library_RADAR" package="BPF2" value="BPF2" x="100.86" y="212.01" smashed="yes" rot="R180"/>
-<element name="U$3" library="My_Library_RADAR" package="BPF2" value="BPF2" x="82.72" y="146.97" smashed="yes"/>
 <element name="RF_SW_3" library="My_Library_RADAR" package="16_QFN" value="M3SWA2-34DR+" x="136.16" y="230.16" smashed="yes" rot="R225">
 <attribute name="VALUE" x="138.315259375" y="229.441578125" size="0.508" layer="27" rot="R225"/>
@@
 <wire x1="52.948040625" y1="145.5082" x2="52.948040625" y2="146.0495" width="0.2" layer="1"/>
 <wire x1="52.948040625" y1="146.0495" x2="52.962915625" y2="146.064375" width="0.2" layer="1"/>
-</signal>
+<contactref element="J56" pad="2"/><contactref element="J56" pad="3"/><contactref element="J56" pad="4"/><contactref element="J56" pad="5"/><contactref element="J57" pad="2"/><contactref element="J57" pad="3"/><contactref element="J57" pad="4"/><contactref element="J57" pad="5"/><contactref element="J58" pad="2"/><contactref element="J58" pad="3"/><contactref element="J58" pad="4"/><contactref element="J58" pad="5"/><contactref element="J59" pad="2"/><contactref element="J59" pad="3"/><contactref element="J59" pad="4"/><contactref element="J59" pad="5"/></signal>
 <signal name="+1V8_FPGA">
 <contactref element="X10" pad="1"/>
@@
 <signal name="RF_RX" class="2">
 <contactref element="U13" pad="5"/>
-<contactref element="U$3" pad="P$1"/>
 <wire x1="82.72" y1="147.07" x2="82.754690625" y2="147.035309375" width="0.204" layer="1"/>
 <wire x1="82.76" y1="145.5025" x2="82.754690625" y2="147.035309375" width="0.204" layer="1"/>
-</signal>
+<contactref element="J58" pad="1"/><contactref element="R175" pad="1"/></signal>
 <signal name="DAC_IOUT_F_P" class="1">
 <contactref element="U5" pad="2"/>
@@
 <signal name="RF_TX" class="2">
 <contactref element="U5" pad="5"/>
-<contactref element="U$2" pad="P$2"/>
 <wire x1="82.49" y1="213.0575" x2="82.49" y2="212.018640625" width="0.204" layer="1"/>
 <wire x1="82.49" y1="212.018640625" x2="82.445" y2="211.91" width="0.204" layer="1" curve="-45"/>
-</signal>
+<contactref element="J57" pad="1"/><contactref element="R174" pad="2"/></signal>
 <signal name="N$21" class="2">
 <contactref element="U$1" pad="3"/>
@@
 <signal name="RF_TX_FIL" class="2">
 <contactref element="C83" pad="1"/>
-<contactref element="U$2" pad="P$1"/>
-<wire x1="111.220275" y1="212.15" x2="101.1" y2="212.15" width="0.204" layer="1"/>
+="101.1" y2="212.15" width="0.204" layer="1"/>
 <wire x1="111.220275" y1="212.15" x2="115.910275" y2="207.46" width="0.204" layer="1" curve="-90"/>
 <wire x1="115.910275" y1="207.46" x2="115.910275" y2="182.418484375" width="0.204" layer="1"/>
 <wire x1="101.1" y1="212.15" x2="100.86" y2="211.91" width="0.204" layer="1" curve="90"/>
-</signal>
+<contactref element="J56" pad="1"/><contactref element="R174" pad="1"/></signal>
 <signal name="RF_IO" class="2">
 <contactref element="C85" pad="2"/>
@@
 <signal name="RF_RX_FIL" class="2">
 <contactref element="C84" pad="2"/>
-<contactref element="U$3" pad="P$2"/>
-<wire x1="115.93445" y1="151.57" x2="110.93445" y2="146.57" width="0.204" layer="1" curve="-90"/>
+"110.93445" y2="146.57" width="0.204" layer="1" curve="-90"/>
 <wire x1="115.93445" y1="151.57" x2="115.93445" y2="176.76614375" width="0.204" layer="1"/>
 <wire x1="110.93445" y1="146.57" x2="101.635" y2="146.57" width="0.204" layer="1"/>
 <wire x1="101.635" y1="146.57" x2="101.135" y2="147.07" width="0.204" layer="1" curve="-90"/>
-</signal>
+<contactref element="J59" pad="1"/><contactref element="R175" pad="2"/></signal>
 <signal name="RF_IO_2" class="2">
 <contactref element="U16" pad="10"/>
