File: 4_Schematics and Boards Layout/4_6_Schematics/MainBoard/RADAR_Main_Board.brd (EAGLE design)
At the start: 260 x 300 mm, 795 parts, among them IC1 AT93C46A-10SQ-2.7, J1 142-0731-211, J18 142-0731-211, J19 CJT-T-P-HH-ST-TH1, J20 142-0731-211, J21 CJT-T-P-HH-ST-TH1, J22 142-0731-211, J23 142-0731-211, J24 142-0731-211, J25 142-0731-211, J26 142-0731-211, J27 142-0731-211, J28 142-0731-211, J29 142-0731-211, J30 142-0731-211, J31 142-0731-211, J32 142-0731-211, J33 142-0731-211, J34 142-0731-211, J35 142-0731-211, J36 142-0731-211, J37 142-0731-211, J38 142-0731-211, J39 142-0731-211, J40 142-0731-211, J41 142-0731-211, J42 142-0731-211, J43 142-0731-211, J44 142-0731-211, J45 142-0731-211, J46 142-0731-211, J47 142-0731-211, J48 142-0731-211, J49 142-0731-211, J50 142-0731-211, J51 142-0731-211, J52 142-0731-211, J53 142-0731-211, J54 142-0731-211, J55 142-0731-211, J56 142-0731-211, J57 142-0731-211, J58 142-0731-211, J59 142-0731-211, U1 AD9484BCPZ-500, U10 ADS7830IPWR, U11 INA241A4IDGKRDGK0008A-MFG, U13 LTC5552IUDBTRMPBF, U14 SZMMSZ5232BT1G, U15 SZMMSZ5232BT1G, U16 EP4RKU+, U17 SZMMSZ5232BT1G, U2 STM32F746ZGT7, U3 AD9708AR, U37 SZMMSZ5232BT1G, U38 SZMMSZ5232BT1G, U39 SZMMSZ5232BT1G, U4 AD8352ACPZ-R7, U40 SZMMSZ5232BT1G, U41 SZMMSZ5232BT1G, U42 XC7A50T-2FTG256I, U43 SZMMSZ5232BT1G, U44 SZMMSZ5232BT1G, U45 SZMMSZ5232BT1G, U46 SZMMSZ5232BT1G, U47 SZMMSZ5232BT1G, U48 SZMMSZ5232BT1G, U49 SZMMSZ5232BT1G, U5 LTC5552IUDBTRMPBF, U50 SZMMSZ5232BT1G, U51 SZMMSZ5232BT1G, U52 SZMMSZ5232BT1G, U53 SZMMSZ5232BT1G, U54 SZMMSZ5232BT1G, U55 SZMMSZ5232BT1G, U56 SZMMSZ5232BT1G, U57 SZMMSZ5232BT1G, U58 SZMMSZ5232BT1G, U59 SZMMSZ5232BT1G, U6 FT2232HQ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

Commit message: feat(hw): bank 14 to 2.5 V with level-shifted QSPI lines (Lane B B1.1, part 2 of 2)
The half that actually changes the bank.  `VCCO_14` moves to the 2.5 V rail part 1
put on the power board, and because the configuration flash shares that net and is
a 3 V part, every line between the flash and the FPGA is split:

    FPGA_FLASH_DQ0   U42 + U90.A1   ->  FLASH_DQ0_F   U9.DQ0 + U90.B1
    FPGA_FLASH_DQ1   U42 + U90.A2   ->  FLASH_DQ1_F   U9.DQ1 + U90.B2
    FPGA_FLASH_DQ2   U42 + U90.A3   ->  FLASH_DQ2_F   U9.W/DQ2 + U90.B3
    FPGA_FLASH_DQ3   U42 + U90.A4   ->  FLASH_DQ3_F   U9.DQ3/HOLD + U90.B4
    FPGA_FLASH_NCS   U42 + U91.A1   ->  FLASH_NCS_F   U9.S + U91.B1
    FPGA_FLASH_NRST  U42 + U91.A2   ->  FLASH_NRST_F  U9.RESET + U91.B2

`U9.VCC` stays on +3V3_FPGA -- that is the whole point of the split, and it is
asserted below because getting it wrong silently bricks configuration.  DQ0..DQ3
use the 4-bit auto-direction part (they change direction inside a transaction and
the config engine cannot drive a direction pin); FCS_B and D07 use the 2-bit part.
Also added: OE pull-ups to the 2.5 V side, decoupling on both translator supplies,
decoupling for the newly split bank, and the 2-pin Molex that receives the rail.

Verified from the written files: both parse (1993 parts / 806 elements); each
FPGA-side net carries the FPGA ball and the A-side pin while its `_F` twin carries
the flash pin and the B-side pin; all six `VCCO_14` ball pads (L16, M13, N10, P7,
R14, T11) are on +2V5_FPGA and none remains on +3V3_FPGA while `VCCO_0/15/35` stay
at 3.3 V; and `element="U9"` appears only on the 3.3 V rail.  All three artifact
gates green, and interboard_rails now shows +2V5_FPGA spanning both boards.

Two mistakes of mine that the verification caught, both on the board side and both
fixed before this commit: `VCCO_14` is six BGA balls, not one, so a single
"remove the first U42 contactref" also stripped `VCCO_0`'s pad and a guessed pad
number went onto the new rail.  The schemati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
Parts:
- added C354, C355, C356, C357, C358, C359: 0.1uF, rcl:C0201
- added R176, R177: 10k, rcl:R0201
- added U90: TXS0104EPWR, My_Library_RADAR:PW0014A-MFG
- added U91: TXS0102DCUR, My_Library_RADAR:DCU0008A-MFG
- added X57: 22-23-2021, con-molex:22-23-2021
Connections:
- new net +2V5_FPGA: C354.1, C355.1, C358.1, C359.1, R176.2, R177.2, U42.L16, U42.M13, U42.N10, U42.P7, U42.R14, U42.T11, U90.1, U91.3, X57.1
- new net FLASH_DQ0_F: U9.D3, U90.13
- new net FLASH_DQ1_F: U9.D2, U90.12
- new net FLASH_DQ2_F: U9.C4, U90.11
- new net FLASH_DQ3_F: U9.D4, U90.10
- new net FLASH_NCS_F: U9.C2, U91.8
- new net FLASH_NRST_F: U9.A4, U91.1
- new net N$U90_OE: R176.1, U90.8
- new net N$U91_OE: R177.1, U91.6
- net +3V3_FPGA: now also C356.1, C357.1, U90.14, U91.7; no longer C110.2, C112.2, C17.2, U42.L16, U42.M13, U42.N10, U42.P7, U42.R14, U42.T11
- net FPGA_FLASH_DQ0: now also U90.2; no longer U9.D3
- net FPGA_FLASH_DQ1: now also U90.3; no longer U9.D2
- net FPGA_FLASH_DQ2: now also U90.4; no longer U9.C4
- net FPGA_FLASH_DQ3: now also U90.5; no longer U9.D4
- net FPGA_FLASH_NCS: now also U91.5; no longer U9.C2
- net FPGA_FLASH_NRST: now also U91.4; no longer U9.A4
- net GND: now also C354.2, C355.2, C356.2, C357.2, C358.2, C359.2, U90.7, U91.2, X57.2
Changed lines of the file:
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@@
 </pass>
 </autorouter>
-<elements><element name="J56" library="142-0731-211" package="1420731211" value="142-0731-211" x="100.86" y="212.01" smashed="yes"/><element name="J57" library="142-0731-211" package="1420731211" value="142-0731-211" x="101.86" y="233.0" smashed="yes"/><element name="J58" library="142-0731-211" package="1420731211" value="142-0731-211" x="71.0" y="162.0" smashed="yes"/><element name="J59" library="142-0731-211" package="1420731211" value="142-0731-211" x="84.0" y="160.0" smashed="yes"/><element name="R174" library="rcl" package="R0201" value="0R" x="110.0" y="220.0" smashed="yes"/><element name="R175" library="rcl" package="R0201" value="0R" x="77.0" y="169.0" smashed="yes"/>
+<elements><element name="U90" library="My_Library_RADAR" package="PW0014A-MFG" value="TXS0104EPWR" x="36.68" y="149.28" smashed="yes"/><element name="U91" library="My_Library_RADAR" package="DCU0008A-MFG" value="TXS0102DCUR" x="23.04" y="192.82" smashed="yes"/><element name="R176" library="rcl" package="R0201" value="10k" x="56.0" y="196.0" smashed="yes"/><element name="R177" library="rcl" package="R0201" value="10k" x="32.0" y="200.0" smashed="yes"/><element name="C354" library="rcl" package="C0201" value="0.1uF" x="44.0" y="170.0" smashed="yes"/><element name="C355" library="rcl" package="C0201" value="0.1uF" x="52.0" y="170.0" smashed="yes"/><element name="C356" library="rcl" package="C0201" value="0.1uF" x="44.0" y="198.0" smashed="yes"/><element name="C357" library="rcl" package="C0201" value="0.1uF" x="52.0" y="198.0" smashed="yes"/><element name="C358" library="rcl" package="C0201" value="0.1uF" x="36.0" y="170.0" smashed="yes"/><element name="C359" library="rcl" package="C0201" value="0.1uF" x="36.0" y="198.0" smashed="yes"/><element name="X57" library="con-molex" package="22-23-2021" value="22-23-2021" x="6.02" y="230.0" smashed="yes"/><element name="J56" library="142-0731-211" package="1420731211" value="142-0731-211" x="100.86" y="212.01" smashed="yes"/><element name="J57" library="142-0731-211" package="1420731211" value="142-0731-211" x="101.86" y="233.0" smashed="yes"/><element name="J58" library="142-0731-211" package="1420731211" value="142-0731-211" x="71.0" y="162.0" smashed="yes"/><element name="J59" library="142-0731-211" package="1420731211" value="142-0731-211" x="84.0" y="160.0" smashed="yes"/><element name="R174" library="rcl" package="R0201" value="0R" x="110.0" y="220.0" smashed="yes"/><element name="R175" library="rcl" package="R0201" value="0R" x="77.0" y="169.0" smashed="yes"/>
 <element name="C1" library="eagle-ltspice" package="C0201" value="0.1uF" x="64.52" y="156.43" smashed="yes">
 <attribute name="NAME" x="63.885" y="157.065" size="1.27" layer="25"/>
@@
 </element>
 </elements>
-<signals>
+<signals><signal name="N$U91_OE" class="0"><contactref element="U91" pad="6"/><contactref element="R177" pad="1"/></signal><signal name="N$U90_OE" class="0"><contactref element="U90" pad="8"/><contactref element="R176" pad="1"/></signal><signal name="+2V5_FPGA" class="0"><contactref element="U90" pad="1"/><contactref element="U91" pad="3"/><contactref element="R176" pad="2"/><contactref element="R177" pad="2"/><contactref element="C354" pad="1"/><contactref element="C355" pad="1"/><contactref element="C358" pad="1"/><contactref element="C359" pad="1"/><contactref element="X57" pad="1"/><contactref element="U42" pad="L16"/><contactref element="U42" pad="M13"/><contactref element="U42" pad="N10"/><contactref element="U42" pad="P7"/><contactref element="U42" pad="R14"/><contactref element="U42" pad="T11"/></signal><signal name="FLASH_NRST_F" class="0"><contactref element="U9" pad="A4"/><contactref element="U91" pad="1"/></signal><signal name="FLASH_NCS_F" class="0"><contactref element="U9" pad="C2"/><contactref element="U91" pad="8"/></signal><signal name="FLASH_DQ3_F" class="0"><contactref element="U9" pad="D4"/><contactref element="U90" pad="10"/></signal><signal name="FLASH_DQ2_F" class="0"><contactref element="U9" pad="C4"/><contactref element="U90" pad="11"/></signal><signal name="FLASH_DQ1_F" class="0"><contactref element="U9" pad="D2"/><contactref element="U90" pad="12"/></signal><signal name="FLASH_DQ0_F" class="0"><contactref element="U9" pad="D3"/><contactref element="U90" pad="13"/></signal>
 <signal name="+3V3">
 <contactref element="X24" pad="1"/>
@@
 <wire x1="52.948040625" y1="145.5082" x2="52.948040625" y2="146.0495" width="0.2" layer="1"/>
 <wire x1="52.948040625" y1="146.0495" x2="52.962915625" y2="146.064375" width="0.2" layer="1"/>
-<contactref element="J56" pad="2"/><contactref element="J56" pad="3"/><contactref element="J56" pad="4"/><contactref element="J56" pad="5"/><contactref element="J57" pad="2"/><contactref element="J57" pad="3"/><contactref element="J57" pad="4"/><contactref element="J57" pad="5"/><contactref element="J58" pad="2"/><contactref element="J58" pad="3"/><contactref element="J58" pad="4"/><contactref element="J58" pad="5"/><contactref element="J59" pad="2"/><contactref element="J59" pad="3"/><contactref element="J59" pad="4"/><contactref element="J59" pad="5"/></signal>
+<contactref element="J56" pad="2"/><contactref element="J56" pad="3"/><contactref element="J56" pad="4"/><contactref element="J56" pad="5"/><contactref element="J57" pad="2"/><contactref element="J57" pad="3"/><contactref element="J57" pad="4"/><contactref element="J57" pad="5"/><contactref element="J58" pad="2"/><contactref element="J58" pad="3"/><contactref element="J58" pad="4"/><contactref element="J58" pad="5"/><contactref element="J59" pad="2"/><contactref element="J59" pad="3"/><contactref element="J59" pad="4"/><contactref element="J59" pad="5"/><contactref element="U90" pad="7"/><contactref element="U91" pad="2"/><contactref element="C354" pad="2"/><contactref element="C355" pad="2"/><contactref element="C356" pad="2"/><contactref element="C357" pad="2"/><contactref element="C358" pad="2"/><contactref element="C359" pad="2"/><contactref element="X57" pad="2"/></signal>
 <signal name="+1V8_FPGA">
 <contactref element="X10" pad="1"/>
@@
 <signal name="+3V3_FPGA">
 <contactref element="X16" pad="1"/>
-<contactref element="U42" pad="L6"/>
 <contactref element="C176" pad="2"/>
 <contactref element="C182" pad="2"/>
@@
 <contactref element="C177" pad="2"/>
 <contactref element="C178" pad="2"/>
-<contactref element="U42" pad="L16"/>
-<contactref element="U42" pad="M13"/>
-<contactref element="U42" pad="N10"/>
-<contactref element="U42" pad="P7"/>
-<contactref element="U42" pad="R14"/>
-<contactref element="U42" pad="T11"/>
-<contactref element="C17" pad="2"/>
+>
+>
 <contactref element="C113" pad="2"/>
-<contactref element="C112" pad="2"/>
 <contactref element="C111" pad="2"/>
-<contactref element="C110" pad="2"/>
 <contactref element="C108" pad="2"/>
 <contactref element="C109" pad="2"/>
@@
 <wire x1="60.52" y1="184.72" x2="60.925" y2="184.315" width="0.1" layer="12"/>
 <wire x1="60.925" y1="184.315" x2="60.925" y2="184.025" width="0.1" layer="12"/>
-</signal>
+<contactref element="U90" pad="14"/><contactref element="U91" pad="7"/><contactref element="C356" pad="1"/><contactref element="C357" pad="1"/><contactref element="U42" pad="L6"/></signal>
 <signal name="-5V5_PA">
 <contactref element="X19" pad="1"/>
@@
 </signal>
 <signal name="FPGA_FLASH_NRST">
-<contactref element="U9" pad="A4"/>
 <contactref element="R50" pad="1"/>
 <contactref element="U42" pad="L13"/>
@@
 <wire x1="71.201834375" y1="183.998165625" x2="71.1" y2="184.1" width="0.1" layer="16"/>
 <via x="71.1" y="184.1" extent="1-16" drill="0.15"/>
-</signal>
+<contactref element="U91" pad="4"/></signal>
 <signal name="N$25" class="2">
 <contactref element="U9" pad="B2"/>
@@
 </signal>
 <signal name="FPGA_FLASH_NCS">
-<contactref element="U9" pad="C2"/>
 <contactref element="R52" pad="1"/>
 <contactref element="U42" pad="L12"/>
@@
 <via x="30.65" y="182.9" extent="1-16" drill="0.15"/>
 <via x="29.4" y="182.9" extent="1-16" drill="0.15"/>
-</signal>
+<contactref element="U91" pad="5"/></signal>
 <signal name="FPGA_FLASH_DQ2">
-<contactref element="U9" pad="C4"/>
 <contactref element="R53" pad="1"/>
 <contactref element="U42" pad="K15"/>
@@
 <via x="39.65" y="182.4" extent="1-16" drill="0.15"/>
 <via x="31.3" y="182.6" extent="1-16" drill="0.15"/>
-</signal>
+<contactref element="U90" pad="4"/></signal>
 <signal name="FPGA_FLASH_DQ1">
-<contactref element="U9" pad="D2"/>
 <contactref element="U42" pad="J14"/>
 <wire x1="55.18" y1="182.78" x2="55.551234375" y2="182.408765625" width="0.15" layer="1"/>
@@
 <wire x1="23.55" y1="184.3" x2="23.5329" y2="184.3370125" width="0.1" layer="14"/>
 <wire x1="55.6" y1="182.4" x2="55.551234375" y2="182.408765625" width="0.1" layer="14"/>
-</signal>
+<contactref element="U90" pad="3"/></signal>
 <signal name="FPGA_FLASH_DQ0">
-<contactref element="U9" pad="D3"/>
 <contactref element="U42" pad="J13"/>
 <wire x1="54.18" y1="182.78" x2="54.551234375" y2="182.408765625" width="0.15" layer="1"/>
@@
 <wire x1="22.6" y1="185.3" x2="22.57865625" y2="185.3312625" width="0.1" layer="12"/>
 <wire x1="54.6" y1="182.45" x2="54.551234375" y2="182.408765625" width="0.1" layer="12"/>
-</signal>
+<contactref element="U90" pad="2"/></signal>
 <signal name="FPGA_FLASH_DQ3">
-<contactref element="U9" pad="D4"/>
 <contactref element="R54" pad="2"/>
 <contactref element="U42" pad="K16"/>
@@
 <via x="47.6" y="189.1" extent="1-16" drill="0.15"/>
 <via x="41.3" y="189.1" extent="1-16" drill="0.15"/>
-</signal>
+<contactref element="U90" pad="5"/></signal>
 <signal name="FPGA_PUDC_B">
 <contactref element="U42" pad="L15"/>

Commit message: feat(hw): gate-bias fail-safe, negative-rail margin, PA drain bulk (Lane B B2.2/B1.5/B2.3)
B2.2 -- and this is the finding that matters.  Every one of the 16 gate-bias
channels is an inverting amplifier referenced to ground (Vout = -(Rf/Rin) x VDAC,
+ input on GND), so a DAC in reset puts **0 V on all 16 gates**.  QPA2962 is a
depletion-mode GaN HEMT, where 0 V means *fully on* -- with 22 V on the drains.
That is a power-up hazard, not a nuance.

The plan frames the fix as hardware default *plus* MCU sequence; the hardware half
is here.  One 10k pull-down per channel from VGn to the same negative rail that
supplies its op-amp (R178-R193), so the gates sit at the negative rail whenever
the op-amps are not actively driving: during power-up, power-down, and if an
op-amp is unpowered.  Deliberately not attempted: forcing the gates negative while
the op-amp *is* driving, which would mean moving the + input off ground and
re-characterising all 16 bias channels -- a topology decision with firmware
consequences, recorded rather than guessed.

B1.5 -- the same move feeds it: the four OPA4703 V- pins leave -5V5_PA, whose
LM2662 is at 100 % of rating, for -5V0_ADAR12/34 at ~60 % (two op-amps per rail).
Channels pull down to the rail their own op-amp runs from, so the LM2662 is off
the gate-bias path entirely.

B2.3 -- PA drain bulk was ~20 uF against the ~100 uF the 30 us / 1.68 A pulse
wants; eight more 10 uF 1206 ceramics (C10-C17) on VIN_M use the device this board
already carries, so no new footprint.

Verified: all four files parse (main 2009 parts / 822 elements, PA 51 / 33); no
OPA V- pin or pad remains on -5V5_PA and each ADAR rail carries two op-amps and
eight pull-downs; every VGn net gained exactly one new pull-down (its existing
feedback resistor is the other R on the net); the eight new caps are on VIN_M and
GND; no duplicate designators; gates green.  Both BOMs keep the repo's grouping --
the 10k/R0201 and 10uF/C1206 rows were extended rather than duplicated.

Un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
Parts:
- added R178, R179, R180, R181, R182, R183, R184, R185, R186, R187, R188, R189, R190, R191, R192, R193: 10k, rcl:R0201
Connections:
- net -5V0_ADAR12: now also OPA_1.11, OPA_2.11, R178.2, R179.2, R180.2, R181.2, R182.2, R183.2, R184.2, R185.2
- net -5V0_ADAR34: now also OPA_3.11, OPA_4.11, R186.2, R187.2, R188.2, R189.2, R190.2, R191.2, R192.2, R193.2
- net -5V5_PA: no longer OPA_1.11, OPA_2.11, OPA_3.11, OPA_4.11
- net VG_1: now also R178.1
- net VG_10: now also R186.1
- net VG_11: now also R183.1
- net VG_12: now also R187.1
- net VG_13: now also R184.1
- net VG_14: now also R188.1
- net VG_15: now also R185.1
- net VG_16: now also R189.1
- net VG_2: now also R190.1
- net VG_3: now also R179.1
- net VG_4: now also R191.1
- net VG_5: now also R180.1
- net VG_6: now also R192.1
- net VG_7: now also R181.1
- net VG_8: now also R193.1
- net VG_9: now also R182.1

Commit message: fix(hw): revert B1.5, connect the PG pins, and generate the harness map
Five fixes from the remaining-items plan. Two of them are corrections to work already
committed, and one is a correction to the plan itself.

REVERT B1.5.  Its premise was wrong.  The rail budget has -5V5_PA at 100 mA against a 200 mA
LM2662 -- 50 %, not "100 % of rating" as the item claimed -- while -5V0_ADAR12/34 are the
rails that are 1.2x over (240 mA vs 200 mA).  What was moved is negligible anyway: the
OPA4703 datasheet gives 200 uA per amplifier, so ~3 mA of quads plus ~1.6 mA of the new gate
pull-downs.  So the change added load to the two overloaded rails and left U22, C105 and one
harness connector feeding nothing.  All four OPA V- pins and all sixteen gate pull-downs are
back on -5V5_PA, which also puts each pull-down on the same negative rail as the op-amp it
backs up -- the better arrangement.  The real item is B3.1 (the ADAR negative rails).

B1.4/B3.2 PRECONDITION.  U32/U34/U35 each had a PG pin connected to nothing.  TPS7A8300 PG
is active-high open-drain asserting at 89 % of target, so it needs a pull-up to be a defined
level at all.  Nets PG_3V3_ADTR / PG_3V3_XO / PG_2V5_FPGA now carry the pin, and R61-R63
(10 kohm to +3V3) pull them up -- the signal names the connector decision will route.  10 kohm
rather than the datasheet's 100 kohm test condition, because the 10k/M0805 row and its
verified MPN (AE0805BR-0710KL) already exist and 330 uA vs 33 uA when asserted is immaterial
for a fault line.  This is needed by every routing option, so it is not gated on that
decision.

Correction to the plan, found while implementing: a single open-drain PG wire CANNOT be
fail-safe.  "Rail good" (high-Z) and "harness disconnected" are electrically identical no
matter which side carries the pull-up.  The plan claimed otherwise; the honest statement is
that the line is fail-silent on an open harness, and the mitigations are a firmware line-test
(drive low, release, read back) or accepting it.

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
Connections:
- net -5V0_ADAR12: no longer OPA_1.11, OPA_2.11, R178.2, R179.2, R180.2, R181.2, R182.2, R183.2, R184.2, R185.2
- net -5V0_ADAR34: no longer OPA_3.11, OPA_4.11, R186.2, R187.2, R188.2, R189.2, R190.2, R191.2, R192.2, R193.2
- net -5V5_PA: now also OPA_1.11, OPA_2.11, OPA_3.11, OPA_4.11, R178.2, R179.2, R180.2, R181.2, R182.2, R183.2, R184.2, R185.2, R186.2, R187.2, R188.2, R189.2, R190.2, R191.2, R192.2, R193.2
Changed lines of the file:
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@@
 <wire x1="224.023103125" y1="238.949965625" x2="224.15309375" y2="239.07995625" width="0.3" layer="16"/>
 <wire x1="224.15309375" y1="239.07995625" x2="224.15309375" y2="239.44690625" width="0.3" layer="16"/>
-<contactref element="OPA_2" pad="11"/><contactref element="OPA_1" pad="11"/><contactref element="R178" pad="2"/><contactref element="R179" pad="2"/><contactref element="R180" pad="2"/><contactref element="R181" pad="2"/><contactref element="R182" pad="2"/><contactref element="R183" pad="2"/><contactref element="R184" pad="2"/><contactref element="R185" pad="2"/></signal>
+</signal>
 <signal name="+5V0_PA_1">
 <contactref element="X14" pad="1"/>
@@
 <wire x1="152.0012" y1="138.96051875" x2="152.0012" y2="143.9988" width="0.3" layer="16"/>
 <wire x1="152.0012" y1="143.9988" x2="152" y2="144" width="0.3" layer="16"/>
-<contactref element="OPA_3" pad="11"/><contactref element="OPA_4" pad="11"/><contactref element="R186" pad="2"/><contactref element="R187" pad="2"/><contactref element="R188" pad="2"/><contactref element="R189" pad="2"/><contactref element="R190" pad="2"/><contactref element="R191" pad="2"/><contactref element="R192" pad="2"/><contactref element="R193" pad="2"/></signal>
+</signal>
 <signal name="+3V3_ADAR12">
 <contactref element="X20" pad="1"/>
@@
 <wire x1="62.9" y1="26.35" x2="62.9" y2="25.0194" width="0.15" layer="1"/>
 <wire x1="33" y1="26" x2="33" y2="24.8194" width="0.25" layer="1"/>
-</signal>
+<contactref element="OPA_1" pad="11"/><contactref element="OPA_2" pad="11"/><contactref element="OPA_3" pad="11"/><contactref element="OPA_4" pad="11"/><contactref element="R178" pad="2"/><contactref element="R179" pad="2"/><contactref element="R180" pad="2"/><contactref element="R181" pad="2"/><contactref element="R182" pad="2"/><contactref element="R183" pad="2"/><contactref element="R184" pad="2"/><contactref element="R185" pad="2"/><contactref element="R186" pad="2"/><contactref element="R187" pad="2"/><contactref element="R188" pad="2"/><contactref element="R189" pad="2"/><contactref element="R190" pad="2"/><contactref element="R191" pad="2"/><contactref element="R192" pad="2"/><contactref element="R193" pad="2"/></signal>
 <signal name="+5V0_0">
 <contactref element="X18" pad="1"/>

Commit message: feat(backlog): close the six remaining Lane B decisions (#5 #7 #8 #9 #10 #24)
#5 PA operating mode: PA_BIAS_SEQUENCE.{h,c} make the gate/drain order a tested
   contract (enable: gate off -> drain -> settle -> operating bias; disable: gate
   off -> drain off; every failure path lands safe). 17/17, wired into startup and
   Emergency_Stop in main.cpp.
#7 harmonic filter: docs/harmonic-filter.md - spec, the existing SMA interface, the
   measurement that must set the filter order, and the three options.
#8 rail-good routing: three TPS7A8300 PG signals each get their own 2-position
   connector pair (power X38-X40 -> main X25-X27 -> U2.PC0-PC2, verified free).
   RAIL_FAULT.{h,c} samples and latches them, 19/19, wired into the main loop and
   telemetry. The pins are read with pull-downs, so an open harness reads LOW and is
   reported as a fault - the earlier "fail-silent" note was wrong and is corrected.
#9 negative rails: U36/U37 parallel U20/U21 on -5V0_ADAR12/34, each with its own
   47 uF pumping cap and the shared output cap, exactly as TI's datasheet requires.
   Two in parallel halve the output resistance and double the headroom (240 mA of a
   400 mA capability instead of 1.2x over a 200 mA part).
#10 keying: negative rails move to the 3-position part and the PA drain feeds to a
   4-position part with two pins per rail (which also halves the 4 A per pin). The
   4-position part is authored from the repo's own 22-23-2031 geometry. One rail was
   spelled two ways across boards (+3V3_ADAR_12 vs +3V3_ADAR12) and is now unified.
   The harness map's keying column is generated from the parts, not typed.
#24 laminate: the PA board moves to RO4350B (recorded in FAB_NOTES.md); the patch
   array is gerbers-only and flagged as un-respinnable.

Verification: netlist_integrity caught two real regressions during this work (gate
names the part did not instantiate; designators dropped from the authored BOM) and
both are fixed. All six artifact gates and ruff are green.
Parts:
- added X25, X26, X27: 22-23-2021, con-molex:22-23-2021
- X11, X13, X15, X19, X22, X6: device con-molex:22-23-2021 -> con-molex:22-23-2031
- X14, X5, X7: device con-molex:22-23-2021 -> con-molex:22-23-2041
Connections:
- new net PG_2V5_FPGA: X27.1
- new net PG_3V3_ADTR: X25.1
- new net PG_3V3_XO: X26.1
- net GND: now also X11.3, X13.3, X14.3, X14.4, X15.3, X19.3, X22.3, X25.2, X26.2, X27.2, X5.3, X5.4, X6.3, X7.3, X7.4
