File: 4_Schematics and Boards Layout/4_6_Schematics/MainBoard/RADAR_Main_Board.brd (EAGLE design)
At the start: 260 x 300 mm, 825 parts, among them IC1 AT93C46A-10SQ-2.7, J1 142-0731-211, J18 142-0731-211, J19 CJT-T-P-HH-ST-TH1, J20 142-0731-211, J21 CJT-T-P-HH-ST-TH1, J22 142-0731-211, J23 142-0731-211, J24 142-0731-211, J25 142-0731-211, J26 142-0731-211, J27 142-0731-211, J28 142-0731-211, J29 142-0731-211, J30 142-0731-211, J31 142-0731-211, J32 142-0731-211, J33 142-0731-211, J34 142-0731-211, J35 142-0731-211, J36 142-0731-211, J37 142-0731-211, J38 142-0731-211, J39 142-0731-211, J40 142-0731-211, J41 142-0731-211, J42 142-0731-211, J43 142-0731-211, J44 142-0731-211, J45 142-0731-211, J46 142-0731-211, J47 142-0731-211, J48 142-0731-211, J49 142-0731-211, J50 142-0731-211, J51 142-0731-211, J52 142-0731-211, J53 142-0731-211, J54 142-0731-211, J55 142-0731-211, J56 142-0731-211, J57 142-0731-211, J58 142-0731-211, J59 142-0731-211, U1 AD9484BCPZ-500, U10 ADS7830IPWR, U11 INA241A4IDGKRDGK0008A-MFG, U13 LTC5552IUDBTRMPBF, U14 SZMMSZ5232BT1G, U15 SZMMSZ5232BT1G, U16 EP4RKU+, U17 SZMMSZ5232BT1G, U2 STM32F746ZGT7, U3 AD9708AR, U37 SZMMSZ5232BT1G, U38 SZMMSZ5232BT1G, U39 SZMMSZ5232BT1G, U4 AD8352ACPZ-R7, U40 SZMMSZ5232BT1G, U41 SZMMSZ5232BT1G, U42 XC7A50T-2FTG256I, U43 SZMMSZ5232BT1G, U44 SZMMSZ5232BT1G, U45 SZMMSZ5232BT1G, U46 SZMMSZ5232BT1G, U47 SZMMSZ5232BT1G, U48 SZMMSZ5232BT1G, U49 SZMMSZ5232BT1G, U5 LTC5552IUDBTRMPBF, U50 SZMMSZ5232BT1G, U51 SZMMSZ5232BT1G, U52 SZMMSZ5232BT1G, U53 SZMMSZ5232BT1G, U54 SZMMSZ5232BT1G, U55 SZMMSZ5232BT1G, U56 SZMMSZ5232BT1G, U57 SZMMSZ5232BT1G, U58 SZMMSZ5232BT1G, U59 SZMMSZ5232BT1G, U6 FT2232HQ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

Commit message: fix(tools): the BOM gate now checks which row a part sits on, not just that it exists
regenerate_bom.py compared designator *presence* between the board and the sheet, so a
designator could sit on the wrong row and pass. That is exactly how the harness keying change
went wrong earlier: the new rows were cloned and inherited the whole 2-position list, and the
gate stayed green.

It now compares the board's value against the value on the sheet row the designator appears in,
normalising the micro glyph and accepting a containment match so that "100nF" vs "100nF/50V"
is not a finding. Verified by fault injection: moving X31 onto the 22-23-2021 row makes the
check name it, and restoring makes it clean again.

It found two real defects, both fixed here:

- X19 on the main board still carried value 22-23-2021 after its part became 22-23-2031 (the
  earlier element-value fix omitted it), so the board disagreed with its own package.
- C17, C55, C176 and C285 read 47uF on the board while the ordered part is CM03X5R475M06AH055.
  The three-digit code 475 is 47 x 10^5 pF = 4.7 uF and no 0201 case holds 47 uF, so the board
  value was the typo and the sheet's 4.7uF was right. Corrected in both the schematic and the
  board element.

Also closes the loop on the four issues verified this round: #4 (shunt MPN corrected, INA241A4
sense amps in the BOM), #11 (six gates in CI), #18 (laminate recorded), #25 (no board-only
elements).
Parts:
- C17, C176, C285, C55: value 47uF -> 4.7uF
- X11, X13, X15, X19, X22, X6: value 22-23-2021 -> 22-23-2031
- X14, X5, X7: value 22-23-2021 -> 22-23-2041
Changed lines of the file:
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@@
 <attribute name="VALUE" x="166.508715625" y="160.409765625" size="1.27" layer="27" rot="R135"/>
 </element>
-<element name="C17" library="eagle-ltspice" package="C0201" value="47uF" x="59.1121125" y="192.78626875" smashed="yes" rot="R135">
+<element name="C17" library="eagle-ltspice" package="C0201" value="4.7uF" x="59.1121125" y="192.78626875" smashed="yes" rot="R135">
 <attribute name="NAME" x="59.1121125" y="191.88824375" size="1.27" layer="25" rot="R135"/>
 <attribute name="SPICEMODEL" value="NONE" x="82.460778125" y="625.634615625" size="1.778" layer="27" rot="R135" display="off"/>
@@
 <attribute name="VALUE" x="136.396175" y="127.153896875" size="1.27" layer="27" rot="R135"/>
 </element>
-<element name="C176" library="eagle-ltspice" package="C0201" value="47uF" x="62.645" y="174.87" smashed="yes">
+<element name="C176" library="eagle-ltspice" package="C0201" value="4.7uF" x="62.645" y="174.87" smashed="yes">
 <attribute name="NAME" x="62.01" y="175.505" size="1.27" layer="25"/>
 <attribute name="SPICEMODEL" value="NONE" x="175.675" y="-137.55" size="1.778" layer="27" display="off"/>
@@
 <attribute name="VALUE" x="59.385" y="134.98" size="1.27" layer="27" rot="R180"/>
 </element>
-<element name="C55" library="eagle-ltspice" package="C0201" value="47uF" x="39.629215625" y="193.434096875" smashed="yes" rot="R225">
+<element name="C55" library="eagle-ltspice" package="C0201" value="4.7uF" x="39.629215625" y="193.434096875" smashed="yes" rot="R225">
 <attribute name="NAME" x="40.527240625" y="193.434096875" size="1.27" layer="25" rot="R225"/>
 <attribute name="SPICEMODEL" value="NONE" x="-407.5875375" y="202.414353125" size="1.778" layer="27" rot="R225" display="off"/>
@@
 <attribute name="VALUE" x="-0.5" y="167.7" size="1.016" layer="27" ratio="10" rot="R270"/>
 </element>
-<element name="X11" library="con-molex" package="22-23-2031" value="22-23-2021" x="246.88" y="107.47" smashed="yes" rot="R90">
+<element name="X11" library="con-molex" package="22-23-2031" value="22-23-2031" x="246.88" y="107.47" smashed="yes" rot="R90">
 <attribute name="MF" value="MOLEX" x="470.4" y="144.3" size="1.778" layer="27" rot="R90" display="off"/>
 <attribute name="MPN" value="22-23-2021" x="470.4" y="144.3" size="1.778" layer="27" rot="R90" display="off"/>
@@
 <attribute name="VALUE" x="251.56" y="75.24" size="1.016" layer="27" ratio="10" rot="R90"/>
 </element>
-<element name="X13" library="con-molex" package="22-23-2031" value="22-23-2021" x="202.06" y="277.23" smashed="yes" rot="R180">
+<element name="X13" library="con-molex" package="22-23-2031" value="22-23-2031" x="202.06" y="277.23" smashed="yes" rot="R180">
 <attribute name="MF" value="MOLEX" x="147.45" y="500.75" size="1.778" layer="27" rot="R180" display="off"/>
 <attribute name="MPN" value="22-23-2021" x="147.45" y="500.75" size="1.778" layer="27" rot="R180" display="off"/>
@@
 <attribute name="VALUE" x="204.6" y="282.31" size="1.016" layer="27" ratio="10" rot="R180"/>
 </element>
-<element name="X14" library="con-molex" package="22-23-2041" value="22-23-2021" x="118.5" y="278.78" smashed="yes" rot="R180">
+<element name="X14" library="con-molex" package="22-23-2041" value="22-23-2041" x="118.5" y="278.78" smashed="yes" rot="R180">
 <attribute name="MF" value="MOLEX" x="55" y="502.3" size="1.778" layer="27" rot="R180" display="off"/>
 <attribute name="MPN" value="22-23-2021" x="55" y="502.3" size="1.778" layer="27" rot="R180" display="off"/>
@@
 <attribute name="VALUE" x="121.04" y="283.86" size="1.016" layer="27" ratio="10" rot="R180"/>
 </element>
-<element name="X15" library="con-molex" package="22-23-2031" value="22-23-2021" x="186.61" y="90.97" smashed="yes">
+<element name="X15" library="con-molex" package="22-23-2031" value="22-23-2031" x="186.61" y="90.97" smashed="yes">
 <attribute name="MF" value="MOLEX" x="259" y="-132.55" size="1.778" layer="27" display="off"/>
 <attribute name="MPN" value="22-23-2021" x="259" y="-132.55" size="1.778" layer="27" display="off"/>
@@
 <attribute name="VALUE" x="0.44" y="144.1" size="1.016" layer="27" ratio="10" rot="R270"/>
 </element>
-<element name="X19" library="con-molex" package="22-23-2031" value="22-23-2021" x="4.97" y="47.25" smashed="yes" rot="R270">
+<element name="X19" library="con-molex" package="22-23-2031" value="22-23-2031" x="4.97" y="47.25" smashed="yes" rot="R270">
 <attribute name="MF" value="MOLEX" x="-218.55" y="-60.7" size="1.778" layer="27" rot="R270" display="off"/>
 <attribute name="MPN" value="22-23-2021" x="-218.55" y="-60.7" size="1.778" layer="27" rot="R270" display="off"/>
@@
 <attribute name="VALUE" x="138.852584375" y="25.10651875" size="1.016" layer="27" ratio="10" rot="R180"/>
 </element>
-<element name="X5" library="con-molex" package="22-23-2041" value="22-23-2021" x="242.67" y="278.03" smashed="yes" rot="R180">
+<element name="X5" library="con-molex" package="22-23-2041" value="22-23-2041" x="242.67" y="278.03" smashed="yes" rot="R180">
 <attribute name="MF" value="MOLEX" x="-38" y="482.5" size="1.778" layer="27" rot="R180" display="off"/>
 <attribute name="MPN" value="22-23-2021" x="-38" y="482.5" size="1.778" layer="27" rot="R180" display="off"/>
@@
 <attribute name="VALUE" x="-0.13" y="19.66" size="1.016" layer="27" ratio="10" rot="R270"/>
 </element>
-<element name="X6" library="con-molex" package="22-23-2031" value="22-23-2021" x="246.53" y="43.94" smashed="yes" rot="R90">
+<element name="X6" library="con-molex" package="22-23-2031" value="22-23-2031" x="246.53" y="43.94" smashed="yes" rot="R90">
 <attribute name="MF" value="MOLEX" x="451" y="333.5" size="1.778" layer="27" rot="R90" display="off"/>
 <attribute name="MPN" value="22-23-2021" x="451" y="333.5" size="1.778" layer="27" rot="R90" display="off"/>
@@
 <attribute name="VALUE" x="251.61" y="41.4" size="1.016" layer="27" ratio="10" rot="R90"/>
 </element>
-<element name="X7" library="con-molex" package="22-23-2041" value="22-23-2021" x="123.05" y="91.97" smashed="yes">
+<element name="X7" library="con-molex" package="22-23-2041" value="22-23-2041" x="123.05" y="91.97" smashed="yes">
 <attribute name="MF" value="MOLEX" x="421.5" y="-112.5" size="1.778" layer="27" display="off"/>
 <attribute name="MPN" value="22-23-2021" x="421.5" y="-112.5" size="1.778" layer="27" display="off"/>
@@
 <attribute name="VALUE" x="193.44" y="281.68" size="1.016" layer="27" ratio="10" rot="R180"/>
 </element>
-<element name="X22" library="con-molex" package="22-23-2031" value="22-23-2021" x="180.4" y="276.6" smashed="yes" rot="R180">
+<element name="X22" library="con-molex" package="22-23-2031" value="22-23-2031" x="180.4" y="276.6" smashed="yes" rot="R180">
 <attribute name="MF" value="MOLEX" x="180.4" y="276.6" size="1.778" layer="27" rot="R180" display="off"/>
 <attribute name="MPN" value="22-23-2021" x="180.4" y="276.6" size="1.778" layer="27" rot="R180" display="off"/>
@@
 <attribute name="VALUE" x="81.675" y="188.96" size="1.27" layer="27" rot="R90"/>
 </element>
-<element name="C285" library="eagle-ltspice" package="C0201" value="47uF" x="38.1" y="177.475" smashed="yes">
+<element name="C285" library="eagle-ltspice" package="C0201" value="4.7uF" x="38.1" y="177.475" smashed="yes">
 <attribute name="NAME" x="37.465" y="178.11" size="1.27" layer="25"/>
 <attribute name="SPICEMODEL" value="NONE" x="38.1" y="192.175" size="1.778" layer="27" display="off"/>

Commit message: feat(hw): ADAR supply order, test points, strobe acknowledgement (#13 #15 #20)
#20 ADAR1000 supply order - the requirement, verified and locked
  The pin table says AVDD3 (+3.3 V) must come up "before or at the same time as the
  AVDD1(-5V) supply"; the "−5 V first" sentence elsewhere in the same datasheet is about an
  external PA's drain (the gate-bias rule).  The firmware already asserts the 3.3 V ADAR rails
  before the 5.0 V rail that creates -5 V through the LM2662 inverters, so this needed no code
  change - it needed the requirement written down at the call site and a test that fails if a
  later edit swaps the order.  docs/power-up-order.md records every device's requirement with
  its citation (ADAR1000 pin table, ADTR1107 Recommended Bias Sequencing, M3SWA2 dual supply,
  LTC5552/AD8352 single supply) and the structural fact that every negative rail here is
  inverted from a positive one, so "negative first" is not physically available.

#15 test points - 15 added where there were zero
  The Harwin S1751-46R (1.63 x 3.25 mm SMT test point, two pads on one node) authored from its
  own land pattern, placed on the power board at the bring-up rails and the three rail-good
  signals, with a BOM row.  docs/probe-map.md already said which pin to meter; this gives the
  probe somewhere to land.

#13 strobe acknowledgement - the MCU can now tell whether the FPGA acted
  strobe_ack.v turns the top's accepted-frame pulse into a level the MCU can poll: a request
  clears it, consumption sets it, so "still low at the next request" means the strobe was
  dropped.  Wired from the already-synchronized pulse, exposed through the 50T wrapper,
  constrained to B16 (bank 15, LVCMOS33 - the same bank as the strobes it answers, so no level
  shift), and carried in the netlist from U42 to U2.PC3.  The FPGA's config net (DONE with
  INIT_B and their pull-ups) now reaches U2.PC4 as FPGA_CFG_OK.  MCU side: STROBE_ACK.{h,c}
  scores each request before the next one is issued - the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
Connections:
- removed net N$115: R144.1, U42.H10
- new net FPGA_DONE: R144.1, U2.44, U42.H10
- new net FPGA_STROBE_ACK: U2.29, U42.B16
- net PG_2V5_FPGA: now also U2.28
- net PG_3V3_ADTR: now also U2.26
- net PG_3V3_XO: now also U2.27
Routing:
- net N$115: track 10.6 -> 0.00 mm, vias 1 -> 0
- net FPGA_DONE: track 0.00 -> 10.6 mm, vias 0 -> 1
Changed lines of the file:
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@@
 </element>
 </elements>
-<signals><signal name="PG_2V5_FPGA" class="0"><contactref element="X27" pad="1"/></signal><signal name="PG_3V3_XO" class="0"><contactref element="X26" pad="1"/></signal><signal name="PG_3V3_ADTR" class="0"><contactref element="X25" pad="1"/></signal><signal name="N$U91_OE" class="0"><contactref element="U91" pad="6"/><contactref element="R177" pad="1"/></signal><signal name="N$U90_OE" class="0"><contactref element="U90" pad="8"/><contactref element="R176" pad="1"/></signal><signal name="+2V5_FPGA" class="0"><contactref element="U90" pad="1"/><contactref element="U91" pad="3"/><contactref element="R176" pad="2"/><contactref element="R177" pad="2"/><contactref element="C354" pad="1"/><contactref element="C355" pad="1"/><contactref element="C358" pad="1"/><contactref element="C359" pad="1"/><contactref element="X57" pad="1"/><contactref element="U42" pad="L16"/><contactref element="U42" pad="M13"/><contactref element="U42" pad="N10"/><contactref element="U42" pad="P7"/><contactref element="U42" pad="R14"/><contactref element="U42" pad="T11"/></signal><signal name="FLASH_NRST_F" class="0"><contactref element="U9" pad="A4"/><contactref element="U91" pad="1"/></signal><signal name="FLASH_NCS_F" class="0"><contactref element="U9" pad="C2"/><contactref element="U91" pad="8"/></signal><signal name="FLASH_DQ3_F" class="0"><contactref element="U9" pad="D4"/><contactref element="U90" pad="10"/></signal><signal name="FLASH_DQ2_F" class="0"><contactref element="U9" pad="C4"/><contactref element="U90" pad="11"/></signal><signal name="FLASH_DQ1_F" class="0"><contactref element="U9" pad="D2"/><contactref element="U90" pad="12"/></signal><signal name="FLASH_DQ0_F" class="0"><contactref element="U9" pad="D3"/><contactref element="U90" pad="13"/></signal>
+<signals><signal name="FPGA_STROBE_ACK" class="0"><contactref element="U42" pad="B16"/><contactref element="U2" pad="29"/></signal><signal name="PG_2V5_FPGA" class="0"><contactref element="X27" pad="1"/><contactref element="U2" pad="28"/></signal><signal name="PG_3V3_XO" class="0"><contactref element="X26" pad="1"/><contactref element="U2" pad="27"/></signal><signal name="PG_3V3_ADTR" class="0"><contactref element="X25" pad="1"/><contactref element="U2" pad="26"/></signal><signal name="N$U91_OE" class="0"><contactref element="U91" pad="6"/><contactref element="R177" pad="1"/></signal><signal name="N$U90_OE" class="0"><contactref element="U90" pad="8"/><contactref element="R176" pad="1"/></signal><signal name="+2V5_FPGA" class="0"><contactref element="U90" pad="1"/><contactref element="U91" pad="3"/><contactref element="R176" pad="2"/><contactref element="R177" pad="2"/><contactref element="C354" pad="1"/><contactref element="C355" pad="1"/><contactref element="C358" pad="1"/><contactref element="C359" pad="1"/><contactref element="X57" pad="1"/><contactref element="U42" pad="L16"/><contactref element="U42" pad="M13"/><contactref element="U42" pad="N10"/><contactref element="U42" pad="P7"/><contactref element="U42" pad="R14"/><contactref element="U42" pad="T11"/></signal><signal name="FLASH_NRST_F" class="0"><contactref element="U9" pad="A4"/><contactref element="U91" pad="1"/></signal><signal name="FLASH_NCS_F" class="0"><contactref element="U9" pad="C2"/><contactref element="U91" pad="8"/></signal><signal name="FLASH_DQ3_F" class="0"><contactref element="U9" pad="D4"/><contactref element="U90" pad="10"/></signal><signal name="FLASH_DQ2_F" class="0"><contactref element="U9" pad="C4"/><contactref element="U90" pad="11"/></signal><signal name="FLASH_DQ1_F" class="0"><contactref element="U9" pad="D2"/><contactref element="U90" pad="12"/></signal><signal name="FLASH_DQ0_F" class="0"><contactref element="U9" pad="D3"/><contactref element="U90" pad="13"/></signal>
 <signal name="+3V3">
 <contactref element="X24" pad="1"/>
@@
 <via x="43.55" y="187.3" extent="1-16" drill="0.15"/>
 </signal>
-<signal name="N$115">
+<signal name="FPGA_DONE">
 <contactref element="R144" pad="1"/>
 <contactref element="U42" pad="H10"/>
@@
 <wire x1="59.8" y1="184.1" x2="59.815" y2="184.08" width="0.1" layer="1"/>
 <wire x1="51.3" y1="183.8" x2="51.18" y2="183.78" width="0.1" layer="1"/>
-</signal>
+<contactref element="U2" pad="44"/></signal>
 <signal name="N$116">
 <contactref element="U42" pad="K10"/>
