File: 4_Schematics and Boards Layout/4_6_Schematics/MainBoard/RADAR_Main_Board.sch (EAGLE design)
At the start: 795 parts, among them IC1 AT93C46A-10SQ-2.7, J1 142-0731-211, J18 142-0731-211, J19 CJT-T-P-HH-ST-TH1, J20 142-0731-211, J21 CJT-T-P-HH-ST-TH1, J22 142-0731-211, J23 142-0731-211, J24 142-0731-211, J25 142-0731-211, J26 142-0731-211, J27 142-0731-211, J28 142-0731-211, J29 142-0731-211, J30 142-0731-211, J31 142-0731-211, J32 142-0731-211, J33 142-0731-211, J34 142-0731-211, J35 142-0731-211, J36 142-0731-211, J37 142-0731-211, J38 142-0731-211, J39 142-0731-211, J40 142-0731-211, J41 142-0731-211, J42 142-0731-211, J43 142-0731-211, J44 142-0731-211, J45 142-0731-211, J46 142-0731-211, J47 142-0731-211, J48 142-0731-211, J49 142-0731-211, J50 142-0731-211, J51 142-0731-211, J52 142-0731-211, J53 142-0731-211, J54 142-0731-211, J55 142-0731-211, J56 142-0731-211, J57 142-0731-211, J58 142-0731-211, J59 142-0731-211, U1 AD9484BCPZ-500, U10 ADS7830IPWR, U11 INA241A4IDGKRDGK0008A-MFG, U13 LTC5552IUDBTRMPBF, U14 SZMMSZ5232BT1G, U15 SZMMSZ5232BT1G, U16 EP4RKU+, U17 SZMMSZ5232BT1G, U2 STM32F746ZGT7, U3 AD9708AR, U37 SZMMSZ5232BT1G, U38 SZMMSZ5232BT1G, U39 SZMMSZ5232BT1G, U4 AD8352ACPZ-R7, U40 SZMMSZ5232BT1G, U41 SZMMSZ5232BT1G, U42 XC7A50T-2FTG256I, U43 SZMMSZ5232BT1G, U44 SZMMSZ5232BT1G, U45 SZMMSZ5232BT1G, U46 SZMMSZ5232BT1G, U47 SZMMSZ5232BT1G, U48 SZMMSZ5232BT1G, U49 SZMMSZ5232BT1G, U5 LTC5552IUDBTRMPBF, U50 SZMMSZ5232BT1G, U51 SZMMSZ5232BT1G, U52 SZMMSZ5232BT1G, U53 SZMMSZ5232BT1G, U54 SZMMSZ5232BT1G, U55 SZMMSZ5232BT1G, U56 SZMMSZ5232BT1G, U57 SZMMSZ5232BT1G, U58 SZMMSZ5232BT1G, U59 SZMMSZ5232BT1G, U6 FT2232HQ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

Commit message: feat(hw): bank 14 to 2.5 V with level-shifted QSPI lines (Lane B B1.1, part 2 of 2)
The half that actually changes the bank.  `VCCO_14` moves to the 2.5 V rail part 1
put on the power board, and because the configuration flash shares that net and is
a 3 V part, every line between the flash and the FPGA is split:

    FPGA_FLASH_DQ0   U42 + U90.A1   ->  FLASH_DQ0_F   U9.DQ0 + U90.B1
    FPGA_FLASH_DQ1   U42 + U90.A2   ->  FLASH_DQ1_F   U9.DQ1 + U90.B2
    FPGA_FLASH_DQ2   U42 + U90.A3   ->  FLASH_DQ2_F   U9.W/DQ2 + U90.B3
    FPGA_FLASH_DQ3   U42 + U90.A4   ->  FLASH_DQ3_F   U9.DQ3/HOLD + U90.B4
    FPGA_FLASH_NCS   U42 + U91.A1   ->  FLASH_NCS_F   U9.S + U91.B1
    FPGA_FLASH_NRST  U42 + U91.A2   ->  FLASH_NRST_F  U9.RESET + U91.B2

`U9.VCC` stays on +3V3_FPGA -- that is the whole point of the split, and it is
asserted below because getting it wrong silently bricks configuration.  DQ0..DQ3
use the 4-bit auto-direction part (they change direction inside a transaction and
the config engine cannot drive a direction pin); FCS_B and D07 use the 2-bit part.
Also added: OE pull-ups to the 2.5 V side, decoupling on both translator supplies,
decoupling for the newly split bank, and the 2-pin Molex that receives the rail.

Verified from the written files: both parse (1993 parts / 806 elements); each
FPGA-side net carries the FPGA ball and the A-side pin while its `_F` twin carries
the flash pin and the B-side pin; all six `VCCO_14` ball pads (L16, M13, N10, P7,
R14, T11) are on +2V5_FPGA and none remains on +3V3_FPGA while `VCCO_0/15/35` stay
at 3.3 V; and `element="U9"` appears only on the 3.3 V rail.  All three artifact
gates green, and interboard_rails now shows +2V5_FPGA spanning both boards.

Two mistakes of mine that the verification caught, both on the board side and both
fixed before this commit: `VCCO_14` is six BGA balls, not one, so a single
"remove the first U42 contactref" also stripped `VCCO_0`'s pad and a guessed pad
number went onto the new rail.  The schemati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
Parts:
- added C354, C355, C356, C357, C358, C359: 0.1uF, rcl:C-EUC0201
- added R176, R177: 10k, rcl:R-EU_R0201
- added U90: TXS0104EPWRPW0014A-MFG, My_Library_RADAR:TXS0104EPWRPW0014A-MFG
- added U91: TXS0102DCURDCU0008A-MFG, My_Library_RADAR:TXS0102DCURDCU0008A-MFG
- added X57: 22-23-202122-23-2021, con-molex:22-23-202122-23-2021
Connections:
- new net +2V5_FPGA: C354.1, C355.1, C358.1, C359.1, R176.2, R177.2, U42G$2.VCCO_14, U90.VCCA, U91.VCCA, X57-1.S
- new net FLASH_DQ0_F: U9.DQ0, U90.B1
- new net FLASH_DQ1_F: U9.DQ1, U90.B2
- new net FLASH_DQ2_F: U9.W/DQ2, U90.B3
- new net FLASH_DQ3_F: U9.DQ3/HOLD, U90.B4
- new net FLASH_NCS_F: U9.S, U91.B1
- new net FLASH_NRST_F: U9.RESET, U91.B2
- new net N$U90_OE: R176.1, U90.OE
- new net N$U91_OE: R177.1, U91.OE
- net +3V3_FPGA: now also C356.1, C357.1, U90.VCCB, U91.VCCB; no longer U42G$2.VCCO_14
- net FPGA_FLASH_DQ0: now also U90.A1; no longer U9.DQ0
- net FPGA_FLASH_DQ1: now also U90.A2; no longer U9.DQ1
- net FPGA_FLASH_DQ2: now also U90.A3; no longer U9.W/DQ2
- net FPGA_FLASH_DQ3: now also U90.A4; no longer U9.DQ3/HOLD
- net FPGA_FLASH_NCS: now also U91.A1; no longer U9.S
- net FPGA_FLASH_NRST: now also U91.A2; no longer U9.RESET
- net GND: now also C354.2, C355.2, C356.2, C357.2, C358.2, C359.2, U90.GND, U91.GND, X57-2.S
Changed lines of the file:
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@@
 <part name="GND1113" library="supply1" deviceset="GND" device=""/>
 <part name="R151" library="eagle-ltspice" deviceset="R" device="R0201" value="10k"/>
-<part name="U89" library="My_Library_RADAR" deviceset="ADS7830IPWR" device=""/>
+<part name="U90" library="My_Library_RADAR" deviceset="TXS0104EPWR" device="PW0014A-MFG"/><part name="U91" library="My_Library_RADAR" deviceset="TXS0102DCUR" device="DCU0008A-MFG"/><part name="R176" library="rcl" deviceset="R-EU_" device="R0201" value="10k"/><part name="R177" library="rcl" deviceset="R-EU_" device="R0201" value="10k"/><part name="C354" library="rcl" deviceset="C-EU" device="C0201" value="0.1uF"/><part name="C355" library="rcl" deviceset="C-EU" device="C0201" value="0.1uF"/><part name="C356" library="rcl" deviceset="C-EU" device="C0201" value="0.1uF"/><part name="C357" library="rcl" deviceset="C-EU" device="C0201" value="0.1uF"/><part name="C358" library="rcl" deviceset="C-EU" device="C0201" value="0.1uF"/><part name="C359" library="rcl" deviceset="C-EU" device="C0201" value="0.1uF"/><part name="X57" library="con-molex" deviceset="22-23-2021" device="22-23-2021"/><part name="U89" library="My_Library_RADAR" deviceset="ADS7830IPWR" device=""/>
 <part name="GND1116" library="supply1" deviceset="GND" device=""/>
 <part name="GND1117" library="supply1" deviceset="GND" device=""/>
@@
 <busses>
 </busses>
-<nets>
+<nets><net name="N$U91_OE" class="0"><segment><pinref part="U91" gate="G$1" pin="OE"/><pinref part="R177" gate="G$1" pin="1"/></segment></net><net name="N$U90_OE" class="0"><segment><pinref part="U90" gate="G$1" pin="OE"/><pinref part="R176" gate="G$1" pin="1"/></segment></net><net name="+2V5_FPGA" class="0"><segment><pinref part="U90" gate="G$1" pin="VCCA"/><pinref part="U91" gate="G$1" pin="VCCA"/><pinref part="R176" gate="G$1" pin="2"/><pinref part="R177" gate="G$1" pin="2"/><pinref part="C354" gate="G$1" pin="1"/><pinref part="C355" gate="G$1" pin="1"/><pinref part="C358" gate="G$1" pin="1"/><pinref part="C359" gate="G$1" pin="1"/><pinref part="X57" gate="-1" pin="S"/><pinref part="U42" gate="G$2" pin="VCCO_14"/></segment></net><net name="FLASH_NRST_F" class="0"><segment><pinref part="U9" gate="G$1" pin="RESET"/><pinref part="U91" gate="G$1" pin="B2"/></segment></net><net name="FLASH_NCS_F" class="0"><segment><pinref part="U9" gate="G$1" pin="S"/><pinref part="U91" gate="G$1" pin="B1"/></segment></net><net name="FLASH_DQ3_F" class="0"><segment><pinref part="U9" gate="G$1" pin="DQ3/HOLD"/><pinref part="U90" gate="G$1" pin="B4"/></segment></net><net name="FLASH_DQ2_F" class="0"><segment><pinref part="U9" gate="G$1" pin="W/DQ2"/><pinref part="U90" gate="G$1" pin="B3"/></segment></net><net name="FLASH_DQ1_F" class="0"><segment><pinref part="U9" gate="G$1" pin="DQ1"/><pinref part="U90" gate="G$1" pin="B2"/></segment></net><net name="FLASH_DQ0_F" class="0"><segment><pinref part="U9" gate="G$1" pin="DQ0"/><pinref part="U90" gate="G$1" pin="B1"/></segment></net>
 <net name="+3V3" class="0">
 <segment>
@@
 <pinref part="X22" gate="-2" pin="S"/>
 <pinref part="GND1079" gate="1" pin="GND"/>
-</segment>
+<pinref part="U90" gate="G$1" pin="GND"/><pinref part="U91" gate="G$1" pin="GND"/><pinref part="C354" gate="G$1" pin="2"/><pinref part="C355" gate="G$1" pin="2"/><pinref part="C356" gate="G$1" pin="2"/><pinref part="C357" gate="G$1" pin="2"/><pinref part="C358" gate="G$1" pin="2"/><pinref part="C359" gate="G$1" pin="2"/><pinref part="X57" gate="-2" pin="S"/></segment>
 </net>
 <net name="+1V8_FPGA" class="0">
@@
 <wire x1="162.56" y1="248.92" x2="160.02" y2="248.92" width="0.1524" layer="91"/>
 <label x="147.32" y="248.92" size="1.778" layer="95"/>
-</segment>
+<pinref part="U90" gate="G$1" pin="VCCB"/><pinref part="U91" gate="G$1" pin="VCCB"/><pinref part="C356" gate="G$1" pin="1"/><pinref part="C357" gate="G$1" pin="1"/></segment>
 </net>
 <net name="-5V5_PA" class="0">
@@
 <net name="FPGA_FLASH_NRST" class="0">
 <segment>
-<pinref part="U9" gate="A" pin="RESET"/>
 <pinref part="R50" gate="G$1" pin="1"/>
 <wire x1="556.26" y1="53.34" x2="548.64" y2="53.34" width="0.1524" layer="91"/>
@@
 <pinref part="U42" gate="G$2" pin="IO_L5N_T0_D07_14"/>
 <junction x="152.4" y="111.76"/>
-</segment>
+<pinref part="U91" gate="G$1" pin="A2"/></segment>
 </net>
 <net name="N$25" class="2">
@@
 <net name="FPGA_FLASH_NCS" class="0">
 <segment>
-<pinref part="U9" gate="A" pin="S"/>
 <pinref part="R52" gate="G$1" pin="1"/>
 <wire x1="556.26" y1="33.02" x2="548.64" y2="33.02" width="0.1524" layer="91"/>
@@
 <pinref part="U42" gate="G$2" pin="IO_L6P_T0_FCS_B_14"/>
 <junction x="152.4" y="109.22"/>
-</segment>
+<pinref part="U91" gate="G$1" pin="A1"/></segment>
 </net>
 <net name="FPGA_FLASH_DQ2" class="0">
 <segment>
-<pinref part="U9" gate="A" pin="W/DQ2"/>
 <pinref part="R53" gate="G$1" pin="1"/>
 <wire x1="607.06" y1="30.48" x2="614.68" y2="30.48" width="0.1524" layer="91"/>
@@
 <pinref part="U42" gate="G$2" pin="IO_L2P_T0_D02_14"/>
 <junction x="152.4" y="129.54"/>
-</segment>
+<pinref part="U90" gate="G$1" pin="A3"/></segment>
 </net>
 <net name="FPGA_FLASH_DQ1" class="0">
 <segment>
-<pinref part="U9" gate="A" pin="DQ1"/>
 <wire x1="607.06" y1="38.1" x2="612.14" y2="38.1" width="0.1524" layer="91"/>
 <label x="612.14" y="38.1" size="1.778" layer="95"/>
@@
 <pinref part="U42" gate="G$2" pin="IO_L1N_T0_D01_DIN_14"/>
 <junction x="152.4" y="132.08"/>
-</segment>
+<pinref part="U90" gate="G$1" pin="A2"/></segment>
 </net>
 <net name="FPGA_FLASH_DQ0" class="0">
 <segment>
-<pinref part="U9" gate="A" pin="DQ0"/>
 <wire x1="607.06" y1="40.64" x2="612.14" y2="40.64" width="0.1524" layer="91"/>
 <label x="612.14" y="40.64" size="1.778" layer="95"/>
@@
 <pinref part="U42" gate="G$2" pin="IO_L1P_T0_D00_MOSI_14"/>
 <junction x="152.4" y="134.62"/>
-</segment>
+<pinref part="U90" gate="G$1" pin="A1"/></segment>
 </net>
 <net name="FPGA_FLASH_DQ3" class="0">
 <segment>
-<pinref part="U9" gate="A" pin="DQ3/HOLD"/>
 <pinref part="R54" gate="G$1" pin="2"/>
 <wire x1="607.06" y1="43.18" x2="614.68" y2="43.18" width="0.1524" layer="91"/>
@@
 <pinref part="U42" gate="G$2" pin="IO_L2N_T0_D03_14"/>
 <junction x="152.4" y="127"/>
-</segment>
+<pinref part="U90" gate="G$1" pin="A4"/></segment>
 </net>
 <net name="FPGA_PUDC_B" class="0">
@@
 </segment>
 <segment>
-<pinref part="U42" gate="G$2" pin="VCCO_14"/>
 <wire x1="238.76" y1="142.24" x2="238.76" y2="147.32" width="0.1524" layer="91"/>
 <label x="238.76" y="147.32" size="1.778" layer="95"/>
@@
 <attribute name="VALUE" x="839.47" y="301.498" size="1.778" layer="96"/>
 </instance>
-<instance part="U89" gate="A" x="185.42" y="388.62" smashed="yes">
+<instance part="U90" gate="G$1" x="57.68" y="191.28" smashed="yes"><attribute name="NAME" x="55.68" y="192.78" size="1.524" layer="95"/></instance><instance part="U91" gate="G$1" x="30.04" y="191.82" smashed="yes"><attribute name="NAME" x="28.04" y="193.32" size="1.524" layer="95"/></instance><instance part="R176" gate="G$1" x="64.0" y="204.0" smashed="yes"><attribute name="NAME" x="62.0" y="205.5" size="1.524" layer="95"/></instance><instance part="R177" gate="G$1" x="36.0" y="204.0" smashed="yes"><attribute name="NAME" x="34.0" y="205.5" size="1.524" layer="95"/></instance><instance part="C354" gate="G$1" x="52.0" y="178.0" smashed="yes"><attribute name="NAME" x="50.0" y="179.5" size="1.524" layer="95"/></instance><instance part="C355" gate="G$1" x="60.0" y="178.0" smashed="yes"><attribute name="NAME" x="58.0" y="179.5" size="1.524" layer="95"/></instance><instance part="C356" gate="G$1" x="52.0" y="206.0" smashed="yes"><attribute name="NAME" x="50.0" y="207.5" size="1.524" layer="95"/></instance><instance part="C357" gate="G$1" x="60.0" y="206.0" smashed="yes"><attribute name="NAME" x="58.0" y="207.5" size="1.524" layer="95"/></instance><instance part="C358" gate="G$1" x="44.0" y="178.0" smashed="yes"><attribute name="NAME" x="42.0" y="179.5" size="1.524" layer="95"/></instance><instance part="C359" gate="G$1" x="44.0" y="206.0" smashed="yes"><attribute name="NAME" x="42.0" y="207.5" size="1.524" layer="95"/></instance><instance part="X57" gate="G$1" x="14.02" y="236.0" smashed="yes"><attribute name="NAME" x="12.02" y="237.5" size="1.524" layer="95"/></instance><instance part="X57" gate="-2" x="14.02" y="233.46" smashed="yes"><attribute name="NAME" x="12.02" y="232.7" size="1.524" layer="95"/></instance><instance part="U89" gate="A" x="185.42" y="388.62" smashed="yes">
 <attribute name="NAME" x="218.7956" y="397.7386" size="2.0828" layer="95" ratio="6" rot="SR0"/>
 <attribute name="VALUE" x="218.1606" y="395.1986" size="2.0828" layer="96" ratio="6" rot="SR0"/>

Commit message: feat(hw): gate-bias fail-safe, negative-rail margin, PA drain bulk (Lane B B2.2/B1.5/B2.3)
B2.2 -- and this is the finding that matters.  Every one of the 16 gate-bias
channels is an inverting amplifier referenced to ground (Vout = -(Rf/Rin) x VDAC,
+ input on GND), so a DAC in reset puts **0 V on all 16 gates**.  QPA2962 is a
depletion-mode GaN HEMT, where 0 V means *fully on* -- with 22 V on the drains.
That is a power-up hazard, not a nuance.

The plan frames the fix as hardware default *plus* MCU sequence; the hardware half
is here.  One 10k pull-down per channel from VGn to the same negative rail that
supplies its op-amp (R178-R193), so the gates sit at the negative rail whenever
the op-amps are not actively driving: during power-up, power-down, and if an
op-amp is unpowered.  Deliberately not attempted: forcing the gates negative while
the op-amp *is* driving, which would mean moving the + input off ground and
re-characterising all 16 bias channels -- a topology decision with firmware
consequences, recorded rather than guessed.

B1.5 -- the same move feeds it: the four OPA4703 V- pins leave -5V5_PA, whose
LM2662 is at 100 % of rating, for -5V0_ADAR12/34 at ~60 % (two op-amps per rail).
Channels pull down to the rail their own op-amp runs from, so the LM2662 is off
the gate-bias path entirely.

B2.3 -- PA drain bulk was ~20 uF against the ~100 uF the 30 us / 1.68 A pulse
wants; eight more 10 uF 1206 ceramics (C10-C17) on VIN_M use the device this board
already carries, so no new footprint.

Verified: all four files parse (main 2009 parts / 822 elements, PA 51 / 33); no
OPA V- pin or pad remains on -5V5_PA and each ADAR rail carries two op-amps and
eight pull-downs; every VGn net gained exactly one new pull-down (its existing
feedback resistor is the other R on the net); the eight new caps are on VIN_M and
GND; no duplicate designators; gates green.  Both BOMs keep the repo's grouping --
the 10k/R0201 and 10uF/C1206 rows were extended rather than duplicated.

Un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
Parts:
- added R178, R179, R180, R181, R182, R183, R184, R185, R186, R187, R188, R189, R190, R191, R192, R193: 10k, rcl:R-EU_R0201
Connections:
- net -5V0_ADAR12: now also OPA_1.V-, OPA_2.V-, R178.2, R179.2, R180.2, R181.2, R182.2, R183.2, R184.2, R185.2
- net -5V0_ADAR34: now also OPA_3.V-, OPA_4.V-, R186.2, R187.2, R188.2, R189.2, R190.2, R191.2, R192.2, R193.2
- net -5V5_PA: no longer OPA_1.V-, OPA_2.V-, OPA_3.V-, OPA_4.V-
- net VG_1: now also R178.1
- net VG_10: now also R186.1
- net VG_11: now also R183.1
- net VG_12: now also R187.1
- net VG_13: now also R184.1
- net VG_14: now also R188.1
- net VG_15: now also R185.1
- net VG_16: now also R189.1
- net VG_2: now also R190.1
- net VG_3: now also R179.1
- net VG_4: now also R191.1
- net VG_5: now also R180.1
- net VG_6: now also R192.1
- net VG_7: now also R181.1
- net VG_8: now also R193.1
- net VG_9: now also R182.1

Commit message: fix(hw): stale sense-amp annotation, and +3V3_XO bulk (Lane B B3.5)
Two grounded fixes, both from the progress audit rather than from the tracker's word.

1. Stale annotation. The main-board sheet has read "6 X INA241A3" twice since before this
   work: once wrong in the part (B2.5 made every sense amplifier an INA241A4) and once
   wrong in the count (the netlist has 16 of them). They sit in two columns of 8
   (U11,U73-U79 at x=419.10 and U80-U87 at x=650.24), so each label annotates one column:
   now "8 X INA241A4" twice, and 2 x 8 = the 16 in the netlist. The neighbouring labels
   ("2 X DAC5578", "3 X ADS7830") already match the netlist, which is the check that made
   this one's staleness visible instead of assumed.

2. B3.5 -- +3V3_XO. Steady state is ~1.25 A (1.2 A OCXO) on a 3 A TPS7A8300: 42 %, fine.
   Added four 22 uF C0603 (C169-C172) on the rail, reusing the part the board already
   carries -- the same BOM row and MPN (KGM15CR51E226MT, qty 54 -> 58) rather than a new
   line. This cuts the rail's source impedance at the heater's step load.

   What it does NOT do, stated plainly: cover a cold-start inrush. A capacitor holds a rail
   for t = C*dV/dI, so the ~32 uF now fitted buys microseconds, not milliseconds. The
   OCXO's inrush current is in no vendor source reachable from here (the part has no
   findable datasheet), so the cold-start capture remains a bench step -- and if it exceeds
   the regulator's 3 A, the fixes are sequencing (U34.EN is tied to +5V0_5 today, so that
   costs an MCU pin) or a soft-start, not more bulk.

Verified: both files parse; all four caps are on +3V3_XO and GND in schematic *and* board;
BOM row is 58 unique refs with all four present; no duplicate designators introduced; three
artifact gates exit 0.

Recorded while checking, not fixed (no decidable answer in the files):
  * X36 appears twice as a board element on the power board -- two connectors, one refdes,
    pre-existing at HEAD. Real BOM/assembly ambiguity, unde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
Other:
- note added: "8 X INA241A4"
- note removed: "6 X INA241A3"
Changed lines of the file:
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@@
 <text x="124.46" y="139.7" size="1.778" layer="98">AD9484</text>
 <text x="266.7" y="81.28" size="1.778" layer="98">3 X ADS7830</text>
-<text x="289.56" y="60.96" size="1.778" layer="98">6 X INA241A3</text>
-<text x="289.56" y="40.64" size="1.778" layer="98">6 X INA241A3</text>
+<text x="289.56" y="60.96" size="1.778" layer="98">8 X INA241A4</text>
+<text x="289.56" y="40.64" size="1.778" layer="98">8 X INA241A4</text>
 </plain>
 <instances>

Commit message: fix(hw): revert B1.5, connect the PG pins, and generate the harness map
Five fixes from the remaining-items plan. Two of them are corrections to work already
committed, and one is a correction to the plan itself.

REVERT B1.5.  Its premise was wrong.  The rail budget has -5V5_PA at 100 mA against a 200 mA
LM2662 -- 50 %, not "100 % of rating" as the item claimed -- while -5V0_ADAR12/34 are the
rails that are 1.2x over (240 mA vs 200 mA).  What was moved is negligible anyway: the
OPA4703 datasheet gives 200 uA per amplifier, so ~3 mA of quads plus ~1.6 mA of the new gate
pull-downs.  So the change added load to the two overloaded rails and left U22, C105 and one
harness connector feeding nothing.  All four OPA V- pins and all sixteen gate pull-downs are
back on -5V5_PA, which also puts each pull-down on the same negative rail as the op-amp it
backs up -- the better arrangement.  The real item is B3.1 (the ADAR negative rails).

B1.4/B3.2 PRECONDITION.  U32/U34/U35 each had a PG pin connected to nothing.  TPS7A8300 PG
is active-high open-drain asserting at 89 % of target, so it needs a pull-up to be a defined
level at all.  Nets PG_3V3_ADTR / PG_3V3_XO / PG_2V5_FPGA now carry the pin, and R61-R63
(10 kohm to +3V3) pull them up -- the signal names the connector decision will route.  10 kohm
rather than the datasheet's 100 kohm test condition, because the 10k/M0805 row and its
verified MPN (AE0805BR-0710KL) already exist and 330 uA vs 33 uA when asserted is immaterial
for a fault line.  This is needed by every routing option, so it is not gated on that
decision.

Correction to the plan, found while implementing: a single open-drain PG wire CANNOT be
fail-safe.  "Rail good" (high-Z) and "harness disconnected" are electrically identical no
matter which side carries the pull-up.  The plan claimed otherwise; the honest statement is
that the line is fail-silent on an open harness, and the mitigations are a firmware line-test
(drive low, release, read back) or accepting it.

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
Connections:
- net -5V0_ADAR12: no longer OPA_1.V-, OPA_2.V-, R178.2, R179.2, R180.2, R181.2, R182.2, R183.2, R184.2, R185.2
- net -5V0_ADAR34: no longer OPA_3.V-, OPA_4.V-, R186.2, R187.2, R188.2, R189.2, R190.2, R191.2, R192.2, R193.2
- net -5V5_PA: now also OPA_1.V-, OPA_2.V-, OPA_3.V-, OPA_4.V-, R178.2, R179.2, R180.2, R181.2, R182.2, R183.2, R184.2, R185.2, R186.2, R187.2, R188.2, R189.2, R190.2, R191.2, R192.2, R193.2
Changed lines of the file:
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@@
 <wire x1="162.56" y1="193.04" x2="160.02" y2="193.04" width="0.1524" layer="91"/>
 <label x="144.78" y="193.04" size="1.778" layer="95"/>
-<pinref part="OPA_2" gate="A" pin="V-"/><pinref part="OPA_1" gate="A" pin="V-"/><pinref part="R178" gate="G$1" pin="2"/><pinref part="R179" gate="G$1" pin="2"/><pinref part="R180" gate="G$1" pin="2"/><pinref part="R181" gate="G$1" pin="2"/><pinref part="R182" gate="G$1" pin="2"/><pinref part="R183" gate="G$1" pin="2"/><pinref part="R184" gate="G$1" pin="2"/><pinref part="R185" gate="G$1" pin="2"/></segment>
+</segment>
 </net>
 <net name="+5V0_PA_1" class="0">
@@
 <wire x1="203.2" y1="193.04" x2="200.66" y2="193.04" width="0.1524" layer="91"/>
 <label x="185.42" y="193.04" size="1.778" layer="95"/>
-<pinref part="OPA_3" gate="A" pin="V-"/><pinref part="OPA_4" gate="A" pin="V-"/><pinref part="R186" gate="G$1" pin="2"/><pinref part="R187" gate="G$1" pin="2"/><pinref part="R188" gate="G$1" pin="2"/><pinref part="R189" gate="G$1" pin="2"/><pinref part="R190" gate="G$1" pin="2"/><pinref part="R191" gate="G$1" pin="2"/><pinref part="R192" gate="G$1" pin="2"/><pinref part="R193" gate="G$1" pin="2"/></segment>
+</segment>
 </net>
 <net name="+3V3_ADAR12" class="0">
@@
 <wire x1="203.2" y1="231.14" x2="200.66" y2="231.14" width="0.1524" layer="91"/>
 <label x="190.5" y="231.14" size="1.778" layer="95"/>
-</segment>
+<pinref part="OPA_1" gate="A" pin="V-"/><pinref part="OPA_2" gate="A" pin="V-"/><pinref part="OPA_3" gate="A" pin="V-"/><pinref part="OPA_4" gate="A" pin="V-"/><pinref part="R178" gate="G$1" pin="2"/><pinref part="R179" gate="G$1" pin="2"/><pinref part="R180" gate="G$1" pin="2"/><pinref part="R181" gate="G$1" pin="2"/><pinref part="R182" gate="G$1" pin="2"/><pinref part="R183" gate="G$1" pin="2"/><pinref part="R184" gate="G$1" pin="2"/><pinref part="R185" gate="G$1" pin="2"/><pinref part="R186" gate="G$1" pin="2"/><pinref part="R187" gate="G$1" pin="2"/><pinref part="R188" gate="G$1" pin="2"/><pinref part="R189" gate="G$1" pin="2"/><pinref part="R190" gate="G$1" pin="2"/><pinref part="R191" gate="G$1" pin="2"/><pinref part="R192" gate="G$1" pin="2"/><pinref part="R193" gate="G$1" pin="2"/></segment>
 </net>
 <net name="+5V0_0" class="0">
