File: 4_Schematics and Boards Layout/4_6_Schematics/MainBoard/RADAR_Main_Board.sch (EAGLE design)
At the start: 825 parts, among them IC1 AT93C46A-10SQ-2.7, J1 142-0731-211, J18 142-0731-211, J19 CJT-T-P-HH-ST-TH1, J20 142-0731-211, J21 CJT-T-P-HH-ST-TH1, J22 142-0731-211, J23 142-0731-211, J24 142-0731-211, J25 142-0731-211, J26 142-0731-211, J27 142-0731-211, J28 142-0731-211, J29 142-0731-211, J30 142-0731-211, J31 142-0731-211, J32 142-0731-211, J33 142-0731-211, J34 142-0731-211, J35 142-0731-211, J36 142-0731-211, J37 142-0731-211, J38 142-0731-211, J39 142-0731-211, J40 142-0731-211, J41 142-0731-211, J42 142-0731-211, J43 142-0731-211, J44 142-0731-211, J45 142-0731-211, J46 142-0731-211, J47 142-0731-211, J48 142-0731-211, J49 142-0731-211, J50 142-0731-211, J51 142-0731-211, J52 142-0731-211, J53 142-0731-211, J54 142-0731-211, J55 142-0731-211, J56 142-0731-211, J57 142-0731-211, J58 142-0731-211, J59 142-0731-211, U1 AD9484BCPZ-500, U10 ADS7830IPWR, U11 INA241A4IDGKRDGK0008A-MFG, U13 LTC5552IUDBTRMPBF, U14 SZMMSZ5232BT1G, U15 SZMMSZ5232BT1G, U16 EP4RKU+, U17 SZMMSZ5232BT1G, U2 STM32F746ZGT7, U3 AD9708AR, U37 SZMMSZ5232BT1G, U38 SZMMSZ5232BT1G, U39 SZMMSZ5232BT1G, U4 AD8352ACPZ-R7, U40 SZMMSZ5232BT1G, U41 SZMMSZ5232BT1G, U42 XC7A50T-2FTG256I, U43 SZMMSZ5232BT1G, U44 SZMMSZ5232BT1G, U45 SZMMSZ5232BT1G, U46 SZMMSZ5232BT1G, U47 SZMMSZ5232BT1G, U48 SZMMSZ5232BT1G, U49 SZMMSZ5232BT1G, U5 LTC5552IUDBTRMPBF, U50 SZMMSZ5232BT1G, U51 SZMMSZ5232BT1G, U52 SZMMSZ5232BT1G, U53 SZMMSZ5232BT1G, U54 SZMMSZ5232BT1G, U55 SZMMSZ5232BT1G, U56 SZMMSZ5232BT1G, U57 SZMMSZ5232BT1G, U58 SZMMSZ5232BT1G, U59 SZMMSZ5232BT1G, U6 FT2232HQ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

Commit message: fix(tools): the BOM gate now checks which row a part sits on, not just that it exists
regenerate_bom.py compared designator *presence* between the board and the sheet, so a
designator could sit on the wrong row and pass. That is exactly how the harness keying change
went wrong earlier: the new rows were cloned and inherited the whole 2-position list, and the
gate stayed green.

It now compares the board's value against the value on the sheet row the designator appears in,
normalising the micro glyph and accepting a containment match so that "100nF" vs "100nF/50V"
is not a finding. Verified by fault injection: moving X31 onto the 22-23-2021 row makes the
check name it, and restoring makes it clean again.

It found two real defects, both fixed here:

- X19 on the main board still carried value 22-23-2021 after its part became 22-23-2031 (the
  earlier element-value fix omitted it), so the board disagreed with its own package.
- C17, C55, C176 and C285 read 47uF on the board while the ordered part is CM03X5R475M06AH055.
  The three-digit code 475 is 47 x 10^5 pF = 4.7 uF and no 0201 case holds 47 uF, so the board
  value was the typo and the sheet's 4.7uF was right. Corrected in both the schematic and the
  board element.

Also closes the loop on the four issues verified this round: #4 (shunt MPN corrected, INA241A4
sense amps in the BOM), #11 (six gates in CI), #18 (laminate recorded), #25 (no board-only
elements).
Parts:
- C17, C176, C285, C55: value 47uF -> 4.7uF
Changed lines of the file:
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@@
 <part name="C50" library="eagle-ltspice" deviceset="C" device="C0201" value="100nF"/>
 <part name="GND62" library="supply1" deviceset="GND" device=""/>
-<part name="C17" library="eagle-ltspice" deviceset="C" device="C0201" value="47uF"/>
+<part name="C17" library="eagle-ltspice" deviceset="C" device="C0201" value="4.7uF"/>
 <part name="C108" library="eagle-ltspice" deviceset="C" device="C0201" value="4.7uF"/>
 <part name="C109" library="eagle-ltspice" deviceset="C" device="C0201" value="4.7uF"/>
@@
 <part name="C123" library="eagle-ltspice" deviceset="C" device="C0201" value="10nF"/>
 <part name="GND646" library="supply1" deviceset="GND" device=""/>
-<part name="C55" library="eagle-ltspice" deviceset="C" device="C0201" value="47uF"/>
+<part name="C55" library="eagle-ltspice" deviceset="C" device="C0201" value="4.7uF"/>
 <part name="C153" library="eagle-ltspice" deviceset="C" device="C0201" value="4.7uF"/>
 <part name="C154" library="eagle-ltspice" deviceset="C" device="C0201" value="4.7uF"/>
@@
 <part name="GND743" library="supply1" deviceset="GND" device=""/>
 <part name="GND744" library="supply1" deviceset="GND" device=""/>
-<part name="C176" library="eagle-ltspice" deviceset="C" device="C0201" value="47uF"/>
+<part name="C176" library="eagle-ltspice" deviceset="C" device="C0201" value="4.7uF"/>
 <part name="C177" library="eagle-ltspice" deviceset="C" device="C0201" value="4.7uF"/>
 <part name="C178" library="eagle-ltspice" deviceset="C" device="C0201" value="4.7uF"/>
@@
 <part name="GND1079" library="supply1" deviceset="GND" device=""/>
 <part name="JP20" library="pinhead" deviceset="PINHD-1X2" device=""/>
-<part name="C285" library="eagle-ltspice" deviceset="C" device="C0201" value="47uF"/>
+<part name="C285" library="eagle-ltspice" deviceset="C" device="C0201" value="4.7uF"/>
 <part name="C287" library="eagle-ltspice" deviceset="C" device="C0201" value="4.7uF"/>
 <part name="C289" library="eagle-ltspice" deviceset="C" device="C0201" value="4.7uF"/>

Commit message: feat(hw): ADAR supply order, test points, strobe acknowledgement (#13 #15 #20)
#20 ADAR1000 supply order - the requirement, verified and locked
  The pin table says AVDD3 (+3.3 V) must come up "before or at the same time as the
  AVDD1(-5V) supply"; the "−5 V first" sentence elsewhere in the same datasheet is about an
  external PA's drain (the gate-bias rule).  The firmware already asserts the 3.3 V ADAR rails
  before the 5.0 V rail that creates -5 V through the LM2662 inverters, so this needed no code
  change - it needed the requirement written down at the call site and a test that fails if a
  later edit swaps the order.  docs/power-up-order.md records every device's requirement with
  its citation (ADAR1000 pin table, ADTR1107 Recommended Bias Sequencing, M3SWA2 dual supply,
  LTC5552/AD8352 single supply) and the structural fact that every negative rail here is
  inverted from a positive one, so "negative first" is not physically available.

#15 test points - 15 added where there were zero
  The Harwin S1751-46R (1.63 x 3.25 mm SMT test point, two pads on one node) authored from its
  own land pattern, placed on the power board at the bring-up rails and the three rail-good
  signals, with a BOM row.  docs/probe-map.md already said which pin to meter; this gives the
  probe somewhere to land.

#13 strobe acknowledgement - the MCU can now tell whether the FPGA acted
  strobe_ack.v turns the top's accepted-frame pulse into a level the MCU can poll: a request
  clears it, consumption sets it, so "still low at the next request" means the strobe was
  dropped.  Wired from the already-synchronized pulse, exposed through the 50T wrapper,
  constrained to B16 (bank 15, LVCMOS33 - the same bank as the strobes it answers, so no level
  shift), and carried in the netlist from U42 to U2.PC3.  The FPGA's config net (DONE with
  INIT_B and their pull-ups) now reaches U2.PC4 as FPGA_CFG_OK.  MCU side: STROBE_ACK.{h,c}
  scores each request before the next one is issued - the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
Connections:
- removed net N$115: R144.1, U42G$1.DONE_0
- new net FPGA_DONE: R144.1, U2A.PC4, U42G$1.DONE_0
- new net FPGA_STROBE_ACK: U2A.PC3, U42G$3.IO_L10N_T1_AD11N_15
Changed lines of the file:
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@@
 <busses>
 </busses>
-<nets><net name="PG_2V5_FPGA" class="0"><segment><pinref part="X27" gate="-1" pin="S"/><pinref part="U2" gate="A" pin="PC2"/></segment></net><net name="PG_3V3_XO" class="0"><segment><pinref part="X26" gate="-1" pin="S"/><pinref part="U2" gate="A" pin="PC1"/></segment></net><net name="PG_3V3_ADTR" class="0"><segment><pinref part="X25" gate="-1" pin="S"/><pinref part="U2" gate="A" pin="PC0"/></segment></net><net name="N$U91_OE" class="0"><segment><pinref part="U91" gate="G$1" pin="OE"/><pinref part="R177" gate="G$1" pin="1"/></segment></net><net name="N$U90_OE" class="0"><segment><pinref part="U90" gate="G$1" pin="OE"/><pinref part="R176" gate="G$1" pin="1"/></segment></net><net name="+2V5_FPGA" class="0"><segment><pinref part="U90" gate="G$1" pin="VCCA"/><pinref part="U91" gate="G$1" pin="VCCA"/><pinref part="R176" gate="G$1" pin="2"/><pinref part="R177" gate="G$1" pin="2"/><pinref part="C354" gate="G$1" pin="1"/><pinref part="C355" gate="G$1" pin="1"/><pinref part="C358" gate="G$1" pin="1"/><pinref part="C359" gate="G$1" pin="1"/><pinref part="X57" gate="-1" pin="S"/><pinref part="U42" gate="G$2" pin="VCCO_14"/></segment></net><net name="FLASH_NRST_F" class="0"><segment><pinref part="U9" gate="A" pin="RESET"/><pinref part="U91" gate="G$1" pin="B2"/></segment></net><net name="FLASH_NCS_F" class="0"><segment><pinref part="U9" gate="A" pin="S"/><pinref part="U91" gate="G$1" pin="B1"/></segment></net><net name="FLASH_DQ3_F" class="0"><segment><pinref part="U9" gate="A" pin="DQ3/HOLD"/><pinref part="U90" gate="G$1" pin="B4"/></segment></net><net name="FLASH_DQ2_F" class="0"><segment><pinref part="U9" gate="A" pin="W/DQ2"/><pinref part="U90" gate="G$1" pin="B3"/></segment></net><net name="FLASH_DQ1_F" class="0"><segment><pinref part="U9" gate="A" pin="DQ1"/><pinref part="U90" gate="G$1" pin="B2"/></segment></net><net name="FLASH_DQ0_F" class="0"><segment><pinref part="U9" gate="A" pin="DQ0"/><pinref part="U90" gate="G$1" pin="B1"/></segment></net>
+<nets><net name="FPGA_STROBE_ACK" class="0"><segment><pinref part="U42" gate="G$3" pin="IO_L10N_T1_AD11N_15"/><pinref part="U2" gate="A" pin="PC3"/></segment></net><net name="PG_2V5_FPGA" class="0"><segment><pinref part="X27" gate="-1" pin="S"/><pinref part="U2" gate="A" pin="PC2"/></segment></net><net name="PG_3V3_XO" class="0"><segment><pinref part="X26" gate="-1" pin="S"/><pinref part="U2" gate="A" pin="PC1"/></segment></net><net name="PG_3V3_ADTR" class="0"><segment><pinref part="X25" gate="-1" pin="S"/><pinref part="U2" gate="A" pin="PC0"/></segment></net><net name="N$U91_OE" class="0"><segment><pinref part="U91" gate="G$1" pin="OE"/><pinref part="R177" gate="G$1" pin="1"/></segment></net><net name="N$U90_OE" class="0"><segment><pinref part="U90" gate="G$1" pin="OE"/><pinref part="R176" gate="G$1" pin="1"/></segment></net><net name="+2V5_FPGA" class="0"><segment><pinref part="U90" gate="G$1" pin="VCCA"/><pinref part="U91" gate="G$1" pin="VCCA"/><pinref part="R176" gate="G$1" pin="2"/><pinref part="R177" gate="G$1" pin="2"/><pinref part="C354" gate="G$1" pin="1"/><pinref part="C355" gate="G$1" pin="1"/><pinref part="C358" gate="G$1" pin="1"/><pinref part="C359" gate="G$1" pin="1"/><pinref part="X57" gate="-1" pin="S"/><pinref part="U42" gate="G$2" pin="VCCO_14"/></segment></net><net name="FLASH_NRST_F" class="0"><segment><pinref part="U9" gate="A" pin="RESET"/><pinref part="U91" gate="G$1" pin="B2"/></segment></net><net name="FLASH_NCS_F" class="0"><segment><pinref part="U9" gate="A" pin="S"/><pinref part="U91" gate="G$1" pin="B1"/></segment></net><net name="FLASH_DQ3_F" class="0"><segment><pinref part="U9" gate="A" pin="DQ3/HOLD"/><pinref part="U90" gate="G$1" pin="B4"/></segment></net><net name="FLASH_DQ2_F" class="0"><segment><pinref part="U9" gate="A" pin="W/DQ2"/><pinref part="U90" gate="G$1" pin="B3"/></segment></net><net name="FLASH_DQ1_F" class="0"><segment><pinref part="U9" gate="A" pin="DQ1"/><pinref part="U90" gate="G$1" pin="B2"/></segment></net><net name="FLASH_DQ0_F" class="0"><segment><pinref part="U9" gate="A" pin="DQ0"/><pinref part="U90" gate="G$1" pin="B1"/></segment></net>
 <net name="+3V3" class="0">
 <segment>
@@
 </segment>
 </net>
-<net name="N$115" class="0">
+<net name="FPGA_DONE" class="0">
 <segment>
 <pinref part="R144" gate="G$1" pin="1"/>
@@
 <pinref part="U42" gate="G$1" pin="DONE_0"/>
 <junction x="83.82" y="127"/>
-</segment>
-</net>
+<pinref part="U2" gate="A" pin="PC4"/></segment></net>
 <net name="N$116" class="0">
 <segment>
