File: 4_Schematics and Boards Layout/4_6_Schematics/MainBoard/RADAR_Main_Board.sch (EAGLE design)
At the start: 836 parts, among them IC1 AT93C46A-10SQ-2.7, J1 142-0731-211, J18 142-0731-211, J19 CJT-T-P-HH-ST-TH1, J20 142-0731-211, J21 CJT-T-P-HH-ST-TH1, J22 142-0731-211, J23 142-0731-211, J24 142-0731-211, J25 142-0731-211, J26 142-0731-211, J27 142-0731-211, J28 142-0731-211, J29 142-0731-211, J30 142-0731-211, J31 142-0731-211, J32 142-0731-211, J33 142-0731-211, J34 142-0731-211, J35 142-0731-211, J36 142-0731-211, J37 142-0731-211, J38 142-0731-211, J39 142-0731-211, J40 142-0731-211, J41 142-0731-211, J42 142-0731-211, J43 142-0731-211, J44 142-0731-211, J45 142-0731-211, J46 142-0731-211, J47 142-0731-211, J48 142-0731-211, J49 142-0731-211, J50 142-0731-211, J51 142-0731-211, J52 142-0731-211, J53 142-0731-211, J54 142-0731-211, J55 142-0731-211, J56 142-0731-211, J57 142-0731-211, J58 142-0731-211, J59 142-0731-211, U1 AD9484BCPZ-500, U10 ADS7830IPWR, U11 INA241A4IDGKRDGK0008A-MFG, U13 LTC5552IUDBTRMPBF, U14 SZMMSZ5232BT1G, U15 SZMMSZ5232BT1G, U16 EP4RKU+, U17 SZMMSZ5232BT1G, U2 STM32F746ZGT7, U3 AD9708AR, U37 SZMMSZ5232BT1G, U38 SZMMSZ5232BT1G, U39 SZMMSZ5232BT1G, U4 AD8352ACPZ-R7, U40 SZMMSZ5232BT1G, U41 SZMMSZ5232BT1G, U42 XC7A50T-2FTG256I, U43 SZMMSZ5232BT1G, U44 SZMMSZ5232BT1G, U45 SZMMSZ5232BT1G, U46 SZMMSZ5232BT1G, U47 SZMMSZ5232BT1G, U48 SZMMSZ5232BT1G, U49 SZMMSZ5232BT1G, U5 LTC5552IUDBTRMPBF, U50 SZMMSZ5232BT1G, U51 SZMMSZ5232BT1G, U52 SZMMSZ5232BT1G, U53 SZMMSZ5232BT1G, U54 SZMMSZ5232BT1G, U55 SZMMSZ5232BT1G, U56 SZMMSZ5232BT1G, U57 SZMMSZ5232BT1G, U58 SZMMSZ5232BT1G, U59 SZMMSZ5232BT1G, U6 FT2232HQ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

Commit message: fix(bom): correct five Yageo value codes to their E96 forms (#22)
The errata found that RC0201FR / RC0402FR are Yageo's 1% (F) = E96 series and that none of the five
values in the BOM is an E96 code - while the nearest E96 value resolves at a distributor in every case
and the BOM's form resolves nowhere.  This applies the correction.

  2.443k / RC0201FR-072K44L  ->  2.43k  / RC0201FR-072K43L    (26 designators)
  3k2    / RC0201FR-073K2L   ->  3.16k  / RC0201FR-073K16L   (R33)
  500R   / RC0201FR-07500RL  ->  499R   / RC0201FR-07499RL   (R110, R112-R114)
  840R   / RC0201FR-07840RL  ->  845R   / RC0201FR-07845RL   (R78-R81)
  830R   / RC0402FR-07830RL  ->  825R   / RC0402FR-07825RL   (R36)

Applied in all three places that have to agree - the schematic part's value, the board element's
value, and the BOM row's Value and MPN - because the BOM gate compares the board's value against the
sheet's, and a half-applied change is exactly the defect that check exists to catch.  Each BOM row
carries the reason in its remark column so the change is auditable rather than silent.

Why this is safe: every substitution is smaller than the 1% tolerance the parts already carry
(-0.5%, -1.25%, -0.2%, +0.6%, -0.6%), and all instances of each part number change together, so any
matched set keeps its ratio.

Effect: the five corrected part numbers resolve, so the orderability count moves from 171 to 176 of
179 rows.  The three remaining are the Murata parts whose series is confirmed but whose individual
pages did not surface - a search limit rather than a BOM defect.

The gate caught the change as intended: bom_orderability failed immediately after the edit because
the new part numbers were not yet in the verified list, which is the check doing its job.

Full CI sweep on the pinned interpreter: ruff clean; eight gates green; make test 7/7, 51/51, 36/36;
unit tests 171 passed 3 skipped; cross-layer 45 passed; FPGA regression 32/32.
Parts:
- R103, R104, R105, R106, R119, R120, R121, R122, R89, R90, R91, R92, R95, R96, R97, R98: value 2.443k -> 2.43k
- R110, R112, R113, R114: value 500R -> 499R
- R33: value 3k2 -> 3.16k
- R36: value 830R -> 825R
- R78, R79, R80, R81: value 840R -> 845R
Changed lines of the file:
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@@
 <part name="R77" library="eagle-ltspice" deviceset="R" device="R0201" value="4.7k"/>
 <part name="GND408" library="supply1" deviceset="GND" device=""/>
-<part name="R78" library="eagle-ltspice" deviceset="R" device="R0201" value="840R"/>
-<part name="R79" library="eagle-ltspice" deviceset="R" device="R0201" value="840R"/>
-<part name="R80" library="eagle-ltspice" deviceset="R" device="R0201" value="840R"/>
-<part name="R81" library="eagle-ltspice" deviceset="R" device="R0201" value="840R"/>
+<part name="R78" library="eagle-ltspice" deviceset="R" device="R0201" value="845R"/>
+<part name="R79" library="eagle-ltspice" deviceset="R" device="R0201" value="845R"/>
+<part name="R80" library="eagle-ltspice" deviceset="R" device="R0201" value="845R"/>
+<part name="R81" library="eagle-ltspice" deviceset="R" device="R0201" value="845R"/>
 <part name="ADTR1107_1" library="My_Library_RADAR" deviceset="ADTR1107ACCZ" device=""/>
 <part name="GND291" library="supply1" deviceset="GND" device=""/>
@@
 <part name="R29" library="eagle-ltspice" deviceset="R" device="R0201" value="22R"/>
 <part name="R30" library="eagle-ltspice" deviceset="R" device="R0201" value="22R"/>
-<part name="R33" library="eagle-ltspice" deviceset="R" device="R0201" value="3k2"/>
+<part name="R33" library="eagle-ltspice" deviceset="R" device="R0201" value="3.16k"/>
 <part name="C37" library="eagle-ltspice" deviceset="C" device="C0201" value="0.1uF"/>
 <part name="GND50" library="supply1" deviceset="GND" device=""/>
@@
 <part name="GND90" library="supply1" deviceset="GND" device=""/>
 <part name="GND91" library="supply1" deviceset="GND" device=""/>
-<part name="R36" library="rcl" deviceset="R-EU_" device="R0402" value="830R"/>
+<part name="R36" library="rcl" deviceset="R-EU_" device="R0402" value="825R"/>
 <part name="R37" library="rcl" deviceset="R-EU_" device="R0402" value="1k"/>
 <part name="GND92" library="supply1" deviceset="GND" device=""/>
@@
 <part name="GND697" library="supply1" deviceset="GND" device=""/>
 <part name="GND698" library="supply1" deviceset="GND" device=""/>
-<part name="R89" library="eagle-ltspice" deviceset="R" device="R0201" value="2.443k"/>
-<part name="R90" library="eagle-ltspice" deviceset="R" device="R0201" value="2.443k"/>
-<part name="R91" library="eagle-ltspice" deviceset="R" device="R0201" value="2.443k"/>
-<part name="R92" library="eagle-ltspice" deviceset="R" device="R0201" value="2.443k"/>
+<part name="R89" library="eagle-ltspice" deviceset="R" device="R0201" value="2.43k"/>
+<part name="R90" library="eagle-ltspice" deviceset="R" device="R0201" value="2.43k"/>
+<part name="R91" library="eagle-ltspice" deviceset="R" device="R0201" value="2.43k"/>
+<part name="R92" library="eagle-ltspice" deviceset="R" device="R0201" value="2.43k"/>
 <part name="X_8" library="con-molex" deviceset="22-23-2021" device=""/>
 <part name="GND1" library="supply1" deviceset="GND" device=""/>
@@
 <part name="GND1001" library="supply1" deviceset="GND" device=""/>
 <part name="GND1002" library="supply1" deviceset="GND" device=""/>
-<part name="R95" library="eagle-ltspice" deviceset="R" device="R0201" value="2.443k"/>
-<part name="R96" library="eagle-ltspice" deviceset="R" device="R0201" value="2.443k"/>
-<part name="R97" library="eagle-ltspice" deviceset="R" device="R0201" value="2.443k"/>
-<part name="R98" library="eagle-ltspice" deviceset="R" device="R0201" value="2.443k"/>
+<part name="R95" library="eagle-ltspice" deviceset="R" device="R0201" value="2.43k"/>
+<part name="R96" library="eagle-ltspice" deviceset="R" device="R0201" value="2.43k"/>
+<part name="R97" library="eagle-ltspice" deviceset="R" device="R0201" value="2.43k"/>
+<part name="R98" library="eagle-ltspice" deviceset="R" device="R0201" value="2.43k"/>
 <part name="X_3" library="con-molex" deviceset="22-23-2021" device=""/>
 <part name="GND1003" library="supply1" deviceset="GND" device=""/>
@@
 <part name="GND1009" library="supply1" deviceset="GND" device=""/>
 <part name="GND1010" library="supply1" deviceset="GND" device=""/>
-<part name="R103" library="eagle-ltspice" deviceset="R" device="R0201" value="2.443k"/>
-<part name="R104" library="eagle-ltspice" deviceset="R" device="R0201" value="2.443k"/>
-<part name="R105" library="eagle-ltspice" deviceset="R" device="R0201" value="2.443k"/>
-<part name="R106" library="eagle-ltspice" deviceset="R" device="R0201" value="2.443k"/>
+<part name="R103" library="eagle-ltspice" deviceset="R" device="R0201" value="2.43k"/>
+<part name="R104" library="eagle-ltspice" deviceset="R" device="R0201" value="2.43k"/>
+<part name="R105" library="eagle-ltspice" deviceset="R" device="R0201" value="2.43k"/>
+<part name="R106" library="eagle-ltspice" deviceset="R" device="R0201" value="2.43k"/>
 <part name="X_6" library="con-molex" deviceset="22-23-2021" device=""/>
 <part name="GND1011" library="supply1" deviceset="GND" device=""/>
@@
 <part name="GND1017" library="supply1" deviceset="GND" device=""/>
 <part name="GND1018" library="supply1" deviceset="GND" device=""/>
-<part name="R119" library="eagle-ltspice" deviceset="R" device="R0201" value="2.443k"/>
-<part name="R120" library="eagle-ltspice" deviceset="R" device="R0201" value="2.443k"/>
-<part name="R121" library="eagle-ltspice" deviceset="R" device="R0201" value="2.443k"/>
-<part name="R122" library="eagle-ltspice" deviceset="R" device="R0201" value="2.443k"/>
+<part name="R119" library="eagle-ltspice" deviceset="R" device="R0201" value="2.43k"/>
+<part name="R120" library="eagle-ltspice" deviceset="R" device="R0201" value="2.43k"/>
+<part name="R121" library="eagle-ltspice" deviceset="R" device="R0201" value="2.43k"/>
+<part name="R122" library="eagle-ltspice" deviceset="R" device="R0201" value="2.43k"/>
 <part name="X_1" library="con-molex" deviceset="22-23-2021" device=""/>
 <part name="GND1019" library="supply1" deviceset="GND" device=""/>
@@
 <part name="X53" library="con-cypressindustries" deviceset="MINI-USB-" device="32005-201"/>
 <part name="GND1136" library="supply1" deviceset="GND" device=""/>
-<part name="R110" library="eagle-ltspice" deviceset="R" device="R0201" value="500R"/>
+<part name="R110" library="eagle-ltspice" deviceset="R" device="R0201" value="499R"/>
 <part name="D3" library="SparkFun-LED" deviceset="LED-BLUE" device="0603" value="Blue"/>
-<part name="R112" library="eagle-ltspice" deviceset="R" device="R0201" value="500R"/>
-<part name="R113" library="eagle-ltspice" deviceset="R" device="R0201" value="500R"/>
-<part name="R114" library="eagle-ltspice" deviceset="R" device="R0201" value="500R"/>
+<part name="R112" library="eagle-ltspice" deviceset="R" device="R0201" value="499R"/>
+<part name="R113" library="eagle-ltspice" deviceset="R" device="R0201" value="499R"/>
+<part name="R114" library="eagle-ltspice" deviceset="R" device="R0201" value="499R"/>
 <part name="D2" library="SparkFun-LED" deviceset="LED-BLUE" device="0603" value="Blue"/>
 <part name="D4" library="SparkFun-LED" deviceset="LED-BLUE" device="0603" value="Blue"/>
