File: 4_Schematics and Boards Layout/4_6_Schematics/PowerAmplifierBoard/RF_PA.brd (EAGLE design)
At the start: 35 x 60 mm, 25 parts, among them J1 142-0731-211, J2 142-0731-211, X2 22-23-2021, X3 22-23-2031

Commit message: feat(hw): gate-bias fail-safe, negative-rail margin, PA drain bulk (Lane B B2.2/B1.5/B2.3)
B2.2 -- and this is the finding that matters.  Every one of the 16 gate-bias
channels is an inverting amplifier referenced to ground (Vout = -(Rf/Rin) x VDAC,
+ input on GND), so a DAC in reset puts **0 V on all 16 gates**.  QPA2962 is a
depletion-mode GaN HEMT, where 0 V means *fully on* -- with 22 V on the drains.
That is a power-up hazard, not a nuance.

The plan frames the fix as hardware default *plus* MCU sequence; the hardware half
is here.  One 10k pull-down per channel from VGn to the same negative rail that
supplies its op-amp (R178-R193), so the gates sit at the negative rail whenever
the op-amps are not actively driving: during power-up, power-down, and if an
op-amp is unpowered.  Deliberately not attempted: forcing the gates negative while
the op-amp *is* driving, which would mean moving the + input off ground and
re-characterising all 16 bias channels -- a topology decision with firmware
consequences, recorded rather than guessed.

B1.5 -- the same move feeds it: the four OPA4703 V- pins leave -5V5_PA, whose
LM2662 is at 100 % of rating, for -5V0_ADAR12/34 at ~60 % (two op-amps per rail).
Channels pull down to the rail their own op-amp runs from, so the LM2662 is off
the gate-bias path entirely.

B2.3 -- PA drain bulk was ~20 uF against the ~100 uF the 30 us / 1.68 A pulse
wants; eight more 10 uF 1206 ceramics (C10-C17) on VIN_M use the device this board
already carries, so no new footprint.

Verified: all four files parse (main 2009 parts / 822 elements, PA 51 / 33); no
OPA V- pin or pad remains on -5V5_PA and each ADAR rail carries two op-amps and
eight pull-downs; every VGn net gained exactly one new pull-down (its existing
feedback resistor is the other R on the net); the eight new caps are on VIN_M and
GND; no duplicate designators; gates green.  Both BOMs keep the repo's grouping --
the 10k/R0201 and 10uF/C1206 rows were extended rather than duplicated.

Un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
Parts:
- added C10, C11, C12, C13, C14, C15, C16, C17: 10µF, rcl:C1206
Connections:
- net GND: now also C10.2, C11.2, C12.2, C13.2, C14.2, C15.2, C16.2, C17.2
- net VIN_M: now also C10.1, C11.1, C12.1, C13.1, C14.1, C15.1, C16.1, C17.1
Changed lines of the file:
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@@
 </pass>
 </autorouter>
-<elements>
+<elements><element name="C10" library="rcl" package="C1206" value="10µF" x="22.0" y="27.0" smashed="yes"/><element name="C11" library="rcl" package="C1206" value="10µF" x="21.0" y="33.0" smashed="yes"/><element name="C12" library="rcl" package="C1206" value="10µF" x="27.0" y="31.0" smashed="yes"/><element name="C13" library="rcl" package="C1206" value="10µF" x="15.0" y="30.0" smashed="yes"/><element name="C14" library="rcl" package="C1206" value="10µF" x="22.0" y="39.0" smashed="yes"/><element name="C15" library="rcl" package="C1206" value="10µF" x="15.0" y="36.0" smashed="yes"/><element name="C16" library="rcl" package="C1206" value="10µF" x="28.0" y="37.0" smashed="yes"/><element name="C17" library="rcl" package="C1206" value="10µF" x="30.0" y="25.0" smashed="yes"/>
 <element name="C1" library="rcl" package="C1206" value="10µF" x="6.98" y="23.03" smashed="yes">
 <attribute name="NAME" x="5.71" y="24.3" size="0.6096" layer="25"/>
@@
 <via x="17.539715625" y="12.66049375" extent="1-16" drill="0.15"/>
 <via x="17.552153125" y="12.0386875" extent="1-16" drill="0.15"/>
-</signal>
+<contactref element="C10" pad="2"/><contactref element="C11" pad="2"/><contactref element="C12" pad="2"/><contactref element="C13" pad="2"/><contactref element="C14" pad="2"/><contactref element="C15" pad="2"/><contactref element="C16" pad="2"/><contactref element="C17" pad="2"/></signal>
 <signal name="N$5">
 <contactref element="C4" pad="2"/>
@@
 <wire x1="28.6" y1="32.577" x2="25" y2="36.177" width="0.6" layer="1"/>
 <wire x1="17.455" y1="15.6275" x2="17.455" y2="15.6569" width="0.6" layer="1"/>
-</signal>
+<contactref element="C10" pad="1"/><contactref element="C11" pad="1"/><contactref element="C12" pad="1"/><contactref element="C13" pad="1"/><contactref element="C14" pad="1"/><contactref element="C15" pad="1"/><contactref element="C16" pad="1"/><contactref element="C17" pad="1"/></signal>
 <signal name="N$10">
 <contactref element="R7" pad="2"/>
