File: 4_Schematics and Boards Layout/4_6_Schematics/PowerBoard/PowerBoard.brd (EAGLE design)
At the start: 260 x 300 mm, 313 parts, among them U1 TPS562208DDCT, U10 TPS562208DDCT, U11 TPS562208DDCT, U12 TPS562208DDCT, U13 TPS562208DDCT, U14 TPS562208DDCT, U15 TPS562208DDCT, U16 TPS562208DDCT, U17 TPS562208DDCT, U18 LM2662MX/NOPB, U19 LM2662MX/NOPB, U2 TPS562208DDCT, U20 LM2662MX/NOPB, U21 LM2662MX/NOPB, U22 LM2662MX/NOPB, U23 ADM7151ACPZ-04-R7, U24 TPS562208DDCT, U25 ADM7151ACPZ-04-R7, U26 TPS562208DDCT, U27 ADM7151ACPZ-04-R7, U28 TPS562208DDCT, U29 ADM7151ACPZ-04-R7, U3 TPS562208DDCT, U30 ADM7151ACPZ-04-R7, U31 TPS562208DDCT, U32 TPS7A8300RGRR, U33 TPS562208DDCT, U34 TPS7A8300RGRR, U4 TPS562208DDCT, U5 ADM7151ACPZ-04-R7, U6 TPS562208DDCT, U7 TPS562208DDCT, U8 TPS562208DDCT, U9 TPS562208DDCT, X10 22-23-2021, X11 22-23-2021, X12 22-23-2021, X13 22-23-2021, X14 22-23-2021, X15 22-23-2021, X16 22-23-2021, X17 22-23-2021, X18 22-23-2021, X19 22-23-2021, X2 22-23-2021, X20 22-23-2021, X21 22-23-2021, X22 22-23-2021, X23 22-23-2021, X24 22-23-2021, X25 22-23-2021, X26 22-23-2021, X27 22-23-2021, X28 22-23-2021, X29 22-23-2021, X3 22-23-2021, X30 22-23-2021, X31 22-23-2021, X32 22-23-2021, X33 22-23-2021, X34 22-23-2021, X35 22-23-2021, X36 22-23-2021, X4 22-23-2021, X5 22-23-2021, X6 22-23-2021, X7 22-23-2021, X8 22-23-2021, X9 22-23-2021

Commit message: feat(hw): the 2.5 V rail source for bank 14 (Lane B B1.1, part 1 of 2)
Bank 14 has to reach 2.5 V before the ADC lanes can be LVDS_25, and the supply
has to come from somewhere.  A third TPS7A8300 -- the part that already regulates
twice on the power board (U32 = +3V3_ADTR, U34 = +3V3_XO) -- so the topology,
including the BIAS, NR/SS and SNS capacitors the device needs, is copied from a
working instance rather than designed here.

The set point is derived from the board's own 3.3 V instances, not from memory:

    3.3 V = VREF x (1 + 35.7k/11.5k)       -> VREF = 0.804 V
    2.5 V -> R1/R2 = 2.109; keep the board's 11.5k bottom -> R1 = 24.3k
    0.804 x (1 + 24.3/11.5) = 2.503 V

Capacitors mirror the existing rails' values and packages (22 uF in and out,
10 uF BIAS, 10 nF NR/SS, 10 nF SNS, all C0603); EN is tied to the input rail
because a configuration-bank supply must be up when the FPGA configures.  The
rail leaves the board on the same 2-pin Molex the other rails use, including
X34's two-instance supply-pin pattern.

Placement was searched for clearance from every existing element (a 20-pin LDO
anchored at >12 mm, the passives >=2.5 mm).  Verified: both files parse (572
parts / 322 elements), the rail's net membership matches between schematic and
board (U35 OUT/OUT_2/OUT_3 to pads 20/1/19, plus R59, C165 and the connector),
all three artifact gates green, and the new rail appears in interboard_rails.csv
as a cross-board rail.  The BOM keeps the repo's grouping: C164-C168 and R60 and
U35 join their existing value rows, and 24.3k is the one new row, using the
ERJ-P06 series and the code scheme of the 35.7k part already fitted.

Harmless on its own by design: bank 14 stays on 3.3 V and nothing consumes this
rail yet.  Part 2 -- the two translators, the six line splits and the VCCO_14
move -- is what actually changes the bank, and it has to land with this.
Parts:
- added C164, C165: 22µF, rcl:C0603
- added C166: 10µF, rcl:C0603
- added C167, C168: 10nF, rcl:C0603
- added R59: 24.3k, rcl:M0805
- added R60: 11.5k, rcl:M0805
- added U35: TPS7A8300RGRR, My_Library_RADAR:TPS7A8300RGRR
Connections:
- new net +2V5_FPGA: C165.1, R59.1, U35.1, U35.19, U35.20, X36.1
- new net N$2V5_BIAS: C166.1, U35.12
- new net N$2V5_FB: C168.2, R59.2, R60.1, U35.3
- new net N$2V5_NRSS: C167.1, U35.13
- new net N$2V5_SNS: C168.1, U35.2
- net +5V0_5: now also C164.1, U35.14, U35.15, U35.16, U35.17
- net GND: now also C164.2, C165.2, C166.2, C167.2, R60.2, U35.18, U35.21, U35.8
Changed lines of the file:
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@@
 </pass>
 </autorouter>
-<elements>
+<elements><element name="U35" library="My_Library_RADAR" package="TPS7A8300RGRR" value="TPS7A8300RGRR" x="145.8" y="119.80000000000001" smashed="yes"/><element name="R59" library="rcl" package="M0805" value="24.3k" x="170.0" y="138.0" smashed="yes"/><element name="R60" library="rcl" package="M0805" value="11.5k" x="174.0" y="142.0" smashed="yes"/><element name="C164" library="rcl" package="C0603" value="22µF" x="160.0" y="126.0" smashed="yes"/><element name="C165" library="rcl" package="C0603" value="22µF" x="176.0" y="124.0" smashed="yes"/><element name="C166" library="rcl" package="C0603" value="10µF" x="180.0" y="136.0" smashed="yes"/><element name="C167" library="rcl" package="C0603" value="10nF" x="184.0" y="142.0" smashed="yes"/><element name="C168" library="rcl" package="C0603" value="10nF" x="167.0" y="143.0" smashed="yes"/><element name="X36" library="con-molex" package="22-23-2021" value="22-23-2021" x="190.0" y="131.3" smashed="yes"/>
 <element name="C1" library="rcl" package="C0805" value="0.1µF" x="86.28" y="21.19" smashed="yes" rot="R90">
 <attribute name="NAME" x="87.28" y="24.76" size="1.27" layer="25" rot="R180"/>
@@
 </element>
 </elements>
-<signals>
+<signals><signal name="N$2V5_NRSS" class="0"><contactref element="U35" pad="13"/><contactref element="C167" pad="1"/></signal><signal name="N$2V5_BIAS" class="0"><contactref element="U35" pad="12"/><contactref element="C166" pad="1"/></signal><signal name="N$2V5_SNS" class="0"><contactref element="U35" pad="2"/><contactref element="C168" pad="1"/></signal><signal name="N$2V5_FB" class="0"><contactref element="U35" pad="3"/><contactref element="R59" pad="2"/><contactref element="R60" pad="1"/><contactref element="C168" pad="2"/></signal><signal name="+2V5_FPGA" class="0"><contactref element="U35" pad="20"/><contactref element="U35" pad="1"/><contactref element="U35" pad="19"/><contactref element="R59" pad="1"/><contactref element="C165" pad="1"/><contactref element="X36" pad="1"/></signal>
 <signal name="GND">
 <contactref element="U1" pad="1"/>
@@
 <via x="150.2" y="73.4" extent="1-16" drill="0.6"/>
 <via x="154.8" y="73.4" extent="1-16" drill="0.6"/>
-</signal>
+<contactref element="U35" pad="18"/><contactref element="U35" pad="8"/><contactref element="U35" pad="21"/><contactref element="R60" pad="2"/><contactref element="C164" pad="2"/><contactref element="C165" pad="2"/><contactref element="C166" pad="2"/><contactref element="C167" pad="2"/><contactref element="X36" pad="2"/></signal>
 <signal name="N$1">
 <contactref element="U1" pad="2"/>
@@
 <wire x1="172.724746875" y1="278.2" x2="173.249746875" y2="277.675" width="0.3" layer="1"/>
 <wire x1="173.249746875" y1="277.675" x2="173.749875" y2="277.675" width="0.3" layer="1"/>
-</signal>
+<contactref element="U35" pad="17"/><contactref element="U35" pad="15"/><contactref element="U35" pad="16"/><contactref element="U35" pad="14"/><contactref element="C164" pad="1"/></signal>
 <signal name="N$110">
 </signal>

Commit message: fix(hw): stale sense-amp annotation, and +3V3_XO bulk (Lane B B3.5)
Two grounded fixes, both from the progress audit rather than from the tracker's word.

1. Stale annotation. The main-board sheet has read "6 X INA241A3" twice since before this
   work: once wrong in the part (B2.5 made every sense amplifier an INA241A4) and once
   wrong in the count (the netlist has 16 of them). They sit in two columns of 8
   (U11,U73-U79 at x=419.10 and U80-U87 at x=650.24), so each label annotates one column:
   now "8 X INA241A4" twice, and 2 x 8 = the 16 in the netlist. The neighbouring labels
   ("2 X DAC5578", "3 X ADS7830") already match the netlist, which is the check that made
   this one's staleness visible instead of assumed.

2. B3.5 -- +3V3_XO. Steady state is ~1.25 A (1.2 A OCXO) on a 3 A TPS7A8300: 42 %, fine.
   Added four 22 uF C0603 (C169-C172) on the rail, reusing the part the board already
   carries -- the same BOM row and MPN (KGM15CR51E226MT, qty 54 -> 58) rather than a new
   line. This cuts the rail's source impedance at the heater's step load.

   What it does NOT do, stated plainly: cover a cold-start inrush. A capacitor holds a rail
   for t = C*dV/dI, so the ~32 uF now fitted buys microseconds, not milliseconds. The
   OCXO's inrush current is in no vendor source reachable from here (the part has no
   findable datasheet), so the cold-start capture remains a bench step -- and if it exceeds
   the regulator's 3 A, the fixes are sequencing (U34.EN is tied to +5V0_5 today, so that
   costs an MCU pin) or a soft-start, not more bulk.

Verified: both files parse; all four caps are on +3V3_XO and GND in schematic *and* board;
BOM row is 58 unique refs with all four present; no duplicate designators introduced; three
artifact gates exit 0.

Recorded while checking, not fixed (no decidable answer in the files):
  * X36 appears twice as a board element on the power board -- two connectors, one refdes,
    pre-existing at HEAD. Real BOM/assembly ambiguity, unde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
Parts:
- added C169, C170, C171, C172: 22µF, rcl:C0603
Connections:
- net +3V3_XO: now also C169.1, C170.1, C171.1, C172.1
- net GND: now also C169.2, C170.2, C171.2, C172.2
Changed lines of the file:
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@@
 </pass>
 </autorouter>
-<elements><element name="U35" library="My_Library_RADAR" package="TPS7A8300RGRR" value="TPS7A8300RGRR" x="145.8" y="119.80000000000001" smashed="yes"/><element name="R59" library="rcl" package="M0805" value="24.3k" x="170.0" y="138.0" smashed="yes"/><element name="R60" library="rcl" package="M0805" value="11.5k" x="174.0" y="142.0" smashed="yes"/><element name="C164" library="rcl" package="C0603" value="22µF" x="160.0" y="126.0" smashed="yes"/><element name="C165" library="rcl" package="C0603" value="22µF" x="176.0" y="124.0" smashed="yes"/><element name="C166" library="rcl" package="C0603" value="10µF" x="180.0" y="136.0" smashed="yes"/><element name="C167" library="rcl" package="C0603" value="10nF" x="184.0" y="142.0" smashed="yes"/><element name="C168" library="rcl" package="C0603" value="10nF" x="167.0" y="143.0" smashed="yes"/><element name="X36" library="con-molex" package="22-23-2021" value="22-23-2021" x="190.0" y="131.3" smashed="yes"/>
+<elements><element name="C169" library="rcl" package="C0603" value="22µF" x="149.7" y="245.89999999999998" smashed="yes"/><element name="C170" library="rcl" package="C0603" value="22µF" x="149.7" y="247.89999999999998" smashed="yes"/><element name="C171" library="rcl" package="C0603" value="22µF" x="149.7" y="252.39999999999998" smashed="yes"/><element name="C172" library="rcl" package="C0603" value="22µF" x="149.7" y="256.4" smashed="yes"/><element name="U35" library="My_Library_RADAR" package="TPS7A8300RGRR" value="TPS7A8300RGRR" x="145.8" y="119.80000000000001" smashed="yes"/><element name="R59" library="rcl" package="M0805" value="24.3k" x="170.0" y="138.0" smashed="yes"/><element name="R60" library="rcl" package="M0805" value="11.5k" x="174.0" y="142.0" smashed="yes"/><element name="C164" library="rcl" package="C0603" value="22µF" x="160.0" y="126.0" smashed="yes"/><element name="C165" library="rcl" package="C0603" value="22µF" x="176.0" y="124.0" smashed="yes"/><element name="C166" library="rcl" package="C0603" value="10µF" x="180.0" y="136.0" smashed="yes"/><element name="C167" library="rcl" package="C0603" value="10nF" x="184.0" y="142.0" smashed="yes"/><element name="C168" library="rcl" package="C0603" value="10nF" x="167.0" y="143.0" smashed="yes"/><element name="X36" library="con-molex" package="22-23-2021" value="22-23-2021" x="190.0" y="131.3" smashed="yes"/>
 <element name="C1" library="rcl" package="C0805" value="0.1µF" x="86.28" y="21.19" smashed="yes" rot="R90">
 <attribute name="NAME" x="87.28" y="24.76" size="1.27" layer="25" rot="R180"/>
@@
 <via x="150.2" y="73.4" extent="1-16" drill="0.6"/>
 <via x="154.8" y="73.4" extent="1-16" drill="0.6"/>
-<contactref element="U35" pad="18"/><contactref element="U35" pad="8"/><contactref element="U35" pad="21"/><contactref element="R60" pad="2"/><contactref element="C164" pad="2"/><contactref element="C165" pad="2"/><contactref element="C166" pad="2"/><contactref element="C167" pad="2"/><contactref element="X36" pad="2"/></signal>
+<contactref element="U35" pad="18"/><contactref element="U35" pad="8"/><contactref element="U35" pad="21"/><contactref element="R60" pad="2"/><contactref element="C164" pad="2"/><contactref element="C165" pad="2"/><contactref element="C166" pad="2"/><contactref element="C167" pad="2"/><contactref element="X36" pad="2"/><contactref element="C169" pad="2"/><contactref element="C170" pad="2"/><contactref element="C171" pad="2"/><contactref element="C172" pad="2"/></signal>
 <signal name="N$1">
 <contactref element="U1" pad="2"/>
@@
 <wire x1="182.7" y1="280.1" x2="182.7" y2="281.15" width="0.3" layer="1"/>
 <wire x1="175.250253125" y1="277.675" x2="174.750125" y2="277.675" width="0.3" layer="1"/>
-</signal>
+<contactref element="C169" pad="1"/><contactref element="C170" pad="1"/><contactref element="C171" pad="1"/><contactref element="C172" pad="1"/></signal>
 <signal name="N$13">
 <contactref element="U5" pad="1"/>

Commit message: fix(hw): four netlist defects, and the gate that should have caught them
Chasing the duplicated X36 board element turned up three more defects, and one of them was
electrical.  All four are mine, all from the B1.1 work.

1. Duplicate X36.  Upstream had 35 schematic X parts (X1-X35) but 36 board elements: X36
   existed *only* on the board, wired to +5V0_LO and GND, with no schematic counterpart.
   My B1.1 2.5 V connector then took the refdes X36 -- so the board carried two elements of
   that name while the BOM counted one, which is an assembly ambiguity, not a cosmetic one.
   Fixed the structurally correct way: my connector keeps X36 (it has a schematic part), and
   upstream's orphan element became X37 *and got the schematic part it never had*, so no
   board-only element is left.  BOM 35 -> 36 connectors.

2. Six U9 flash pinrefs used gate="G$1" when the flash's only gate is "A" (upstream writes
   U9 gate="A" pin="RESET").  A pinref naming a gate the part does not instantiate does not
   resolve -- so the B1.1 flash split was NOT actually connected to the flash.  This is the
   one that mattered: the nets now read U9 -> U90/U91 -> U42, i.e. the translators really are
   between the flash and the FPGA.

3. Both of my connectors (power X36, main X57) were instantiated with gate G$1 where the
   deviceset defines -1/-2.  Fixed.

4. None of this was detectable: the BOM/DNP/rail gates look at values, DNP marks and rail
   membership, never at element identity or pin ownership, so all four defects passed CI.

New gate: 9_Firmware/tools/netlist_integrity.py -- seven checks per board: duplicate
schematic-part and board-element designators; a pin claimed by more than one net; a board
element with no schematic part (orphan); a schematic part with no board element (unplaced);
a pinref naming an uninstantiated gate; a board element wired to nothing.  Supply and frame
symbols are exempt (schematic-only by design).  Wired into the CI artifact-gate step beside
the other thre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
Parts:
- added X37: 22-23-2021, con-molex:22-23-2021
- moved X36 133.8 mm to (190.0, 131.3)
Connections:
- net +5V0_LO: now also X37.1; no longer X36.1
- net GND: now also X37.2
Changed lines of the file:
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@@
 <attribute name="VALUE" x="198.33" y="277.51" size="1.016" layer="27" ratio="10" rot="R90"/>
 </element>
-<element name="X36" library="con-molex" package="22-23-2021" value="22-23-2021" x="65.35" y="82.7">
+<element name="X37" library="con-molex" package="22-23-2021" value="22-23-2021" x="65.35" y="82.7">
 <attribute name="MF" value="MOLEX" x="65.35" y="82.7" size="1.778" layer="27" display="off"/>
 <attribute name="OC_NEWARK" value="25C3832" x="65.35" y="82.7" size="1.778" layer="27" display="off"/>
@@
 <via x="150.2" y="73.4" extent="1-16" drill="0.6"/>
 <via x="154.8" y="73.4" extent="1-16" drill="0.6"/>
-<contactref element="U35" pad="18"/><contactref element="U35" pad="8"/><contactref element="U35" pad="21"/><contactref element="R60" pad="2"/><contactref element="C164" pad="2"/><contactref element="C165" pad="2"/><contactref element="C166" pad="2"/><contactref element="C167" pad="2"/><contactref element="X36" pad="2"/><contactref element="C169" pad="2"/><contactref element="C170" pad="2"/><contactref element="C171" pad="2"/><contactref element="C172" pad="2"/></signal>
+<contactref element="U35" pad="18"/><contactref element="U35" pad="8"/><contactref element="U35" pad="21"/><contactref element="R60" pad="2"/><contactref element="C164" pad="2"/><contactref element="C165" pad="2"/><contactref element="C166" pad="2"/><contactref element="C167" pad="2"/><contactref element="X37" pad="2"/><contactref element="C169" pad="2"/><contactref element="C170" pad="2"/><contactref element="C171" pad="2"/><contactref element="C172" pad="2"/></signal>
 <signal name="N$1">
 <contactref element="U1" pad="2"/>
@@
 <contactref element="C140" pad="2"/>
 <contactref element="X6" pad="1"/>
-<contactref element="X36" pad="1"/>
+<contactref element="X37" pad="1"/>
 <polygon width="0.1" layer="1">
 <vertex x="54.6" y="86.2"/>
