File: 4_Schematics and Boards Layout/4_6_Schematics/PowerBoard/PowerBoard.brd (EAGLE design)
At the start: 260 x 300 mm, 326 parts, among them U1 TPS562208DDCT, U10 TPS562208DDCT, U11 TPS562208DDCT, U12 TPS562208DDCT, U13 TPS562208DDCT, U14 TPS562208DDCT, U15 TPS562208DDCT, U16 TPS562208DDCT, U17 TPS562208DDCT, U18 LM2662MX/NOPB, U19 LM2662MX/NOPB, U2 TPS562208DDCT, U20 LM2662MX/NOPB, U21 LM2662MX/NOPB, U22 LM2662MX/NOPB, U23 ADM7151ACPZ-04-R7, U24 TPS562208DDCT, U25 ADM7151ACPZ-04-R7, U26 TPS562208DDCT, U27 ADM7151ACPZ-04-R7, U28 TPS562208DDCT, U29 ADM7151ACPZ-04-R7, U3 TPS562208DDCT, U30 ADM7151ACPZ-04-R7, U31 TPS562208DDCT, U32 TPS7A8300RGRR, U33 TPS562208DDCT, U34 TPS7A8300RGRR, U35 TPS7A8300RGRR, U4 TPS562208DDCT, U5 ADM7151ACPZ-04-R7, U6 TPS562208DDCT, U7 TPS562208DDCT, U8 TPS562208DDCT, U9 TPS562208DDCT, X10 22-23-2021, X11 22-23-2021, X12 22-23-2021, X13 22-23-2021, X14 22-23-2021, X15 22-23-2021, X16 22-23-2021, X17 22-23-2021, X18 22-23-2021, X19 22-23-2021, X2 22-23-2021, X20 22-23-2021, X21 22-23-2021, X22 22-23-2021, X23 22-23-2021, X24 22-23-2021, X25 22-23-2021, X26 22-23-2021, X27 22-23-2021, X28 22-23-2021, X29 22-23-2021, X3 22-23-2021, X30 22-23-2021, X31 22-23-2021, X32 22-23-2021, X33 22-23-2021, X34 22-23-2021, X35 22-23-2021, X36 22-23-2021, X37 22-23-2021, X4 22-23-2021, X5 22-23-2021, X6 22-23-2021, X7 22-23-2021, X8 22-23-2021, X9 22-23-2021

Commit message: fix(hw): revert B1.5, connect the PG pins, and generate the harness map
Five fixes from the remaining-items plan. Two of them are corrections to work already
committed, and one is a correction to the plan itself.

REVERT B1.5.  Its premise was wrong.  The rail budget has -5V5_PA at 100 mA against a 200 mA
LM2662 -- 50 %, not "100 % of rating" as the item claimed -- while -5V0_ADAR12/34 are the
rails that are 1.2x over (240 mA vs 200 mA).  What was moved is negligible anyway: the
OPA4703 datasheet gives 200 uA per amplifier, so ~3 mA of quads plus ~1.6 mA of the new gate
pull-downs.  So the change added load to the two overloaded rails and left U22, C105 and one
harness connector feeding nothing.  All four OPA V- pins and all sixteen gate pull-downs are
back on -5V5_PA, which also puts each pull-down on the same negative rail as the op-amp it
backs up -- the better arrangement.  The real item is B3.1 (the ADAR negative rails).

B1.4/B3.2 PRECONDITION.  U32/U34/U35 each had a PG pin connected to nothing.  TPS7A8300 PG
is active-high open-drain asserting at 89 % of target, so it needs a pull-up to be a defined
level at all.  Nets PG_3V3_ADTR / PG_3V3_XO / PG_2V5_FPGA now carry the pin, and R61-R63
(10 kohm to +3V3) pull them up -- the signal names the connector decision will route.  10 kohm
rather than the datasheet's 100 kohm test condition, because the 10k/M0805 row and its
verified MPN (AE0805BR-0710KL) already exist and 330 uA vs 33 uA when asserted is immaterial
for a fault line.  This is needed by every routing option, so it is not gated on that
decision.

Correction to the plan, found while implementing: a single open-drain PG wire CANNOT be
fail-safe.  "Rail good" (high-Z) and "harness disconnected" are electrically identical no
matter which side carries the pull-up.  The plan claimed otherwise; the honest statement is
that the line is fail-silent on an open harness, and the mitigations are a firmware line-test
(drive low, release, read back) or accepting it.

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
Parts:
- added R61, R62, R63: 10k, rcl:M0805
Connections:
- new net PG_2V5_FPGA: R63.1, U35.4
- new net PG_3V3_ADTR: R61.1, U32.4
- new net PG_3V3_XO: R62.1, U34.4
- net +3V3: now also R61.2, R62.2, R63.2
Changed lines of the file:
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@@
 </pass>
 </autorouter>
-<elements><element name="C169" library="rcl" package="C0603" value="22µF" x="149.7" y="245.89999999999998" smashed="yes"/><element name="C170" library="rcl" package="C0603" value="22µF" x="149.7" y="247.89999999999998" smashed="yes"/><element name="C171" library="rcl" package="C0603" value="22µF" x="149.7" y="252.39999999999998" smashed="yes"/><element name="C172" library="rcl" package="C0603" value="22µF" x="149.7" y="256.4" smashed="yes"/><element name="U35" library="My_Library_RADAR" package="TPS7A8300RGRR" value="TPS7A8300RGRR" x="145.8" y="119.80000000000001" smashed="yes"/><element name="R59" library="rcl" package="M0805" value="24.3k" x="170.0" y="138.0" smashed="yes"/><element name="R60" library="rcl" package="M0805" value="11.5k" x="174.0" y="142.0" smashed="yes"/><element name="C164" library="rcl" package="C0603" value="22µF" x="160.0" y="126.0" smashed="yes"/><element name="C165" library="rcl" package="C0603" value="22µF" x="176.0" y="124.0" smashed="yes"/><element name="C166" library="rcl" package="C0603" value="10µF" x="180.0" y="136.0" smashed="yes"/><element name="C167" library="rcl" package="C0603" value="10nF" x="184.0" y="142.0" smashed="yes"/><element name="C168" library="rcl" package="C0603" value="10nF" x="167.0" y="143.0" smashed="yes"/><element name="X36" library="con-molex" package="22-23-2021" value="22-23-2021" x="190.0" y="131.3" smashed="yes"/>
+<elements><element name="R61" library="rcl" package="M0805" value="10k" x="156.0" y="116.0" smashed="yes"/><element name="R62" library="rcl" package="M0805" value="10k" x="156.0" y="118.0" smashed="yes"/><element name="R63" library="rcl" package="M0805" value="10k" x="156.0" y="120.0" smashed="yes"/><element name="C169" library="rcl" package="C0603" value="22µF" x="149.7" y="245.89999999999998" smashed="yes"/><element name="C170" library="rcl" package="C0603" value="22µF" x="149.7" y="247.89999999999998" smashed="yes"/><element name="C171" library="rcl" package="C0603" value="22µF" x="149.7" y="252.39999999999998" smashed="yes"/><element name="C172" library="rcl" package="C0603" value="22µF" x="149.7" y="256.4" smashed="yes"/><element name="U35" library="My_Library_RADAR" package="TPS7A8300RGRR" value="TPS7A8300RGRR" x="145.8" y="119.80000000000001" smashed="yes"/><element name="R59" library="rcl" package="M0805" value="24.3k" x="170.0" y="138.0" smashed="yes"/><element name="R60" library="rcl" package="M0805" value="11.5k" x="174.0" y="142.0" smashed="yes"/><element name="C164" library="rcl" package="C0603" value="22µF" x="160.0" y="126.0" smashed="yes"/><element name="C165" library="rcl" package="C0603" value="22µF" x="176.0" y="124.0" smashed="yes"/><element name="C166" library="rcl" package="C0603" value="10µF" x="180.0" y="136.0" smashed="yes"/><element name="C167" library="rcl" package="C0603" value="10nF" x="184.0" y="142.0" smashed="yes"/><element name="C168" library="rcl" package="C0603" value="10nF" x="167.0" y="143.0" smashed="yes"/><element name="X36" library="con-molex" package="22-23-2021" value="22-23-2021" x="190.0" y="131.3" smashed="yes"/>
 <element name="C1" library="rcl" package="C0805" value="0.1µF" x="86.28" y="21.19" smashed="yes" rot="R90">
 <attribute name="NAME" x="87.28" y="24.76" size="1.27" layer="25" rot="R180"/>
@@
 </element>
 </elements>
-<signals><signal name="N$2V5_NRSS" class="0"><contactref element="U35" pad="13"/><contactref element="C167" pad="1"/></signal><signal name="N$2V5_BIAS" class="0"><contactref element="U35" pad="12"/><contactref element="C166" pad="1"/></signal><signal name="N$2V5_SNS" class="0"><contactref element="U35" pad="2"/><contactref element="C168" pad="1"/></signal><signal name="N$2V5_FB" class="0"><contactref element="U35" pad="3"/><contactref element="R59" pad="2"/><contactref element="R60" pad="1"/><contactref element="C168" pad="2"/></signal><signal name="+2V5_FPGA" class="0"><contactref element="U35" pad="20"/><contactref element="U35" pad="1"/><contactref element="U35" pad="19"/><contactref element="R59" pad="1"/><contactref element="C165" pad="1"/><contactref element="X36" pad="1"/></signal>
+<signals><signal name="PG_2V5_FPGA" class="0"><contactref element="U35" pad="4"/><contactref element="R63" pad="1"/></signal><signal name="PG_3V3_XO" class="0"><contactref element="U34" pad="4"/><contactref element="R62" pad="1"/></signal><signal name="PG_3V3_ADTR" class="0"><contactref element="U32" pad="4"/><contactref element="R61" pad="1"/></signal><signal name="N$2V5_NRSS" class="0"><contactref element="U35" pad="13"/><contactref element="C167" pad="1"/></signal><signal name="N$2V5_BIAS" class="0"><contactref element="U35" pad="12"/><contactref element="C166" pad="1"/></signal><signal name="N$2V5_SNS" class="0"><contactref element="U35" pad="2"/><contactref element="C168" pad="1"/></signal><signal name="N$2V5_FB" class="0"><contactref element="U35" pad="3"/><contactref element="R59" pad="2"/><contactref element="R60" pad="1"/><contactref element="C168" pad="2"/></signal><signal name="+2V5_FPGA" class="0"><contactref element="U35" pad="20"/><contactref element="U35" pad="1"/><contactref element="U35" pad="19"/><contactref element="R59" pad="1"/><contactref element="C165" pad="1"/><contactref element="X36" pad="1"/></signal>
 <signal name="GND">
 <contactref element="U1" pad="1"/>
@@
 <wire x1="52.7" y1="36.15" x2="37.3" y2="36.15" width="0.5" layer="1"/>
 <wire x1="57.13" y1="31.72" x2="52.7" y2="36.15" width="0.5" layer="1"/>
-</signal>
+<contactref element="R61" pad="2"/><contactref element="R62" pad="2"/><contactref element="R63" pad="2"/></signal>
 <signal name="EN_+3V3_FPGA">
 <contactref element="U4" pad="5"/>

Commit message: feat(backlog): close the six remaining Lane B decisions (#5 #7 #8 #9 #10 #24)
#5 PA operating mode: PA_BIAS_SEQUENCE.{h,c} make the gate/drain order a tested
   contract (enable: gate off -> drain -> settle -> operating bias; disable: gate
   off -> drain off; every failure path lands safe). 17/17, wired into startup and
   Emergency_Stop in main.cpp.
#7 harmonic filter: docs/harmonic-filter.md - spec, the existing SMA interface, the
   measurement that must set the filter order, and the three options.
#8 rail-good routing: three TPS7A8300 PG signals each get their own 2-position
   connector pair (power X38-X40 -> main X25-X27 -> U2.PC0-PC2, verified free).
   RAIL_FAULT.{h,c} samples and latches them, 19/19, wired into the main loop and
   telemetry. The pins are read with pull-downs, so an open harness reads LOW and is
   reported as a fault - the earlier "fail-silent" note was wrong and is corrected.
#9 negative rails: U36/U37 parallel U20/U21 on -5V0_ADAR12/34, each with its own
   47 uF pumping cap and the shared output cap, exactly as TI's datasheet requires.
   Two in parallel halve the output resistance and double the headroom (240 mA of a
   400 mA capability instead of 1.2x over a 200 mA part).
#10 keying: negative rails move to the 3-position part and the PA drain feeds to a
   4-position part with two pins per rail (which also halves the 4 A per pin). The
   4-position part is authored from the repo's own 22-23-2031 geometry. One rail was
   spelled two ways across boards (+3V3_ADAR_12 vs +3V3_ADAR12) and is now unified.
   The harness map's keying column is generated from the parts, not typed.
#24 laminate: the PA board moves to RO4350B (recorded in FAB_NOTES.md); the patch
   array is gerbers-only and flagged as un-respinnable.

Verification: netlist_integrity caught two real regressions during this work (gate
names the part did not instantiate; designators dropped from the authored BOM) and
both are fixed. All six artifact gates and ruff are green.
Parts:
- added C173, C174: T521W476M020ATE045, T521W476M020ATE045:T521W
- added U36, U37: LM2662MX/NOPB, My_Library_RADAR:M08A
- added X38, X39, X40: 22-23-2021, con-molex:22-23-2021
- X18, X19, X20, X21, X24: device con-molex:22-23-2021 -> con-molex:22-23-2031
- X31, X32, X33: device con-molex:22-23-2021 -> con-molex:22-23-2041
Connections:
- new net N$U36_C1M: C173.2, U36.4
- new net N$U36_C1P: C173.1, U36.2
- new net N$U37_C1M: C174.2, U37.4
- new net N$U37_C1P: C174.1, U37.2
- net +5V0_ADAR: now also U36.8, U37.8
- net -5V0_ADAR12: now also U36.5
- net -5V0_ADAR34: now also U37.5
- net GND: now also U36.3, U36.6, U37.3, U37.6, X18.3, X19.3, X20.3, X21.3, X24.3, X31.3, X31.4, X32.3, X32.4, X33.3, X33.4, X38.2, X39.2, X40.2
- net PG_2V5_FPGA: now also X40.1
- net PG_3V3_ADTR: now also X38.1
- net PG_3V3_XO: now also X39.1
