File: 4_Schematics and Boards Layout/4_6_Schematics/PowerBoard/PowerBoard.brd (EAGLE design)
At the start: 260 x 300 mm, 336 parts, among them U1 TPS562208DDCT, U10 TPS562208DDCT, U11 TPS562208DDCT, U12 TPS562208DDCT, U13 TPS562208DDCT, U14 TPS562208DDCT, U15 TPS562208DDCT, U16 TPS562208DDCT, U17 TPS562208DDCT, U18 LM2662MX/NOPB, U19 LM2662MX/NOPB, U2 TPS562208DDCT, U20 LM2662MX/NOPB, U21 LM2662MX/NOPB, U22 LM2662MX/NOPB, U23 ADM7151ACPZ-04-R7, U24 TPS562208DDCT, U25 ADM7151ACPZ-04-R7, U26 TPS562208DDCT, U27 ADM7151ACPZ-04-R7, U28 TPS562208DDCT, U29 ADM7151ACPZ-04-R7, U3 TPS562208DDCT, U30 ADM7151ACPZ-04-R7, U31 TPS562208DDCT, U32 TPS7A8300RGRR, U33 TPS562208DDCT, U34 TPS7A8300RGRR, U35 TPS7A8300RGRR, U36 LM2662MX/NOPB, U37 LM2662MX/NOPB, U4 TPS562208DDCT, U5 ADM7151ACPZ-04-R7, U6 TPS562208DDCT, U7 TPS562208DDCT, U8 TPS562208DDCT, U9 TPS562208DDCT, X10 22-23-2021, X11 22-23-2021, X12 22-23-2021, X13 22-23-2021, X14 22-23-2021, X15 22-23-2021, X16 22-23-2021, X17 22-23-2021, X18 22-23-2021, X19 22-23-2021, X2 22-23-2021, X20 22-23-2021, X21 22-23-2021, X22 22-23-2021, X23 22-23-2021, X24 22-23-2021, X25 22-23-2021, X26 22-23-2021, X27 22-23-2021, X28 22-23-2021, X29 22-23-2021, X3 22-23-2021, X30 22-23-2021, X31 22-23-2021, X32 22-23-2021, X33 22-23-2021, X34 22-23-2021, X35 22-23-2021, X36 22-23-2021, X37 22-23-2021, X38 22-23-2021, X39 22-23-2021, X4 22-23-2021, X40 22-23-2021, X5 22-23-2021, X6 22-23-2021, X7 22-23-2021, X8 22-23-2021, X9 22-23-2021

Commit message: fix(tools): the BOM gate now checks which row a part sits on, not just that it exists
regenerate_bom.py compared designator *presence* between the board and the sheet, so a
designator could sit on the wrong row and pass. That is exactly how the harness keying change
went wrong earlier: the new rows were cloned and inherited the whole 2-position list, and the
gate stayed green.

It now compares the board's value against the value on the sheet row the designator appears in,
normalising the micro glyph and accepting a containment match so that "100nF" vs "100nF/50V"
is not a finding. Verified by fault injection: moving X31 onto the 22-23-2021 row makes the
check name it, and restoring makes it clean again.

It found two real defects, both fixed here:

- X19 on the main board still carried value 22-23-2021 after its part became 22-23-2031 (the
  earlier element-value fix omitted it), so the board disagreed with its own package.
- C17, C55, C176 and C285 read 47uF on the board while the ordered part is CM03X5R475M06AH055.
  The three-digit code 475 is 47 x 10^5 pF = 4.7 uF and no 0201 case holds 47 uF, so the board
  value was the typo and the sheet's 4.7uF was right. Corrected in both the schematic and the
  board element.

Also closes the loop on the four issues verified this round: #4 (shunt MPN corrected, INA241A4
sense amps in the BOM), #11 (six gates in CI), #18 (laminate recorded), #25 (no board-only
elements).
Parts:
- X18, X19, X20, X21, X24: value 22-23-2021 -> 22-23-2031
- X31, X32, X33: value 22-23-2021 -> 22-23-2041
Changed lines of the file:
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@@
 <attribute name="VALUE" x="37.28" y="34.85" size="1.016" layer="27" ratio="10"/>
 </element>
-<element name="X18" library="con-molex" package="22-23-2031" value="22-23-2021" x="195.26" y="154.32" smashed="yes" rot="R180">
+<element name="X18" library="con-molex" package="22-23-2031" value="22-23-2031" x="195.26" y="154.32" smashed="yes" rot="R180">
 <attribute name="MF" value="MOLEX" x="140.65" y="273.7" size="1.778" layer="27" rot="R180" display="off"/>
 <attribute name="MPN" value="22-23-2021" x="140.65" y="273.7" size="1.778" layer="27" rot="R180" display="off"/>
@@
 <attribute name="VALUE" x="197.8" y="159.4" size="1.016" layer="27" ratio="10" rot="R180"/>
 </element>
-<element name="X19" library="con-molex" package="22-23-2031" value="22-23-2021" x="74.48" y="205" smashed="yes" rot="R270">
+<element name="X19" library="con-molex" package="22-23-2031" value="22-23-2031" x="74.48" y="205" smashed="yes" rot="R270">
 <attribute name="MF" value="MOLEX" x="-44.9" y="141.5" size="1.778" layer="27" rot="R270" display="off"/>
 <attribute name="MPN" value="22-23-2021" x="-44.9" y="141.5" size="1.778" layer="27" rot="R270" display="off"/>
@@
 <attribute name="VALUE" x="69.4" y="207.54" size="1.016" layer="27" ratio="10" rot="R270"/>
 </element>
-<element name="X20" library="con-molex" package="22-23-2031" value="22-23-2021" x="136.73" y="128.24" smashed="yes" rot="R270">
+<element name="X20" library="con-molex" package="22-23-2031" value="22-23-2031" x="136.73" y="128.24" smashed="yes" rot="R270">
 <attribute name="MF" value="MOLEX" x="17.35" y="55.85" size="1.778" layer="27" rot="R270" display="off"/>
 <attribute name="MPN" value="22-23-2021" x="17.35" y="55.85" size="1.778" layer="27" rot="R270" display="off"/>
@@
 <attribute name="VALUE" x="131.65" y="130.78" size="1.016" layer="27" ratio="10" rot="R270"/>
 </element>
-<element name="X21" library="con-molex" package="22-23-2031" value="22-23-2021" x="100.73" y="103.18" smashed="yes" rot="R270">
+<element name="X21" library="con-molex" package="22-23-2031" value="22-23-2031" x="100.73" y="103.18" smashed="yes" rot="R270">
 <attribute name="MF" value="MOLEX" x="-18.65" y="21.9" size="1.778" layer="27" rot="R270" display="off"/>
 <attribute name="MPN" value="22-23-2021" x="-18.65" y="21.9" size="1.778" layer="27" rot="R270" display="off"/>
@@
 <attribute name="VALUE" x="85.9" y="93.8" size="1.016" layer="27" ratio="10"/>
 </element>
-<element name="X24" library="con-molex" package="22-23-2031" value="22-23-2021" x="64.53" y="102.55" smashed="yes" rot="R270">
+<element name="X24" library="con-molex" package="22-23-2031" value="22-23-2031" x="64.53" y="102.55" smashed="yes" rot="R270">
 <attribute name="MF" value="MOLEX" x="-54.85" y="-5.4" size="1.778" layer="27" rot="R270" display="off"/>
 <attribute name="MPN" value="22-23-2021" x="-54.85" y="-5.4" size="1.778" layer="27" rot="R270" display="off"/>
@@
 <attribute name="VALUE" x="48.553" y="160.279" size="1.016" layer="27" ratio="10" rot="R90"/>
 </element>
-<element name="X31" library="con-molex" package="22-23-2041" value="22-23-2021" x="85.727" y="161.946" smashed="yes" rot="R90">
+<element name="X31" library="con-molex" package="22-23-2041" value="22-23-2041" x="85.727" y="161.946" smashed="yes" rot="R90">
 <attribute name="MF" value="MOLEX" x="74.827" y="155.546" size="1.778" layer="27" rot="R90" display="off"/>
 <attribute name="MPN" value="22-23-2021" x="74.827" y="155.546" size="1.778" layer="27" rot="R90" display="off"/>
@@
 <attribute name="VALUE" x="90.807" y="159.406" size="1.016" layer="27" ratio="10" rot="R90"/>
 </element>
-<element name="X32" library="con-molex" package="22-23-2041" value="22-23-2021" x="122.442" y="161.78" smashed="yes" rot="R90">
+<element name="X32" library="con-molex" package="22-23-2041" value="22-23-2041" x="122.442" y="161.78" smashed="yes" rot="R90">
 <attribute name="MF" value="MOLEX" x="111.542" y="155.38" size="1.778" layer="27" rot="R90" display="off"/>
 <attribute name="MPN" value="22-23-2021" x="111.542" y="155.38" size="1.778" layer="27" rot="R90" display="off"/>
@@
 <attribute name="VALUE" x="127.522" y="159.24" size="1.016" layer="27" ratio="10" rot="R90"/>
 </element>
-<element name="X33" library="con-molex" package="22-23-2041" value="22-23-2021" x="158.383" y="161.272" smashed="yes" rot="R90">
+<element name="X33" library="con-molex" package="22-23-2041" value="22-23-2041" x="158.383" y="161.272" smashed="yes" rot="R90">
 <attribute name="MF" value="MOLEX" x="147.483" y="154.872" size="1.778" layer="27" rot="R90" display="off"/>
 <attribute name="MPN" value="22-23-2021" x="147.483" y="154.872" size="1.778" layer="27" rot="R90" display="off"/>

Commit message: feat(hw): ADAR supply order, test points, strobe acknowledgement (#13 #15 #20)
#20 ADAR1000 supply order - the requirement, verified and locked
  The pin table says AVDD3 (+3.3 V) must come up "before or at the same time as the
  AVDD1(-5V) supply"; the "−5 V first" sentence elsewhere in the same datasheet is about an
  external PA's drain (the gate-bias rule).  The firmware already asserts the 3.3 V ADAR rails
  before the 5.0 V rail that creates -5 V through the LM2662 inverters, so this needed no code
  change - it needed the requirement written down at the call site and a test that fails if a
  later edit swaps the order.  docs/power-up-order.md records every device's requirement with
  its citation (ADAR1000 pin table, ADTR1107 Recommended Bias Sequencing, M3SWA2 dual supply,
  LTC5552/AD8352 single supply) and the structural fact that every negative rail here is
  inverted from a positive one, so "negative first" is not physically available.

#15 test points - 15 added where there were zero
  The Harwin S1751-46R (1.63 x 3.25 mm SMT test point, two pads on one node) authored from its
  own land pattern, placed on the power board at the bring-up rails and the three rail-good
  signals, with a BOM row.  docs/probe-map.md already said which pin to meter; this gives the
  probe somewhere to land.

#13 strobe acknowledgement - the MCU can now tell whether the FPGA acted
  strobe_ack.v turns the top's accepted-frame pulse into a level the MCU can poll: a request
  clears it, consumption sets it, so "still low at the next request" means the strobe was
  dropped.  Wired from the already-synchronized pulse, exposed through the 50T wrapper,
  constrained to B16 (bank 15, LVCMOS33 - the same bank as the strobes it answers, so no level
  shift), and carried in the netlist from U42 to U2.PC3.  The FPGA's config net (DONE with
  INIT_B and their pull-ups) now reaches U2.PC4 as FPGA_CFG_OK.  MCU side: STROBE_ACK.{h,c}
  scores each request before the next one is issued - the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
Parts:
- added TP1, TP10, TP11, TP12, TP13, TP14, TP15, TP2, TP3, TP4, TP5, TP6, TP7, TP8, TP9: S1751-46R, My_Library_RADAR:S1751-46
Connections:
- net +3V3_ADAR_34 renamed +3V3_ADAR34
- removed net +3V3_ADAR_12: C31.1, C32.1, C35.1, R11.2, U$6.1, X14.1
- new net +3V3_ADAR12: C31.1, C32.1, C35.1, R11.2, TP8.1, TP8.2, U$6.1, X14.1
- net +1V0_FPGA: now also TP1.1, TP1.2
- net +1V8_FPGA: now also TP2.1, TP2.2
- net +2V5_FPGA: now also TP3.1, TP3.2
- net +3V3: now also TP4.1, TP4.2
- net +3V3_ADTR: now also TP6.1, TP6.2
- net +3V3_AN: now also TP5.1, TP5.2
- net +3V3_XO: now also TP7.1, TP7.2
- net +3V4: now also TP10.1, TP10.2
- net +5V5_PA: now also TP12.1, TP12.2
- net -3V4: now also TP11.1, TP11.2
- net -5V0_ADAR12: now also TP9.1, TP9.2
- net PG_2V5_FPGA: now also TP15.1, TP15.2
- net PG_3V3_ADTR: now also TP13.1, TP13.2
- net PG_3V3_XO: now also TP14.1, TP14.2
Routing:
- net +3V3_ADAR_12: track 36.3 -> 0.00 mm
- net +3V3_ADAR12: track 0.00 -> 36.3 mm
- added copper zone on layer 1, net +3V3_ADAR12
- removed copper zone on layer 1, net +3V3_ADAR_12

Commit message: feat(hw): power-sequencing gate, and the BOM check now compares packages (#20 #26)
#20 The issue asked whether three converters with EN tied to VIN break the power-up order, and
   whether to re-stage them. The answer is that they do not, for a structural reason:

     every negative rail on this board is an LM2662 charge pump, and a charge pump has no enable
     pin - it runs whenever its V+ is present.  So a negative rail cannot precede the positive
     rail feeding it.

   Verified rail by rail: U18 (-3V3_SW) is fed from +3V3_SW, which is itself staged on MCU PE14;
   U20/U21/U36/U37 (-5V0_ADAR*) from +5V0_ADAR (staged, U13, PE10); U22 (-5V5_PA) from +5V5_PA
   (staged, U17); U19 (-3V4) from +3V4.  A gate finds thirteen converters with EN tied to their
   input and every one is a POSITIVE rail, which is why they are harmless.

   That is exactly what the GaAs parts require.  The ADTR1107 datasheet states its sequence
   explicitly: transmit power-up is GND, then VDD_SW = 3.3 V, then VSS_SW = -3.3 V - the positive
   switch rail first.  The design meets it, and by construction rather than by sequencing logic.

   9_Firmware/tools/power_sequencing.py locks the property (each pump draws from a positive rail of
   its own family), is wired into CI as the eighth gate, and is documented in docs/power-up-order.md
   with the datasheet citation.  Verified by fault injection: re-sourcing U18 from a negative rail
   yields "U18: -3V3_SW is fed from -3V4, which is not a positive rail" and a non-zero exit.

   Writing that gate also caught me re-making a recorded mistake: it built a {net: body} dict from
   Eagle nets, whose names repeat, so one net silently overwrote another.  It now uses a list.

#26 The residual on this issue was that the check compared values but not packages.  read_sheet now
   returns the sheet's Package column and the check compares it against the board's package, with
   the same normalisation and containment rule.

   It immediately found a real d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
Parts:
- U35: device My_Library_RADAR:TPS7A8300RGRR -> My_Library_RADAR:RGR20_2P05X2P05_TEX
Changed lines of the file:
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@@
 </pass>
 </autorouter>
-<elements><element name="TP15" library="My_Library_RADAR" package="S1751-46" value="S1751-46R" x="104.0" y="88.0" smashed="yes"/><element name="TP14" library="My_Library_RADAR" package="S1751-46" value="S1751-46R" x="98.0" y="88.0" smashed="yes"/><element name="TP13" library="My_Library_RADAR" package="S1751-46" value="S1751-46R" x="92.0" y="88.0" smashed="yes"/><element name="TP12" library="My_Library_RADAR" package="S1751-46" value="S1751-46R" x="86.0" y="88.0" smashed="yes"/><element name="TP11" library="My_Library_RADAR" package="S1751-46" value="S1751-46R" x="80.0" y="88.0" smashed="yes"/><element name="TP10" library="My_Library_RADAR" package="S1751-46" value="S1751-46R" x="134.0" y="80.0" smashed="yes"/><element name="TP9" library="My_Library_RADAR" package="S1751-46" value="S1751-46R" x="128.0" y="80.0" smashed="yes"/><element name="TP8" library="My_Library_RADAR" package="S1751-46" value="S1751-46R" x="122.0" y="80.0" smashed="yes"/><element name="TP7" library="My_Library_RADAR" package="S1751-46" value="S1751-46R" x="116.0" y="80.0" smashed="yes"/><element name="TP6" library="My_Library_RADAR" package="S1751-46" value="S1751-46R" x="110.0" y="80.0" smashed="yes"/><element name="TP5" library="My_Library_RADAR" package="S1751-46" value="S1751-46R" x="104.0" y="80.0" smashed="yes"/><element name="TP4" library="My_Library_RADAR" package="S1751-46" value="S1751-46R" x="98.0" y="80.0" smashed="yes"/><element name="TP3" library="My_Library_RADAR" package="S1751-46" value="S1751-46R" x="92.0" y="80.0" smashed="yes"/><element name="TP2" library="My_Library_RADAR" package="S1751-46" value="S1751-46R" x="86.0" y="80.0" smashed="yes"/><element name="TP1" library="My_Library_RADAR" package="S1751-46" value="S1751-46R" x="80.0" y="80.0" smashed="yes"/><element name="X38" library="con-molex" package="22-23-2021" value="22-23-2021" x="166.0" y="102.0" smashed="yes"/><element name="X39" library="con-molex" package="22-23-2021" value="22-23-2021" x="170.5" y="114.5" smashed="yes"/><element name="X40" library="con-molex" package="22-23-2021" value="22-23-2021" x="171.5" y="152.0" smashed="yes"/><element name="U36" library="My_Library_RADAR" package="M08A" value="LM2662MX/NOPB" x="96.15" y="87.85" smashed="yes"/><element name="C173" library="T521W476M020ATE045" package="T521W" value="T521W476M020ATE045" x="96.15" y="90.35" smashed="yes"/><element name="U37" library="My_Library_RADAR" package="M08A" value="LM2662MX/NOPB" x="103.34" y="109.47999999999999" smashed="yes"/><element name="C174" library="T521W476M020ATE045" package="T521W" value="T521W476M020ATE045" x="103.34" y="111.97999999999999" smashed="yes"/><element name="R61" library="rcl" package="M0805" value="10k" x="156.0" y="116.0" smashed="yes"/><element name="R62" library="rcl" package="M0805" value="10k" x="156.0" y="118.0" smashed="yes"/><element name="R63" library="rcl" package="M0805" value="10k" x="156.0" y="120.0" smashed="yes"/><element name="C169" library="rcl" package="C0603" value="22µF" x="149.7" y="245.89999999999998" smashed="yes"/><element name="C170" library="rcl" package="C0603" value="22µF" x="149.7" y="247.89999999999998" smashed="yes"/><element name="C171" library="rcl" package="C0603" value="22µF" x="149.7" y="252.39999999999998" smashed="yes"/><element name="C172" library="rcl" package="C0603" value="22µF" x="149.7" y="256.4" smashed="yes"/><element name="U35" library="My_Library_RADAR" package="TPS7A8300RGRR" value="TPS7A8300RGRR" x="145.8" y="119.80000000000001" smashed="yes"/><element name="R59" library="rcl" package="M0805" value="24.3k" x="170.0" y="138.0" smashed="yes"/><element name="R60" library="rcl" package="M0805" value="11.5k" x="174.0" y="142.0" smashed="yes"/><element name="C164" library="rcl" package="C0603" value="22µF" x="160.0" y="126.0" smashed="yes"/><element name="C165" library="rcl" package="C0603" value="22µF" x="176.0" y="124.0" smashed="yes"/><element name="C166" library="rcl" package="C0603" value="10µF" x="180.0" y="136.0" smashed="yes"/><element name="C167" library="rcl" package="C0603" value="10nF" x="184.0" y="142.0" smashed="yes"/><element name="C168" library="rcl" package="C0603" value="10nF" x="167.0" y="143.0" smashed="yes"/><element name="X36" library="con-molex" package="22-23-2021" value="22-23-2021" x="190.0" y="131.3" smashed="yes"/>
+<elements><element name="TP15" library="My_Library_RADAR" package="S1751-46" value="S1751-46R" x="104.0" y="88.0" smashed="yes"/><element name="TP14" library="My_Library_RADAR" package="S1751-46" value="S1751-46R" x="98.0" y="88.0" smashed="yes"/><element name="TP13" library="My_Library_RADAR" package="S1751-46" value="S1751-46R" x="92.0" y="88.0" smashed="yes"/><element name="TP12" library="My_Library_RADAR" package="S1751-46" value="S1751-46R" x="86.0" y="88.0" smashed="yes"/><element name="TP11" library="My_Library_RADAR" package="S1751-46" value="S1751-46R" x="80.0" y="88.0" smashed="yes"/><element name="TP10" library="My_Library_RADAR" package="S1751-46" value="S1751-46R" x="134.0" y="80.0" smashed="yes"/><element name="TP9" library="My_Library_RADAR" package="S1751-46" value="S1751-46R" x="128.0" y="80.0" smashed="yes"/><element name="TP8" library="My_Library_RADAR" package="S1751-46" value="S1751-46R" x="122.0" y="80.0" smashed="yes"/><element name="TP7" library="My_Library_RADAR" package="S1751-46" value="S1751-46R" x="116.0" y="80.0" smashed="yes"/><element name="TP6" library="My_Library_RADAR" package="S1751-46" value="S1751-46R" x="110.0" y="80.0" smashed="yes"/><element name="TP5" library="My_Library_RADAR" package="S1751-46" value="S1751-46R" x="104.0" y="80.0" smashed="yes"/><element name="TP4" library="My_Library_RADAR" package="S1751-46" value="S1751-46R" x="98.0" y="80.0" smashed="yes"/><element name="TP3" library="My_Library_RADAR" package="S1751-46" value="S1751-46R" x="92.0" y="80.0" smashed="yes"/><element name="TP2" library="My_Library_RADAR" package="S1751-46" value="S1751-46R" x="86.0" y="80.0" smashed="yes"/><element name="TP1" library="My_Library_RADAR" package="S1751-46" value="S1751-46R" x="80.0" y="80.0" smashed="yes"/><element name="X38" library="con-molex" package="22-23-2021" value="22-23-2021" x="166.0" y="102.0" smashed="yes"/><element name="X39" library="con-molex" package="22-23-2021" value="22-23-2021" x="170.5" y="114.5" smashed="yes"/><element name="X40" library="con-molex" package="22-23-2021" value="22-23-2021" x="171.5" y="152.0" smashed="yes"/><element name="U36" library="My_Library_RADAR" package="M08A" value="LM2662MX/NOPB" x="96.15" y="87.85" smashed="yes"/><element name="C173" library="T521W476M020ATE045" package="T521W" value="T521W476M020ATE045" x="96.15" y="90.35" smashed="yes"/><element name="U37" library="My_Library_RADAR" package="M08A" value="LM2662MX/NOPB" x="103.34" y="109.47999999999999" smashed="yes"/><element name="C174" library="T521W476M020ATE045" package="T521W" value="T521W476M020ATE045" x="103.34" y="111.97999999999999" smashed="yes"/><element name="R61" library="rcl" package="M0805" value="10k" x="156.0" y="116.0" smashed="yes"/><element name="R62" library="rcl" package="M0805" value="10k" x="156.0" y="118.0" smashed="yes"/><element name="R63" library="rcl" package="M0805" value="10k" x="156.0" y="120.0" smashed="yes"/><element name="C169" library="rcl" package="C0603" value="22µF" x="149.7" y="245.89999999999998" smashed="yes"/><element name="C170" library="rcl" package="C0603" value="22µF" x="149.7" y="247.89999999999998" smashed="yes"/><element name="C171" library="rcl" package="C0603" value="22µF" x="149.7" y="252.39999999999998" smashed="yes"/><element name="C172" library="rcl" package="C0603" value="22µF" x="149.7" y="256.4" smashed="yes"/><element name="U35" library="My_Library_RADAR" package="RGR20_2P05X2P05_TEX" value="TPS7A8300RGRR" x="145.8" y="119.80000000000001" smashed="yes"/><element name="R59" library="rcl" package="M0805" value="24.3k" x="170.0" y="138.0" smashed="yes"/><element name="R60" library="rcl" package="M0805" value="11.5k" x="174.0" y="142.0" smashed="yes"/><element name="C164" library="rcl" package="C0603" value="22µF" x="160.0" y="126.0" smashed="yes"/><element name="C165" library="rcl" package="C0603" value="22µF" x="176.0" y="124.0" smashed="yes"/><element name="C166" library="rcl" package="C0603" value="10µF" x="180.0" y="136.0" smashed="yes"/><element name="C167" library="rcl" package="C0603" value="10nF" x="184.0" y="142.0" smashed="yes"/><element name="C168" library="rcl" package="C0603" value="10nF" x="167.0" y="143.0" smashed="yes"/><element name="X36" library="con-molex" package="22-23-2021" value="22-23-2021" x="190.0" y="131.3" smashed="yes"/>
 <element name="C1" library="rcl" package="C0805" value="0.1µF" x="86.28" y="21.19" smashed="yes" rot="R90">
 <attribute name="NAME" x="87.28" y="24.76" size="1.27" layer="25" rot="R180"/>
