File: 4_Schematics and Boards Layout/4_6_Schematics/PowerBoard/PowerBoard.sch (EAGLE design)
At the start: 325 parts, among them U1 TPS562208DDCT, U10 TPS562208DDCT, U11 TPS562208DDCT, U12 TPS562208DDCT, U13 TPS562208DDCT, U14 TPS562208DDCT, U15 TPS562208DDCT, U16 TPS562208DDCT, U17 TPS562208DDCT, U18 LM2662MX/NOPB, U19 LM2662MX/NOPB, U2 TPS562208DDCT, U20 LM2662MX/NOPB, U21 LM2662MX/NOPB, U22 LM2662MX/NOPB, U23 ADM7151ACPZ-04-R7, U24 TPS562208DDCT, U25 ADM7151ACPZ-04-R7, U26 TPS562208DDCT, U27 ADM7151ACPZ-04-R7, U28 TPS562208DDCT, U29 ADM7151ACPZ-04-R7, U3 TPS562208DDCT, U30 ADM7151ACPZ-04-R7, U31 TPS562208DDCT, U32 TPS7A8300RGRR, U33 TPS562208DDCT, U34 TPS7A8300RGRR, U35 TPS7A8300RGRR, U4 TPS562208DDCT, U5 ADM7151ACPZ-04-R7, U6 TPS562208DDCT, U7 TPS562208DDCT, U8 TPS562208DDCT, U9 TPS562208DDCT, X10 22-23-2021, X11 22-23-2021, X12 22-23-2021, X13 22-23-2021, X14 22-23-2021, X15 22-23-2021, X16 22-23-2021, X17 22-23-2021, X18 22-23-2021, X19 22-23-2021, X2 22-23-2021, X20 22-23-2021, X21 22-23-2021, X22 22-23-2021, X23 22-23-2021, X24 22-23-2021, X25 22-23-2021, X26 22-23-2021, X27 22-23-2021, X28 22-23-2021, X29 22-23-2021, X3 22-23-2021, X30 22-23-2021, X31 22-23-2021, X32 22-23-2021, X33 22-23-2021, X34 22-23-2021, X35 22-23-2021, X36 22-23-202122-23-2021, X4 22-23-2021, X5 22-23-2021, X6 22-23-2021, X7 22-23-2021, X8 22-23-2021, X9 22-23-2021

Commit message: fix(hw): four netlist defects, and the gate that should have caught them
Chasing the duplicated X36 board element turned up three more defects, and one of them was
electrical.  All four are mine, all from the B1.1 work.

1. Duplicate X36.  Upstream had 35 schematic X parts (X1-X35) but 36 board elements: X36
   existed *only* on the board, wired to +5V0_LO and GND, with no schematic counterpart.
   My B1.1 2.5 V connector then took the refdes X36 -- so the board carried two elements of
   that name while the BOM counted one, which is an assembly ambiguity, not a cosmetic one.
   Fixed the structurally correct way: my connector keeps X36 (it has a schematic part), and
   upstream's orphan element became X37 *and got the schematic part it never had*, so no
   board-only element is left.  BOM 35 -> 36 connectors.

2. Six U9 flash pinrefs used gate="G$1" when the flash's only gate is "A" (upstream writes
   U9 gate="A" pin="RESET").  A pinref naming a gate the part does not instantiate does not
   resolve -- so the B1.1 flash split was NOT actually connected to the flash.  This is the
   one that mattered: the nets now read U9 -> U90/U91 -> U42, i.e. the translators really are
   between the flash and the FPGA.

3. Both of my connectors (power X36, main X57) were instantiated with gate G$1 where the
   deviceset defines -1/-2.  Fixed.

4. None of this was detectable: the BOM/DNP/rail gates look at values, DNP marks and rail
   membership, never at element identity or pin ownership, so all four defects passed CI.

New gate: 9_Firmware/tools/netlist_integrity.py -- seven checks per board: duplicate
schematic-part and board-element designators; a pin claimed by more than one net; a board
element with no schematic part (orphan); a schematic part with no board element (unplaced);
a pinref naming an uninstantiated gate; a board element wired to nothing.  Supply and frame
symbols are exempt (schematic-only by design).  Wired into the CI artifact-gate step beside
the other thre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
Parts:
- added X37: 22-23-202122-23-2021, con-molex:22-23-202122-23-2021
Connections:
- net +5V0_LO: now also X37-1.S
- net GND: now also X37-2.S
Changed lines of the file:
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@@
 <part name="C162" library="rcl" library_urn="urn:adsk.eagle:library:334" deviceset="C-EU" device="C0603" package3d_urn="urn:adsk.eagle:package:23616/2" value="10nF"/>
 <part name="GND241" library="supply1" library_urn="urn:adsk.eagle:library:371" deviceset="GND" device=""/>
-<part name="C163" library="rcl" library_urn="urn:adsk.eagle:library:334" deviceset="C-EU" device="C0603" package3d_urn="urn:adsk.eagle:package:23616/2" value="10µF"/><part name="U35" library="My_Library_RADAR" deviceset="TPS7A8300RGRR" device=""/><part name="R59" library="rcl" deviceset="R-EU_" device="M0805" value="24.3k"/><part name="R60" library="rcl" deviceset="R-EU_" device="M0805" value="11.5k"/><part name="C164" library="rcl" deviceset="C-EU" device="C0603" value="22µF"/><part name="C165" library="rcl" deviceset="C-EU" device="C0603" value="22µF"/><part name="C166" library="rcl" deviceset="C-EU" device="C0603" value="10µF"/><part name="C167" library="rcl" deviceset="C-EU" device="C0603" value="10nF"/><part name="C168" library="rcl" deviceset="C-EU" device="C0603" value="10nF"/><part name="X36" library="con-molex" deviceset="22-23-2021" device="22-23-2021"/><part name="GND250" library="supply1" deviceset="GND" device=""/>
+<part name="C163" library="rcl" library_urn="urn:adsk.eagle:library:334" deviceset="C-EU" device="C0603" package3d_urn="urn:adsk.eagle:package:23616/2" value="10µF"/><part name="U35" library="My_Library_RADAR" deviceset="TPS7A8300RGRR" device=""/><part name="R59" library="rcl" deviceset="R-EU_" device="M0805" value="24.3k"/><part name="R60" library="rcl" deviceset="R-EU_" device="M0805" value="11.5k"/><part name="C164" library="rcl" deviceset="C-EU" device="C0603" value="22µF"/><part name="C165" library="rcl" deviceset="C-EU" device="C0603" value="22µF"/><part name="C166" library="rcl" deviceset="C-EU" device="C0603" value="10µF"/><part name="C167" library="rcl" deviceset="C-EU" device="C0603" value="10nF"/><part name="C168" library="rcl" deviceset="C-EU" device="C0603" value="10nF"/><part name="X37" library="con-molex" deviceset="22-23-2021" device="22-23-2021"/><part name="X36" library="con-molex" deviceset="22-23-2021" device="22-23-2021"/><part name="GND250" library="supply1" deviceset="GND" device=""/>
 <part name="GND242" library="supply1" library_urn="urn:adsk.eagle:library:371" deviceset="GND" device=""/>
 <part name="X4" library="con-molex" library_urn="urn:adsk.eagle:library:165" deviceset="22-23-2021" device="" package3d_urn="urn:adsk.eagle:package:8078633/1"/>
@@
 <attribute name="VALUE" x="515.62" y="256.54" size="1.778" layer="96"/>
 </instance>
-<instance part="U35" gate="G$1" x="169.8" y="136.8" smashed="yes"><attribute name="NAME" x="167.8" y="138.3" size="1.524" layer="95"/></instance><instance part="R59" gate="G$1" x="176.0" y="142.0" smashed="yes"><attribute name="NAME" x="174.0" y="143.5" size="1.524" layer="95"/></instance><instance part="R60" gate="G$1" x="180.0" y="148.0" smashed="yes"><attribute name="NAME" x="178.0" y="149.5" size="1.524" layer="95"/></instance><instance part="C164" gate="G$1" x="164.0" y="130.0" smashed="yes"><attribute name="NAME" x="162.0" y="131.5" size="1.524" layer="95"/></instance><instance part="C165" gate="G$1" x="182.0" y="130.0" smashed="yes"><attribute name="NAME" x="180.0" y="131.5" size="1.524" layer="95"/></instance><instance part="C166" gate="G$1" x="186.0" y="142.0" smashed="yes"><attribute name="NAME" x="184.0" y="143.5" size="1.524" layer="95"/></instance><instance part="C167" gate="G$1" x="190.0" y="148.0" smashed="yes"><attribute name="NAME" x="188.0" y="149.5" size="1.524" layer="95"/></instance><instance part="C168" gate="G$1" x="174.0" y="148.0" smashed="yes"><attribute name="NAME" x="172.0" y="149.5" size="1.524" layer="95"/></instance><instance part="X36" gate="G$1" x="192.0" y="134.3" smashed="yes"><attribute name="NAME" x="190.0" y="135.8" size="1.524" layer="95"/></instance><instance part="X36" gate="-2" x="192.0" y="131.76000000000002" smashed="yes"><attribute name="NAME" x="190.0" y="131.0" size="1.524" layer="95"/></instance><instance part="GND250" gate="1" x="170" y="150" smashed="yes"><attribute name="VALUE" x="171" y="151" size="1.778" layer="96"/></instance><instance part="U32" gate="A" x="589.28" y="266.7" smashed="yes">
+<instance part="U35" gate="G$1" x="169.8" y="136.8" smashed="yes"><attribute name="NAME" x="167.8" y="138.3" size="1.524" layer="95"/></instance><instance part="R59" gate="G$1" x="176.0" y="142.0" smashed="yes"><attribute name="NAME" x="174.0" y="143.5" size="1.524" layer="95"/></instance><instance part="R60" gate="G$1" x="180.0" y="148.0" smashed="yes"><attribute name="NAME" x="178.0" y="149.5" size="1.524" layer="95"/></instance><instance part="C164" gate="G$1" x="164.0" y="130.0" smashed="yes"><attribute name="NAME" x="162.0" y="131.5" size="1.524" layer="95"/></instance><instance part="C165" gate="G$1" x="182.0" y="130.0" smashed="yes"><attribute name="NAME" x="180.0" y="131.5" size="1.524" layer="95"/></instance><instance part="C166" gate="G$1" x="186.0" y="142.0" smashed="yes"><attribute name="NAME" x="184.0" y="143.5" size="1.524" layer="95"/></instance><instance part="C167" gate="G$1" x="190.0" y="148.0" smashed="yes"><attribute name="NAME" x="188.0" y="149.5" size="1.524" layer="95"/></instance><instance part="C168" gate="G$1" x="174.0" y="148.0" smashed="yes"><attribute name="NAME" x="172.0" y="149.5" size="1.524" layer="95"/></instance><instance part="X37" gate="-1" x="196.0" y="134.3" smashed="yes"><attribute name="NAME" x="194.0" y="135.8" size="1.524" layer="95"/></instance><instance part="X37" gate="-2" x="196.0" y="131.76" smashed="yes"><attribute name="NAME" x="194.0" y="131.0" size="1.524" layer="95"/></instance><instance part="X36" gate="-1" x="192.0" y="134.3" smashed="yes"><attribute name="NAME" x="190.0" y="135.8" size="1.524" layer="95"/></instance><instance part="X36" gate="-2" x="192.0" y="131.76000000000002" smashed="yes"><attribute name="NAME" x="190.0" y="131.0" size="1.524" layer="95"/></instance><instance part="GND250" gate="1" x="170" y="150" smashed="yes"><attribute name="VALUE" x="171" y="151" size="1.778" layer="96"/></instance><instance part="U32" gate="A" x="589.28" y="266.7" smashed="yes">
 <attribute name="NAME" x="607.4156" y="275.8186" size="2.0828" layer="95" ratio="6" rot="SR0"/>
 <attribute name="VALUE" x="606.7806" y="273.2786" size="2.0828" layer="96" ratio="6" rot="SR0"/>
@@
 <pinref part="X35" gate="-2" pin="S"/>
 <pinref part="GND249" gate="1" pin="GND"/>
-<pinref part="U35" gate="G$1" pin="GND"/><pinref part="U35" gate="G$1" pin="GND_2"/><pinref part="U35" gate="G$1" pin="EPAD"/><pinref part="R60" gate="G$1" pin="2"/><pinref part="C164" gate="G$1" pin="2"/><pinref part="C165" gate="G$1" pin="2"/><pinref part="C166" gate="G$1" pin="2"/><pinref part="C167" gate="G$1" pin="2"/><pinref part="X36" gate="-2" pin="S"/><pinref part="GND250" gate="1" pin="GND"/><pinref part="C169" gate="G$1" pin="2"/><pinref part="C170" gate="G$1" pin="2"/><pinref part="C171" gate="G$1" pin="2"/><pinref part="C172" gate="G$1" pin="2"/></segment>
+<pinref part="U35" gate="G$1" pin="GND"/><pinref part="U35" gate="G$1" pin="GND_2"/><pinref part="U35" gate="G$1" pin="EPAD"/><pinref part="R60" gate="G$1" pin="2"/><pinref part="C164" gate="G$1" pin="2"/><pinref part="C165" gate="G$1" pin="2"/><pinref part="C166" gate="G$1" pin="2"/><pinref part="C167" gate="G$1" pin="2"/><pinref part="X36" gate="-2" pin="S"/><pinref part="GND250" gate="1" pin="GND"/><pinref part="C169" gate="G$1" pin="2"/><pinref part="C170" gate="G$1" pin="2"/><pinref part="C171" gate="G$1" pin="2"/><pinref part="C172" gate="G$1" pin="2"/><pinref part="X37" gate="-2" pin="S"/></segment>
 </net>
 <net name="N$1" class="0">
@@
 <pinref part="X6" gate="-1" pin="S"/>
 <label x="27.94" y="195.58" size="1.778" layer="95" rot="R90"/>
-</segment>
+<pinref part="X37" gate="-1" pin="S"/></segment>
 </net>
 <net name="N$71" class="0">

Commit message: fix(hw): revert B1.5, connect the PG pins, and generate the harness map
Five fixes from the remaining-items plan. Two of them are corrections to work already
committed, and one is a correction to the plan itself.

REVERT B1.5.  Its premise was wrong.  The rail budget has -5V5_PA at 100 mA against a 200 mA
LM2662 -- 50 %, not "100 % of rating" as the item claimed -- while -5V0_ADAR12/34 are the
rails that are 1.2x over (240 mA vs 200 mA).  What was moved is negligible anyway: the
OPA4703 datasheet gives 200 uA per amplifier, so ~3 mA of quads plus ~1.6 mA of the new gate
pull-downs.  So the change added load to the two overloaded rails and left U22, C105 and one
harness connector feeding nothing.  All four OPA V- pins and all sixteen gate pull-downs are
back on -5V5_PA, which also puts each pull-down on the same negative rail as the op-amp it
backs up -- the better arrangement.  The real item is B3.1 (the ADAR negative rails).

B1.4/B3.2 PRECONDITION.  U32/U34/U35 each had a PG pin connected to nothing.  TPS7A8300 PG
is active-high open-drain asserting at 89 % of target, so it needs a pull-up to be a defined
level at all.  Nets PG_3V3_ADTR / PG_3V3_XO / PG_2V5_FPGA now carry the pin, and R61-R63
(10 kohm to +3V3) pull them up -- the signal names the connector decision will route.  10 kohm
rather than the datasheet's 100 kohm test condition, because the 10k/M0805 row and its
verified MPN (AE0805BR-0710KL) already exist and 330 uA vs 33 uA when asserted is immaterial
for a fault line.  This is needed by every routing option, so it is not gated on that
decision.

Correction to the plan, found while implementing: a single open-drain PG wire CANNOT be
fail-safe.  "Rail good" (high-Z) and "harness disconnected" are electrically identical no
matter which side carries the pull-up.  The plan claimed otherwise; the honest statement is
that the line is fail-silent on an open harness, and the mitigations are a firmware line-test
(drive low, release, read back) or accepting it.

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
Parts:
- added R61, R62, R63: 10k, rcl:R-EU_M0805
Connections:
- new net PG_2V5_FPGA: R63.1, U35.PG
- new net PG_3V3_ADTR: R61.1, U32.PG
- new net PG_3V3_XO: R62.1, U34.PG
- net +3V3: now also R61.2, R62.2, R63.2

Commit message: feat(backlog): close the six remaining Lane B decisions (#5 #7 #8 #9 #10 #24)
#5 PA operating mode: PA_BIAS_SEQUENCE.{h,c} make the gate/drain order a tested
   contract (enable: gate off -> drain -> settle -> operating bias; disable: gate
   off -> drain off; every failure path lands safe). 17/17, wired into startup and
   Emergency_Stop in main.cpp.
#7 harmonic filter: docs/harmonic-filter.md - spec, the existing SMA interface, the
   measurement that must set the filter order, and the three options.
#8 rail-good routing: three TPS7A8300 PG signals each get their own 2-position
   connector pair (power X38-X40 -> main X25-X27 -> U2.PC0-PC2, verified free).
   RAIL_FAULT.{h,c} samples and latches them, 19/19, wired into the main loop and
   telemetry. The pins are read with pull-downs, so an open harness reads LOW and is
   reported as a fault - the earlier "fail-silent" note was wrong and is corrected.
#9 negative rails: U36/U37 parallel U20/U21 on -5V0_ADAR12/34, each with its own
   47 uF pumping cap and the shared output cap, exactly as TI's datasheet requires.
   Two in parallel halve the output resistance and double the headroom (240 mA of a
   400 mA capability instead of 1.2x over a 200 mA part).
#10 keying: negative rails move to the 3-position part and the PA drain feeds to a
   4-position part with two pins per rail (which also halves the 4 A per pin). The
   4-position part is authored from the repo's own 22-23-2031 geometry. One rail was
   spelled two ways across boards (+3V3_ADAR_12 vs +3V3_ADAR12) and is now unified.
   The harness map's keying column is generated from the parts, not typed.
#24 laminate: the PA board moves to RO4350B (recorded in FAB_NOTES.md); the patch
   array is gerbers-only and flagged as un-respinnable.

Verification: netlist_integrity caught two real regressions during this work (gate
names the part did not instantiate; designators dropped from the authored BOM) and
both are fixed. All six artifact gates and ruff are green.
Parts:
- added C173, C174: T521W476M020ATE045, T521W476M020ATE045:T521W476M020ATE045
- added U36, U37: LM2662MX/NOPB, My_Library_RADAR:LM2662MX/NOPB
- added X38, X39, X40: 22-23-202122-23-2021, con-molex:22-23-202122-23-2021
- X18, X19, X20, X21, X24: value 22-23-2021 -> 22-23-203122-23-2031; device con-molex:22-23-2021 -> con-molex:22-23-203122-23-2031
- X31, X32, X33: value 22-23-2021 -> 22-23-204122-23-2041; device con-molex:22-23-2021 -> con-molex:22-23-204122-23-2041
Connections:
- net +3V3_ADAR_12 renamed +3V3_ADAR12
- net +3V3_ADAR_34 renamed +3V3_ADAR34
- new net N$U36_C1M: C173.2, U36.C1-
- new net N$U36_C1P: C173.1, U36.C1+
- new net N$U37_C1M: C174.2, U37.C1-
- new net N$U37_C1P: C174.1, U37.C1+
- net +5V0_ADAR: now also U36.V+, U37.V+
- net +5V0_PA_1: now also X31.S; no longer X31-1.S
- net +5V0_PA_2: now also X32.S; no longer X32-1.S
- net +5V0_PA_3: now also X33.S; no longer X33-1.S
- net -3V3_SW: now also X18.S; no longer X18-1.S
- net -3V4: now also X24.S; no longer X24-1.S
- net -5V0_ADAR12: now also U36.OUT, X21.S; no longer X21-1.S
- net -5V0_ADAR34: now also U37.OUT, X20.S; no longer X20-1.S
- net -5V5_PA: now also X19.S; no longer X19-1.S
- net GND: now also U36.GND, U36.LV, U37.GND, U37.LV, X18.S, X19.S, X20.S, X21.S, X24.S, X31.S, X32.S, X33.S, X38-2.S, X39-2.S, X40-2.S; no longer X18-2.S, X19-2.S, X20-2.S, X21-2.S, X24-2.S, X31-2.S, X32-2.S, X33-2.S
- net PG_2V5_FPGA: now also X40-1.S
- net PG_3V3_ADTR: now also X38-1.S
- net PG_3V3_XO: now also X39-1.S
