File: 4_Schematics and Boards Layout/4_6_Schematics/PowerBoard/PowerBoard.sch (EAGLE design)
At the start: 336 parts, among them U1 TPS562208DDCT, U10 TPS562208DDCT, U11 TPS562208DDCT, U12 TPS562208DDCT, U13 TPS562208DDCT, U14 TPS562208DDCT, U15 TPS562208DDCT, U16 TPS562208DDCT, U17 TPS562208DDCT, U18 LM2662MX/NOPB, U19 LM2662MX/NOPB, U2 TPS562208DDCT, U20 LM2662MX/NOPB, U21 LM2662MX/NOPB, U22 LM2662MX/NOPB, U23 ADM7151ACPZ-04-R7, U24 TPS562208DDCT, U25 ADM7151ACPZ-04-R7, U26 TPS562208DDCT, U27 ADM7151ACPZ-04-R7, U28 TPS562208DDCT, U29 ADM7151ACPZ-04-R7, U3 TPS562208DDCT, U30 ADM7151ACPZ-04-R7, U31 TPS562208DDCT, U32 TPS7A8300RGRR, U33 TPS562208DDCT, U34 TPS7A8300RGRR, U35 TPS7A8300RGRR, U36 LM2662MX/NOPB, U37 LM2662MX/NOPB, U4 TPS562208DDCT, U5 ADM7151ACPZ-04-R7, U6 TPS562208DDCT, U7 TPS562208DDCT, U8 TPS562208DDCT, U9 TPS562208DDCT, X10 22-23-2021, X11 22-23-2021, X12 22-23-2021, X13 22-23-2021, X14 22-23-2021, X15 22-23-2021, X16 22-23-2021, X17 22-23-2021, X18 22-23-203122-23-2031, X19 22-23-203122-23-2031, X2 22-23-2021, X20 22-23-203122-23-2031, X21 22-23-203122-23-2031, X22 22-23-2021, X23 22-23-2021, X24 22-23-203122-23-2031, X25 22-23-2021, X26 22-23-2021, X27 22-23-2021, X28 22-23-2021, X29 22-23-2021, X3 22-23-2021, X30 22-23-2021, X31 22-23-204122-23-2041, X32 22-23-204122-23-2041, X33 22-23-204122-23-2041, X34 22-23-2021, X35 22-23-2021, X36 22-23-202122-23-2021, X37 22-23-202122-23-2021, X38 22-23-202122-23-2021, X39 22-23-202122-23-2021, X4 22-23-2021, X40 22-23-202122-23-2021, X5 22-23-2021, X6 22-23-2021, X7 22-23-2021, X8 22-23-2021, X9 22-23-2021

Commit message: feat(hw): ADAR supply order, test points, strobe acknowledgement (#13 #15 #20)
#20 ADAR1000 supply order - the requirement, verified and locked
  The pin table says AVDD3 (+3.3 V) must come up "before or at the same time as the
  AVDD1(-5V) supply"; the "−5 V first" sentence elsewhere in the same datasheet is about an
  external PA's drain (the gate-bias rule).  The firmware already asserts the 3.3 V ADAR rails
  before the 5.0 V rail that creates -5 V through the LM2662 inverters, so this needed no code
  change - it needed the requirement written down at the call site and a test that fails if a
  later edit swaps the order.  docs/power-up-order.md records every device's requirement with
  its citation (ADAR1000 pin table, ADTR1107 Recommended Bias Sequencing, M3SWA2 dual supply,
  LTC5552/AD8352 single supply) and the structural fact that every negative rail here is
  inverted from a positive one, so "negative first" is not physically available.

#15 test points - 15 added where there were zero
  The Harwin S1751-46R (1.63 x 3.25 mm SMT test point, two pads on one node) authored from its
  own land pattern, placed on the power board at the bring-up rails and the three rail-good
  signals, with a BOM row.  docs/probe-map.md already said which pin to meter; this gives the
  probe somewhere to land.

#13 strobe acknowledgement - the MCU can now tell whether the FPGA acted
  strobe_ack.v turns the top's accepted-frame pulse into a level the MCU can poll: a request
  clears it, consumption sets it, so "still low at the next request" means the strobe was
  dropped.  Wired from the already-synchronized pulse, exposed through the 50T wrapper,
  constrained to B16 (bank 15, LVCMOS33 - the same bank as the strobes it answers, so no level
  shift), and carried in the netlist from U42 to U2.PC3.  The FPGA's config net (DONE with
  INIT_B and their pull-ups) now reaches U2.PC4 as FPGA_CFG_OK.  MCU side: STROBE_ACK.{h,c}
  scores each request before the next one is issued - the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
Parts:
- added TP1, TP10, TP11, TP12, TP13, TP14, TP15, TP2, TP3, TP4, TP5, TP6, TP7, TP8, TP9: S1751-46, My_Library_RADAR:S1751-46
Connections:
- net +1V0_FPGA: now also TP1.S
- net +1V8_FPGA: now also TP2.S
- net +2V5_FPGA: now also TP3.S
- net +3V3: now also TP4.S
- net +3V3_ADAR12: now also TP8.S
- net +3V3_ADTR: now also TP6.S
- net +3V3_AN: now also TP5.S
- net +3V3_XO: now also TP7.S
- net +3V4: now also TP10.S
- net +5V5_PA: now also TP12.S
- net -3V4: now also TP11.S
- net -5V0_ADAR12: now also TP9.S
- net PG_2V5_FPGA: now also TP15.S
- net PG_3V3_ADTR: now also TP13.S
- net PG_3V3_XO: now also TP14.S
