File: 4_Schematics and Boards Layout/4_6_Schematics/FrequencySynthesizerBoard/Clocks_Freq_Synth_board.sch (EAGLE design)
At the start: 184 parts, among them IC1 AD9523BCPZ, J1 142-0731-211, J10 142-0731-211, J11 142-0731-211, J12 142-0731-211, J13 142-0731-211, J2 142-0731-211, J3 CJT-T-P-HH-ST-TH1, J4 CJT-T-P-HH-ST-TH1, J5 142-0731-211, J6 142-0731-211, J7 142-0731-211, J8 142-0731-211, J9 142-0731-211, U1 ADF4382ABCCZ, U10 ATS1005-3DB-FD-T05, U2 MTX2-143+, U3 MTX2-143+, U4 ATS1005-3DB-FD-T05, U5 ATS1005-3DB-FD-T05, U6 ADF4382ABCCZ, U7 MTX2-143+, U8 ATS1005-3DB-FD-T05, U9 MTX2-143+, X10 22-23-2021, X11 22-23-2021, X12 22-23-2021, X13 22-23-2021, X14 22-23-2021, X15 22-23-2021, X4 ECOC-2522-100.000-3HC, X5 CVHD-950-50.000, X6 CVHD-950-50.000

Commit message: fix(#17 #21): name the clock nets the issue suspected, and research the PA decision inputs
#17 - the parenthetical in the issue ("AD9523_OUT6 is nearly as thin (only R39)") is a symptom, not a
fault.  Tracing it: the chain is complete - IC1.OUT6 -> R39 (22R) -> C15 (10nF) -> J7 - and it is
structurally identical to OUT10 (R40) and OUT11 (R41), which nobody questioned.  What made it read as
a fault is that the driver side of the series resistor carries an anonymous N$ name, so a reader
checking the netlist sees a connector with no source.

So the fix is the naming, not the wiring: N$62 -> AD9523_OUT6_DRV, N$63 -> AD9523_OUT6_SER,
N$65 -> AD9523_OUT10_SER, N$68 -> AD9523_OUT11_SER, in both the schematic and the board.  The script
verifies what each net carries before renaming and refuses if a target is wrong.

No electrical change.  Eight gates green, ruff clean, no stale references.

#21 - the decision inputs, researched from primary sources:

  * Export classification, from Qorvo's own ECCN endpoint rather than a distributor's guess:
    QPA2962 is 3A001.B.2.C, QPA1010 is 3A001.B.2.B.2, and BOTH are export-controlled.  The migration
    does not buy an easier classification.  The evaluation boards are EAR99, which is a practical
    route for evaluation.  Given as the manufacturer's classification plus the vendor pattern
    (high-power X-band GaN parts carry b.2.b.2; broadband driver MMICs carry b.2.c), not as the letter
    of the regulation.

  * Availability, and this reverses the picture: Mouser lists the incumbent QPA2962 as "Lifecycle:
    Restricted ... not currently available", while QPA1010TR7 at DigiKey is "buy now, ships today".
    The part in the current design is the one with the availability problem.

  * Minimum order: the candidate's packaged variant is a 250-piece reel (or die), while the incumbent
    offers 2- and 25-piece options.

So migrating would halve the thermal load, remove the RoHS gap, and use a part that is in stock
rather than one th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
Connections:
- net N$62 renamed AD9523_OUT6_DRV
- net N$63 renamed AD9523_OUT6_SER
- net N$65 renamed AD9523_OUT10_SER
- net N$68 renamed AD9523_OUT11_SER
Changed lines of the file:
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@@
 </segment>
 </net>
-<net name="N$62" class="0">
+<net name="AD9523_OUT6_DRV" class="0">
 <segment>
 <pinref part="IC1" gate="G$1" pin="OUT6"/>
@@
 </segment>
 </net>
-<net name="N$63" class="0">
+<net name="AD9523_OUT6_SER" class="0">
 <segment>
 <pinref part="R39" gate="G$1" pin="2"/>
@@
 </segment>
 </net>
-<net name="N$65" class="0">
+<net name="AD9523_OUT10_SER" class="0">
 <segment>
 <pinref part="C17" gate="G$1" pin="1"/>
@@
 </segment>
 </net>
-<net name="N$68" class="0">
+<net name="AD9523_OUT11_SER" class="0">
 <segment>
 <pinref part="C19" gate="G$1" pin="1"/>
